File: Pojet_V-NOM_KiCAD/_autosave-deplacement.kicad_sch (KiCad schematic)
At the start: 8 parts, among them J301 Conn_01x06, J302 Conn_01x06, U301 ZXBM5210-SP, U302 ZXBM5210-SP

Commit message: Update _autosave-deplacement.kicad_sch
Connections:
- net GND: now also J301.2 (Pin_2), J302.2 (Pin_2)
- net PB6: now also J302.4 (Pin_4)
- net at J302.1 (Pin_1): now also U302.7 (OUT2); no longer U302.1 (OUT1)
- net PB5: now reaches J302.3 (Pin_3)
- net +5V: now reaches J302.5 (Pin_5)
- net +5V: now also J301.5 (Pin_5)
- net at J302.6 (Pin_6): now also U302.1 (OUT1); no longer U302.7 (OUT2)
- net at U301.1 (OUT1): now also J301.6 (Pin_6); no longer J301.1 (Pin_1)
- net at U301.7 (OUT2): now also J301.1 (Pin_1); no longer J301.6 (Pin_6)
- net PA5: now reaches J301.3 (Pin_3)
- net PA6: now reaches J301.4 (Pin_4)
