File: Pojet_V-NOM_KiCAD/Pojet_V-NOM_KiCAD.kicad_sch (KiCad schematic)
At the start: 0 parts

Commit message: Mise à jour du schéma de contrôle
Parts:
- added H1, H2, H3, H4: MountingHole_Pad, MountingHole:MountingHole_3.2mm_M3_Pad_Via, symbol Mechanical:MountingHole_Pad
Connections:
- new net GND: H1.1, H2.1, H3.1, H4.1

Commit message: Mise à jour du schéma principal
Other:
- sheet controle ports: added LED_GREEN, LED_RED, NRST, SPI1_CSN; removed none
Changed lines of the file:
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@@
+	(wire
+		(pts
+			(xy 137.16 148.59) (xy 137.16 156.21)
+		)
+		(stroke
+			(width 0)
+			(type default)
+		)
+	)
+	(wire
+		(pts
+			(xy 180.34 154.94) (xy 180.34 127)
+		)
+		(stroke
+			(width 0)
+			(type default)
+		)
+	)
 	(wire
 		(pts
@@
 	(wire
 		(pts
+			(xy 139.7 154.94) (xy 180.34 154.94)
+		)
+		(stroke
+			(width 0)
+			(type default)
+		)
+	)
+	(wire
+		(pts
+			(xy 182.88 152.4) (xy 182.88 133.35)
+		)
+		(stroke
+			(width 0)
+			(type default)
+		)
+	)
+	(wire
+		(pts
+			(xy 83.82 144.78) (xy 110.49 144.78)
+		)
+		(stroke
+			(width 0)
+			(type default)
+		)
+	)
+	(wire
+		(pts
 			(xy 83.82 139.7) (xy 110.49 139.7)
 		)
@@
 	(wire
 		(pts
+			(xy 142.24 148.59) (xy 142.24 153.67)
+		)
+		(stroke
+			(width 0)
+			(type default)
+		)
+	)
+	(wire
+		(pts
+			(xy 180.34 127) (xy 185.42 127)
+		)
+		(stroke
+			(width 0)
+			(type default)
+		)
+	)
+	(wire
+		(pts
+			(xy 137.16 156.21) (xy 179.07 156.21)
+		)
+		(stroke
+			(width 0)
+			(type default)
+		)
+	)
+	(wire
+		(pts
+			(xy 144.78 152.4) (xy 182.88 152.4)
+		)
+		(stroke
+			(width 0)
+			(type default)
+		)
+	)
+	(wire
+		(pts
+			(xy 142.24 153.67) (xy 181.61 153.67)
+		)
+		(stroke
+			(width 0)
+			(type default)
+		)
+	)
+	(wire
+		(pts
 			(xy 140.97 95.25) (xy 135.89 95.25)
 		)
@@
 	(wire
 		(pts
+			(xy 181.61 153.67) (xy 181.61 130.81)
+		)
+		(stroke
+			(width 0)
+			(type default)
+		)
+	)
+	(wire
+		(pts
 			(xy 113.03 31.75) (xy 181.61 31.75)
 		)
@@
 	(wire
 		(pts
+			(xy 179.07 156.21) (xy 179.07 124.46)
+		)
+		(stroke
+			(width 0)
+			(type default)
+		)
+	)
+	(wire
+		(pts
 			(xy 265.43 26.67) (xy 265.43 27.94)
 		)
@@
 	(wire
 		(pts
+			(xy 144.78 148.59) (xy 144.78 152.4)
+		)
+		(stroke
+			(width 0)
+			(type default)
+		)
+	)
+	(wire
+		(pts
 			(xy 143.51 95.25) (xy 140.97 95.25)
 		)
@@
 	(wire
 		(pts
+			(xy 83.82 114.3) (xy 110.49 114.3)
+		)
+		(stroke
+			(width 0)
+			(type default)
+		)
+	)
+	(wire
+		(pts
 			(xy 265.43 26.67) (xy 262.89 26.67)
 		)
@@
 	(wire
 		(pts
+			(xy 181.61 130.81) (xy 185.42 130.81)
+		)
+		(stroke
+			(width 0)
+			(type default)
+		)
+	)
+	(wire
+		(pts
 			(xy 83.82 137.16) (xy 110.49 137.16)
 		)
@@
 	(wire
 		(pts
+			(xy 83.82 111.76) (xy 110.49 111.76)
+		)
+		(stroke
+			(width 0)
+			(type default)
+		)
+	)
+	(wire
+		(pts
 			(xy 262.89 26.67) (xy 262.89 25.4)
 		)
@@
 	(wire
 		(pts
+			(xy 139.7 148.59) (xy 139.7 154.94)
+		)
+		(stroke
+			(width 0)
+			(type default)
+		)
+	)
+	(wire
+		(pts
 			(xy 215.9 83.82) (xy 215.9 92.71)
 		)
@@
 	(wire
 		(pts
+			(xy 179.07 124.46) (xy 185.42 124.46)
+		)
+		(stroke
+			(width 0)
+			(type default)
+		)
+	)
+	(wire
+		(pts
 			(xy 133.35 95.25) (xy 128.27 95.25)
 		)
@@
 		(pts
 			(xy 267.97 25.4) (xy 267.97 26.67)
+		)
+		(stroke
+			(width 0)
+			(type default)
+		)
+	)
+	(wire
+		(pts
+			(xy 182.88 133.35) (xy 185.42 133.35)
 		)
 		(stroke
@@
 			)
 		)
+		(pin "NRST" input
+			(at 110.49 144.78 180)
+			(effects
+				(font
+					(size 1.27 1.27)
+				)
+				(justify left)
+			)
+		)
+		(pin "SPI1_CSN" output
+			(at 130.81 95.25 90)
+			(effects
+				(font
+					(size 1.27 1.27)
+				)
+				(justify right)
+			)
+		)
+		(pin "LED_RED" output
+			(at 110.49 114.3 180)
+			(effects
+				(font
+					(size 1.27 1.27)
+				)
+				(justify left)
+			)
+		)
+		(pin "LED_GREEN" output
+			(at 110.49 111.76 180)
+			(effects
+				(font
+					(size 1.27 1.27)
+				)
+				(justify left)
+			)
+		)
 		(instances
 			(project "Pojet_V-NOM_KiCAD"
@@
 		)
 		(pin "LED_SOURIS" input
-			(at 83.82 106.68 0)
+			(at 83.82 111.76 0)
 			(effects
 				(font
@@
 		)
 		(pin "LED_CHAT" input
-			(at 83.82 109.22 0)
-			(effects
-				(font
+			(at 83.82 114.3 0)
+			(effects
+				(font

Commit message: Mise à jour du schéma principal
Other:
- sheet Deplacement ports: added none; removed +7.2V
- sheet acquisition ports: added AG_CSN, AG_INT1, AG_INT2, AG_SCLK, AG_SDA, TOF1, TOF2; removed +3.3V, +5V, CS, SDA, Vo_1, Vo_2, sclk
- sheet controle ports: added none; removed 3.3V

Commit message: Maj
Maj lidar et regualteur
Other:
- sheet acquisition ports: added +3.3V, +5V; removed DEV_EN, M_EN, M_SCTR
Changed lines of the file:
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@@
 	(wire
 		(pts
-			(xy 143.51 40.005) (xy 171.45 40.005)
+			(xy 143.51 40.64) (xy 171.45 40.64)
 		)
 		(stroke
@@
 	(wire
 		(pts
-			(xy 146.05 42.545) (xy 171.45 42.545)
+			(xy 146.05 43.18) (xy 171.45 43.18)
 		)
 		(stroke
@@
 	(wire
 		(pts
-			(xy 146.05 71.12) (xy 146.05 42.545)
+			(xy 146.05 71.12) (xy 146.05 43.18)
 		)
 		(stroke
@@
 	(wire
 		(pts
-			(xy 143.51 71.12) (xy 143.51 40.005)
+			(xy 143.51 71.12) (xy 143.51 40.64)
 		)
 		(stroke
@@
 			)
 		)
-		(pin "TX_LIDAR" passive
-			(at 171.45 40.005 180)
-			(effects
-				(font
-					(size 1.27 1.27)
-				)
-				(justify left)
-			)
-		)
-		(pin "RX_LIDAR" passive
-			(at 171.45 42.545 180)
-			(effects
-				(font
-					(size 1.27 1.27)
-				)
-				(justify left)
-			)
-		)
 		(pin "INT1_ACCEL" output
 			(at 171.45 47.625 180)
@@
 			)
 		)
-		(pin "M_SCTR" passive
-			(at 171.45 56.515 180)
-			(effects
-				(font
-					(size 1.27 1.27)
-				)
-				(justify left)
-			)
-		)
-		(pin "DEV_EN" passive
-			(at 171.45 59.055 180)
-			(effects
-				(font
-					(size 1.27 1.27)
-				)
-				(justify left)
-			)
-		)
-		(pin "M_EN" passive
-			(at 171.45 61.595 180)
-			(effects
-				(font
-					(size 1.27 1.27)
-				)
-				(justify left)
-			)
-		)
 		(pin "TOF2" output
 			(at 171.45 34.925 180)
@@
 			(effects
 				(font
+					(size 1.27 1.27)
+				)
+				(justify left)
+			)
+		)
+		(pin "+5V" input
+			(at 196.85 17.145 90)
+			(effects
+				(font
+					(size 1.27 1.27)
+				)
+				(justify right)
+			)
+		)
+		(pin "+3.3V" input
+			(at 190.5 17.145 90)
+			(effects
+				(font
+					(size 1.27 1.27)
+				)
+				(justify right)
+			)
+		)
+		(pin "RX_LIDAR" input
+			(at 171.45 43.18 180)
+			(effects
+				(font
+					(size 1.27 1.27)
+				)
+				(justify left)
+			)
+		)
+		(pin "TX_LIDAR" output
+			(at 171.45 40.64 180)
+			(effects
+				(font

Commit message: maj
Other:
- sheet Deplacement ports: added +7.2V; removed none
- sheet alimentation ports: added none; removed +3.3V, +5V
Changed lines of the file:
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@@
+	(wire
+		(pts
+			(xy 215.9 130.81) (xy 81.28 130.81)
+		)
+		(stroke
+			(width 0)
+			(type default)
+		)
+	)
 	(wire
 		(pts
@@
 		(pts
 			(xy 146.05 71.12) (xy 143.51 71.12)
+		)
+		(stroke
+			(width 0)
+			(type default)
+		)
+	)
+	(wire
+		(pts
+			(xy 81.28 130.81) (xy 81.28 140.97)
 		)
 		(stroke
@@
 			)
 		)
+		(pin "+7.2V" input
+			(at 81.28 140.97 90)
+			(effects
+				(font
+					(size 1.27 1.27)
+				)
+				(justify right)
+			)
+		)
 		(instances
 			(project "Pojet_V-NOM_KiCAD"
@@
 			)
 		)
-		(pin "+3.3V" output
-			(at 215.9 146.05 180)
-			(effects
-				(font
-					(size 1.27 1.27)
-				)
-				(justify left)
-			)
-		)
-		(pin "+5V" output
-			(at 215.9 139.7 180)
-			(effects
-				(font
-					(size 1.27 1.27)
-				)
-				(justify left)
-			)
-		)

Commit message: maj
Other:
- sheet acquisition ports: added none; removed +3.3V, +5V
Changed lines of the file:
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@@
-			)
-		)
-		(pin "+5V" input
-			(at 196.85 17.145 90)
-			(effects
-				(font
-					(size 1.27 1.27)
-				)
-				(justify right)
-			)
-		)
-		(pin "+3.3V" input
-			(at 190.5 17.145 90)
-			(effects
-				(font
-					(size 1.27 1.27)
-				)
-				(justify right)
 			)
 		)
