File: Pojet_V-NOM_KiCAD/Pojet_V-NOM_KiCAD.kicad_sch (KiCad schematic)
At the start: 4 parts

Commit message: Correction schéma accéléromètre
Other:
- sheet acquisition ports: added AG_SDI, AG_SDO; removed AG_SDA
Changed lines of the file:
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@@
+	(wire
+		(pts
+			(xy 205.74 95.25) (xy 162.56 95.25)
+		)
+		(stroke
+			(width 0)
+			(type default)
+		)
+	)
 	(wire
 		(pts
@@
 	(wire
 		(pts
+			(xy 208.28 64.77) (xy 208.28 97.79)
+		)
+		(stroke
+			(width 0)
+			(type default)
+		)
+	)
+	(wire
+		(pts
 			(xy 144.78 124.46) (xy 144.78 146.05)
 		)
@@
 	(wire
 		(pts
+			(xy 208.28 97.79) (xy 162.56 97.79)
+		)
+		(stroke
+			(width 0)
+			(type default)
+		)
+	)
+	(wire
+		(pts
 			(xy 146.05 71.12) (xy 143.51 71.12)
 		)
@@
 		(pts
 			(xy 57.15 41.91) (xy 57.15 43.18)
+		)
+		(stroke
+			(width 0)
+			(type default)
+		)
+	)
+	(wire
+		(pts
+			(xy 205.74 64.77) (xy 205.74 95.25)
 		)
 		(stroke
@@
 		)
 		(pin "AG_INT1" output
-			(at 203.2 64.77 270)
+			(at 215.9 64.77 270)
 			(effects
 				(font
@@
 		)
 		(pin "AG_INT2" output
-			(at 205.74 64.77 270)
+			(at 218.44 64.77 270)
 			(effects
 				(font
@@
 			)
 		)
-		(pin "AG_SDA" input
-			(at 208.28 64.77 270)
-			(effects
-				(font
-					(size 1.27 1.27)
-				)
-				(justify left)
-			)
-		)
 		(pin "AG_SCLK" input
 			(at 210.82 64.77 270)
@@
 			(effects
 				(font
+					(size 1.27 1.27)
+				)
+				(justify left)
+			)
+		)
+		(pin "AG_SDI" input
+			(at 205.74 64.77 270)
+			(effects
+				(font
+					(size 1.27 1.27)
+				)
+				(justify left)
+			)
+		)
+		(pin "AG_SDO" input
+			(at 208.28 64.77 270)
+			(effects
+				(font

Commit message: Branchement final de l'accéléromètre
Other:
- sheet controle ports: added AG_INT1, AG_INT2; removed none
Changed lines of the file:
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@@
+	(wire
+		(pts
+			(xy 218.44 107.95) (xy 162.56 107.95)
+		)
+		(stroke
+			(width 0)
+			(type default)
+		)
+	)
+	(wire
+		(pts
+			(xy 215.9 105.41) (xy 162.56 105.41)
+		)
+		(stroke
+			(width 0)
+			(type default)
+		)
+	)
 	(wire
 		(pts
@@
 	(wire
 		(pts
+			(xy 215.9 64.77) (xy 215.9 105.41)
+		)
+		(stroke
+			(width 0)
+			(type default)
+		)
+	)
+	(wire
+		(pts
 			(xy 129.54 124.46) (xy 129.54 157.48)
 		)
@@
 		(pts
 			(xy 142.24 124.46) (xy 142.24 149.86)
+		)
+		(stroke
+			(width 0)
+			(type default)
+		)
+	)
+	(wire
+		(pts
+			(xy 218.44 64.77) (xy 218.44 107.95)
 		)
 		(stroke
@@
 			)
 		)
+		(pin "AG_INT2" input
+			(at 162.56 107.95 0)
+			(effects
+				(font
+					(size 1.27 1.27)
+				)
+				(justify right)
+			)
+		)
+		(pin "AG_INT1" input
+			(at 162.56 105.41 0)
+			(effects
+				(font
+					(size 1.27 1.27)
+				)
+				(justify right)
+			)
+		)

Commit message: maj regulateur 5V
Other:
- sheet acquisition ports: added none; removed INT1_ACCEL, INT2_ACCEL
Changed lines of the file:
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@@
-			)
-		)
-		(pin "INT1_ACCEL" output
-			(at 171.45 47.625 180)
-			(effects
-				(font
-					(size 1.27 1.27)
-				)
-				(justify left)
-			)
-		)
-		(pin "INT2_ACCEL" output
-			(at 171.45 50.165 180)
-			(effects
-				(font
-					(size 1.27 1.27)
-				)
-				(justify left)
 			)
 		)
@@
 			)
 		)
-		(pin "AG_SDO" input
+		(pin "AG_SDO" output
 			(at 208.28 64.77 270)
 			(effects
@@
 			)
 		)
-		(pin "SPI_MISO" bidirectional
-			(at 162.56 97.79 0)
-			(effects
-				(font
-					(size 1.27 1.27)
-				)
-				(justify right)
-			)
-		)
-		(pin "SPI_SCK" bidirectional
-			(at 162.56 100.33 0)
-			(effects
-				(font
-					(size 1.27 1.27)
-				)
-				(justify right)
-			)
-		)
 		(pin "TIM1_CH1" output
 			(at 127 124.46 270)
@@
 			(effects
 				(font
+					(size 1.27 1.27)
+				)
+				(justify right)
+			)
+		)
+		(pin "SPI_MISO" input
+			(at 162.56 97.79 0)
+			(effects
+				(font
+					(size 1.27 1.27)
+				)
+				(justify right)
+			)
+		)
+		(pin "SPI_SCK" output
+			(at 162.56 100.33 0)
+			(effects
+				(font

Commit message: Corrections rapides du schéma global
Other:
- sheet controle ports: added none; removed AG_USART_RX, AG_USART_TX
Changed lines of the file:
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@@
-	(wire
-		(pts
-			(xy 153.67 71.12) (xy 151.13 71.12)
-		)
-		(stroke
-			(width 0)
-			(type default)
-		)
-	)
 	(wire
 		(pts
@@
 			)
 		)
-		(pin "AG_USART_TX" bidirectional
-			(at 151.13 71.12 90)
-			(effects
-				(font
-					(size 1.27 1.27)
-				)
-				(justify right)
-			)
-		)
 		(pin "TIM3_CH2" output
 			(at 142.24 124.46 270)
@@
 			)
 		)
-		(pin "AG_USART_RX" bidirectional
-			(at 153.67 71.12 90)
-			(effects
-				(font
-					(size 1.27 1.27)
-				)
-				(justify right)
-			)
-		)

Commit message: Correction du schéma global
Other:
- sheet interface_utilisateur ports: added none; removed SWO
Changed lines of the file:
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@@
-			)
-		)
-		(pin "SWO" output
-			(at 86.36 118.11 0)
-			(effects
-				(font
-					(size 1.27 1.27)
-				)
-				(justify right)
 			)
 		)

Commit message: DERNIER MODIF Alim
Other:
- sheet Deplacement ports: added none; removed +7.2V
- sheet alimentation ports: added none; removed +7.2V
Changed lines of the file:
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@@
-	(wire
-		(pts
-			(xy 45.72 158.75) (xy 55.88 158.75)
-		)
-		(stroke
-			(width 0)
-			(type default)
-		)
-	)
 	(wire
 		(pts
@@
 			)
 		)
-		(pin "+7.2V" input
-			(at 55.88 158.75 180)
-			(effects
-				(font
-					(size 1.27 1.27)
-				)
-				(justify left)
-			)
-		)
 		(instances
 			(project "Pojet_V-NOM_KiCAD"
@@
 			)
 		)
-		(pin "+7.2V" output
-			(at 45.72 158.75 0)
-			(effects
-				(font
-					(size 1.27 1.27)
-				)
-				(justify right)
-			)
-		)

Commit message: Fix boutons poussoirs + BTN_START
Other:
- sheet controle ports: added none; removed BTN_RESET
- sheet interface_utilisateur ports: added BTN_START; removed none
Changed lines of the file:
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@@
+	(wire
+		(pts
+			(xy 86.36 95.25) (xy 113.03 95.25)
+		)
+		(stroke
+			(width 0)
+			(type default)
+		)
+	)
 	(wire
 		(pts
@@
 			)
 		)
-		(pin "BTN_RESET" input
-			(at 113.03 100.33 180)
-			(effects
-				(font
-					(size 1.27 1.27)
-				)
-				(justify left)
-			)
-		)
 		(pin "BTN_MODE" input
 			(at 113.03 97.79 180)
@@
 			(effects
 				(font
+					(size 1.27 1.27)
+				)
+				(justify right)
+			)
+		)
+		(pin "BTN_START" output
+			(at 86.36 95.25 0)
+			(effects
+				(font

Commit message: Modifications conseillés par l'enseignant
Other:
- sheet acquisition ports: added AG_MISO, AG_MOSI, EN_LIDAR, EN_MOT, VIT_MOT_LIDAR; removed AG_SDI, AG_SDO
Changed lines of the file:
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@@
-	)
-	(junction
-		(at 146.05 71.12)
-		(diameter 0)
-		(color 0 0 0 0)
-	)
-	(junction
-		(at 135.89 71.12)
-		(diameter 0)
-		(color 0 0 0 0)
-	)
-	(junction
-		(at 143.51 71.12)
-		(diameter 0)
-		(color 0 0 0 0)
-	)
-	(junction
-		(at 138.43 71.12)
-		(diameter 0)
-		(color 0 0 0 0)
 	)
 	(junction
@@
 	(wire
 		(pts
-			(xy 143.51 40.64) (xy 171.45 40.64)
-		)
-		(stroke
-			(width 0)
-			(type default)
-		)
-	)
-	(wire
-		(pts
 			(xy 134.62 167.64) (xy 123.19 167.64)
 		)
@@
 	(wire
 		(pts
-			(xy 146.05 43.18) (xy 171.45 43.18)
+			(xy 132.08 124.46) (xy 132.08 132.08)
 		)
 		(stroke
@@
 	(wire
 		(pts
+			(xy 246.38 132.08) (xy 246.38 64.77)
+		)
+		(stroke
+			(width 0)
+			(type default)
+		)
+	)
+	(wire
+		(pts
 			(xy 86.36 115.57) (xy 113.03 115.57)
 		)
@@
 	(wire
 		(pts
+			(xy 171.45 40.64) (xy 146.05 40.64)
+		)
+		(stroke
+			(width 0)
+			(type default)
+		)
+	)
+	(wire
+		(pts
 			(xy 208.28 64.77) (xy 208.28 97.79)
 		)
@@
 	(wire
 		(pts
-			(xy 146.05 71.12) (xy 146.05 43.18)
-		)
-		(stroke
-			(width 0)
-			(type default)
-		)
-	)
-	(wire
-		(pts
 			(xy 129.54 157.48) (xy 123.19 157.48)
 		)
@@
 	(wire
 		(pts
+			(xy 146.05 40.64) (xy 146.05 71.12)
+		)
+		(stroke
+			(width 0)
+			(type default)
+		)
+	)
+	(wire
+		(pts
 			(xy 86.36 95.25) (xy 113.03 95.25)
 		)
@@
 	(wire
 		(pts
-			(xy 146.05 71.12) (xy 143.51 71.12)
-		)
-		(stroke
-			(width 0)
-			(type default)
-		)
-	)
-	(wire
-		(pts
 			(xy 86.36 105.41) (xy 113.03 105.41)
 		)
@@
 	(wire
 		(pts
-			(xy 138.43 71.12) (xy 135.89 71.12)
-		)
-		(stroke
-			(width 0)
-			(type default)
-		)
-	)
-	(wire
-		(pts
 			(xy 215.9 64.77) (xy 215.9 105.41)
 		)
@@
 	(wire
 		(pts
+			(xy 132.08 132.08) (xy 246.38 132.08)
+		)
+		(stroke
+			(width 0)
+			(type default)
+		)
+	)
+	(wire
+		(pts
 			(xy 123.19 149.86) (xy 142.24 149.86)
 		)
@@
 	(wire
 		(pts
-			(xy 143.51 71.12) (xy 143.51 40.64)
+			(xy 143.51 43.18) (xy 143.51 71.12)
 		)
 		(stroke
@@
 		(pts
 			(xy 213.36 64.77) (xy 213.36 102.87)
+		)
+		(stroke
+			(width 0)
+			(type default)
+		)
+	)
+	(wire
+		(pts
+			(xy 171.45 43.18) (xy 143.51 43.18)
 		)
 		(stroke
@@
 			)
 		)
-		(pin "AG_SDI" input
+		(pin "EN_MOT" input
+			(at 171.45 45.72 180)
+			(effects
+				(font
+					(size 1.27 1.27)
+				)
+				(justify left)
+			)
+		)
+		(pin "EN_LIDAR" input
+			(at 171.45 48.26 180)
+			(effects
+				(font
+					(size 1.27 1.27)
+				)
+				(justify left)
+			)
+		)
+		(pin "VIT_MOT_LIDAR" input
+			(at 246.38 64.77 270)
+			(effects
+				(font
+					(size 1.27 1.27)
+				)
+				(justify left)
+			)
+		)
+		(pin "AG_MOSI" input
 			(at 205.74 64.77 270)
 			(effects
@@
 			)
 		)
-		(pin "AG_SDO" output
+		(pin "AG_MISO" output
 			(at 208.28 64.77 270)
 			(effects
