File: Pojet_V-NOM_KiCAD/_autosave-acquisition.kicad_sch (KiCad schematic)
At the start: 7 parts, among them J601 Conn_01x08, J602 Conn_01x03, J603 Conn_01x03, U2 ADXL343

Commit message: DEPLACEMENT
maj Deplacement
Changed lines of the file:
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@@
 	)
 	(hierarchical_label "Vo1"
-		(shape passive)
+		(shape output)
 		(at 205.74 88.9 180)
 		(fields_autoplaced yes)
@@
 	)
 	(hierarchical_label "Vo2"
-		(shape passive)
+		(shape output)
 		(at 205.74 107.95 180)
 		(fields_autoplaced yes)
