File: Pojet_V-NOM_KiCAD/_autosave-acquisition.kicad_sch (KiCad schematic)
At the start: 6 parts, among them J601 Conn_01x08, J602 Conn_01x03, U2 ADXL343

Commit message: modif
modif
Parts:
- removed J601: Conn_01x08, symbol Connector_Generic:Conn_01x08
- removed J602: Conn_01x03, symbol Connector_Generic:Conn_01x03
- added J3: Conn_01x08, symbol Connector_Generic:Conn_01x08
- added J4, J5: Conn_01x03, symbol Connector_Generic:Conn_01x03
Connections:
- net +5V: now also J3.1 (Pin_1), J5.3 (Pin_3)
- net DEV_EN: now also J3.6 (Pin_6)
- net GND: now also J3.4 (Pin_4), J4.2 (Pin_2), J5.2 (Pin_2)
- net M_EN: now also J3.7 (Pin_7)
- net M_SCTR: now also J3.5 (Pin_5)
- net RX_LIDAR: now also J3.3 (Pin_3)
- net TX_LIDAR: now also J3.2 (Pin_2)
- new net Vo_1: J4.1 (Pin_1)
- new net Vo_2: J5.1 (Pin_1)
