File: Pojet_V-NOM_KiCAD/_autosave-alimentation.kicad_sch (KiCad schematic)
At the start: 1 part

Commit message: modif
modif
Parts:
- removed BT401: Battery, symbol Device:Battery
- added BT1: Battery, symbol Device:Battery
Connections:
- net +7.2V: now also BT1.1 (+)
- net GND: now also BT1.2 (-)
Changed lines of the file:
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@@
 	(paper "A4")
 	(junction
-		(at 142.24 93.98)
+		(at 149.86 85.09)
 		(diameter 0)
 		(color 0 0 0 0)
 	)
 	(junction
-		(at 60.96 92.71)
+		(at 68.58 83.82)
 		(diameter 0)
 		(color 0 0 0 0)
@@
 	(wire
 		(pts
-			(xy 54.61 92.71) (xy 60.96 92.71)
-		)
-		(stroke
-			(width 0)
-			(type default)
-		)
-	)
-	(wire
-		(pts
-			(xy 233.68 93.98) (xy 240.03 93.98)
-		)
-		(stroke
-			(width 0)
-			(type default)
-		)
-	)
-	(wire
-		(pts
-			(xy 60.96 88.9) (xy 60.96 92.71)
-		)
-		(stroke
-			(width 0)
-			(type default)
-		)
-	)
-	(wire
-		(pts
-			(xy 135.89 93.98) (xy 142.24 93.98)
-		)
-		(stroke
-			(width 0)
-			(type default)
-		)
-	)
-	(wire
-		(pts
-			(xy 60.96 92.71) (xy 68.58 92.71)
-		)
-		(stroke
-			(width 0)
-			(type default)
-		)
-	)
-	(wire
-		(pts
-			(xy 44.45 92.71) (xy 41.91 92.71)
-		)
-		(stroke
-			(width 0)
-			(type default)
-		)
-	)
-	(wire
-		(pts
-			(xy 142.24 87.63) (xy 142.24 93.98)
-		)
-		(stroke
-			(width 0)
-			(type default)
-		)
-	)
-	(wire
-		(pts
-			(xy 142.24 93.98) (xy 179.07 93.98)
+			(xy 241.3 85.09) (xy 247.65 85.09)
+		)
+		(stroke
+			(width 0)
+			(type default)
+		)
+	)
+	(wire
+		(pts
+			(xy 62.23 83.82) (xy 68.58 83.82)
+		)
+		(stroke
+			(width 0)
+			(type default)
+		)
+	)
+	(wire
+		(pts
+			(xy 52.07 83.82) (xy 49.53 83.82)
+		)
+		(stroke
+			(width 0)
+			(type default)
+		)
+	)
+	(wire
+		(pts
+			(xy 68.58 80.01) (xy 68.58 83.82)
+		)
+		(stroke
+			(width 0)
+			(type default)
+		)
+	)
+	(wire
+		(pts
+			(xy 143.51 85.09) (xy 149.86 85.09)
+		)
+		(stroke
+			(width 0)
+			(type default)
+		)
+	)
+	(wire
+		(pts
+			(xy 149.86 85.09) (xy 186.69 85.09)
+		)
+		(stroke
+			(width 0)
+			(type default)
+		)
+	)
+	(wire
+		(pts
+			(xy 149.86 78.74) (xy 149.86 85.09)
+		)
+		(stroke
+			(width 0)
+			(type default)
+		)
+	)
+	(wire
+		(pts
+			(xy 68.58 83.82) (xy 76.2 83.82)
 		)
 		(stroke
@@
 	(text "Batterie\n"
 		(exclude_from_sim no)
-		(at 48.768 76.962 0)
+		(at 56.388 68.072 0)
 		(effects
 			(font
@@
 	(hierarchical_label "+3.3V"
 		(shape output)
-		(at 240.03 93.98 0)
+		(at 247.65 85.09 0)
 		(fields_autoplaced yes)
 		(effects
@@
 		)
 	)
-	(hierarchical_label "+7.2V"
+	(hierarchical_label "+5V"
 		(shape output)
-		(at 60.96 88.9 90)
+		(at 149.86 78.74 90)
 		(fields_autoplaced yes)
 		(effects
@@
 		)
 	)
-	(hierarchical_label "+5V"
+	(hierarchical_label "+7.2V"
 		(shape output)
-		(at 142.24 87.63 90)
+		(at 68.58 80.01 90)
 		(fields_autoplaced yes)
 		(effects
@@
 	(symbol
 		(lib_id "power:GND")
-		(at 41.91 92.71 270)
+		(at 49.53 83.82 270)
 		(unit 1)
 		(exclude_from_sim no)
@@
 		(dnp no)
 		(fields_autoplaced yes)
-		(property "Reference" "#PWR016"
-			(at 35.56 92.71 0)
+		(property "Reference" "#PWR05"
+			(at 43.18 83.82 0)
 			(effects
 				(font
@@
 		)
 		(property "Value" "GND"
-			(at 38.1 92.7099 90)
+			(at 45.72 83.8199 90)
 			(effects
 				(font
@@
 		)
 		(property "Footprint" ""
-			(at 41.91 92.71 0)
+			(at 49.53 83.82 0)
 			(effects
 				(font
@@
 		)
 		(property "Datasheet" ""
-			(at 41.91 92.71 0)
+			(at 49.53 83.82 0)
 			(effects
 				(font
@@
 		)
 		(property "Description" "Power symbol creates a global label with name \"GND\" , ground"
-			(at 41.91 92.71 0)
+			(at 49.53 83.82 0)
 			(effects
 				(font
@@
 		)
 		(instances
-			(project ""
+			(project "Pojet_V-NOM_KiCAD"
 				(path "/37e0fdad-f3fd-48e0-8377-111662233a91/aef3d9b2-029f-4338-91be-d4af664a9426"
-					(reference "#PWR016")
+					(reference "#PWR05")
 					(unit 1)
 				)
@@
 	(symbol
 		(lib_id "Device:Battery")
-		(at 49.53 92.71 270)
+		(at 57.15 83.82 270)
 		(unit 1)
 		(exclude_from_sim no)
@@
 		(dnp no)
 		(fields_autoplaced yes)
-		(property "Reference" "BT401"
-			(at 50.1015 85.09 90)
+		(property "Reference" "BT1"
+			(at 57.7215 76.2 90)
 			(effects
 				(font
@@
 		)
 		(property "Value" "Battery"
-			(at 50.1015 87.63 90)
+			(at 57.7215 78.74 90)
 			(effects
 				(font
@@
 		)
 		(property "Footprint" ""
-			(at 51.054 92.71 90)
+			(at 58.674 83.82 90)
 			(effects
 				(font
@@
 		)
 		(property "Datasheet" "~"
-			(at 51.054 92.71 90)
+			(at 58.674 83.82 90)
 			(effects
 				(font
@@
 		)
 		(property "Description" "Multiple-cell battery"
-			(at 49.53 92.71 0)
+			(at 57.15 83.82 0)
 			(effects
 				(font
@@
 			(project "Pojet_V-NOM_KiCAD"
 				(path "/37e0fdad-f3fd-48e0-8377-111662233a91/aef3d9b2-029f-4338-91be-d4af664a9426"
-					(reference "BT401")
+					(reference "BT1")
 					(unit 1)
 				)
@@
 	)
 	(sheet
-		(at 68.58 72.39)
+		(at 76.2 63.5)
 		(size 67.31 44.45)
 		(fields_autoplaced yes)
@@
 		)
 		(property "Sheetname" "Régulateur_5V"
-			(at 68.58 71.0434 0)
+			(at 76.2 62.1534 0)
 			(effects
 				(font
@@
 		)
 		(property "Sheetfile" "Régulateur_5V.kicad_sch"
-			(at 68.58 117.4246 0)
+			(at 76.2 108.5346 0)
 			(effects
 				(font
@@
 		)
 		(pin "+5V" output
-			(at 135.89 93.98 0)
+			(at 143.51 85.09 0)
 			(effects
 				(font
@@
 		)
 		(pin "+7.2V" input
-			(at 68.58 92.71 180)
+			(at 76.2 83.82 180)
 			(effects
 				(font
@@
 			(project "Pojet_V-NOM_KiCAD"
 				(path "/37e0fdad-f3fd-48e0-8377-111662233a91/aef3d9b2-029f-4338-91be-d4af664a9426"
-					(page "8")
+					(page "10")
 				)
 			)
@@
 	)
 	(sheet
-		(at 179.07 72.39)
+		(at 186.69 63.5)
 		(size 54.61 46.99)
 		(fields_autoplaced yes)
@@
 		)
 		(property "Sheetname" "Régulateur_3.3V"
-			(at 179.07 71.0434 0)
+			(at 186.69 62.1534 0)
 			(effects
 				(font
@@
 		)
 		(property "Sheetfile" "Régulateur_3.3V.kicad_sch"
-			(at 179.07 119.9646 0)
+			(at 186.69 111.0746 0)
 			(effects
 				(font
@@
 		)
 		(pin "+3.3V" output
-			(at 233.68 93.98 0)
+			(at 241.3 85.09 0)
 			(effects
 				(font
@@
 		)
 		(pin "+5V" input
-			(at 179.07 93.98 180)
+			(at 186.69 85.09 180)
 			(effects
 				(font
@@
 			(project "Pojet_V-NOM_KiCAD"
 				(path "/37e0fdad-f3fd-48e0-8377-111662233a91/aef3d9b2-029f-4338-91be-d4af664a9426"
-					(page "8")
-				)
-			)
+					(page "9")
+				)
+			)
