File: Pojet_V-NOM_KiCAD/_autosave-Régulateur_3.3V.kicad_sch (KiCad schematic)
At the start: 3 parts

Commit message: modif
modif
Parts:
- removed C5, C6: 1uF, symbol Device:C_Small
- added C12, C13: 1uF, symbol Device:C_Small
Connections:
- net +3.3V: now also C13.1
- net +5V: now also C12.1
- net GND: now also C12.2, C13.2
