File: Pojet_V-NOM_KiCAD/controle.kicad_sch (KiCad schematic)
At the start: 10 parts, among them U1 STM32G431CBU6, Y1 Crystal_GND24_Small

Commit message: maj regulateur 5V
Changed lines of the file:
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@@
 	)
 	(hierarchical_label "SPI_MISO"
-		(shape bidirectional)
+		(shape input)
 		(at 163.83 73.66 0)
 		(fields_autoplaced yes)
@@
 	)
 	(hierarchical_label "SPI_SCK"
-		(shape bidirectional)
+		(shape output)
 		(at 163.83 71.12 0)
 		(fields_autoplaced yes)

Commit message: Corrections rapides du schéma global
Connections:
- net AG_USART_RX is gone; now on net VCP_RX: U1.45 (PB7)
- net AG_USART_TX is gone; now on net VCP_TX: U1.44 (PB6)
- net VCP_RX: no longer U1.24 (PB11)
- net VCP_TX: no longer U1.22 (PB10)
- no-connect marks 9 -> 12
Changed lines of the file:
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@@
+	)
+	(no_connect
+		(at 130.81 121.92)
+	)
+	(no_connect
+		(at 130.81 124.46)
 	)
 	(no_connect
 		(at 130.81 134.62)
+	)
+	(no_connect
+		(at 120.65 87.63)
 	)
 	(no_connect
@@
 		)
 	)
-	(hierarchical_label "AG_USART_TX"
-		(shape bidirectional)
-		(at 130.81 111.76 180)
-		(fields_autoplaced yes)
-		(effects
-			(font
-				(size 1.27 1.27)
-			)
-			(justify right)
-		)
-	)
 	(hierarchical_label "SPI1_CSN"
 		(shape output)
@@
 	(hierarchical_label "VCP_TX"
 		(shape bidirectional)
-		(at 130.81 121.92 180)
+		(at 130.81 111.76 180)
 		(fields_autoplaced yes)
 		(effects
@@
 	(hierarchical_label "VCP_RX"
 		(shape bidirectional)
-		(at 130.81 124.46 180)
+		(at 130.81 114.3 180)
 		(fields_autoplaced yes)
 		(effects
@@
 		(fields_autoplaced yes)
 		(effects
-			(font
-				(size 1.27 1.27)
-			)
-			(justify right)
-		)
-	)
-	(hierarchical_label "AG_USART_RX"
-		(shape bidirectional)
-		(at 130.81 114.3 180)
-		(fields_autoplaced yes)
-		(effects

Commit message: Modifications conseillés par l'enseignant
Connections:
- net EN_LIDAR: now reaches U1.39 (PC10)
- net EN_MOT: now reaches U1.40 (PC11)
- no-connect marks 12 -> 9
Changed lines of the file:
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@@
-	)
-	(no_connect
-		(at 120.65 87.63)
-	)
-	(no_connect
-		(at 130.81 81.28)
 	)
 	(no_connect
@@
 	)
 	(no_connect
-		(at 130.81 83.82)
-	)
-	(no_connect
 		(at 130.81 91.44)
 	)
@@
 	(wire
 		(pts
-			(xy 114.3 78.74) (xy 118.11 78.74)
+			(xy 114.3 78.74) (xy 119.38 78.74)
 		)
 		(stroke
@@
 	(wire
 		(pts
-			(xy 118.11 71.12) (xy 130.81 71.12)
-		)
-		(stroke
-			(width 0)
-			(type default)
-		)
-	)
-	(wire
-		(pts
-			(xy 118.11 71.12) (xy 118.11 78.74)
+			(xy 119.38 71.12) (xy 130.81 71.12)
+		)
+		(stroke
+			(width 0)
+			(type default)
+		)
+	)
+	(wire
+		(pts
+			(xy 119.38 71.12) (xy 119.38 78.74)
 		)
 		(stroke
@@
 		)
 	)
+	(hierarchical_label "EN_MOT"
+		(shape input)
+		(at 130.81 83.82 180)
+		(fields_autoplaced yes)
+		(effects
+			(font
+				(size 1.27 1.27)
+			)
+			(justify right)
+		)
+	)
 	(hierarchical_label "TIM3_CH1"
 		(shape output)
@@
 		(fields_autoplaced yes)
 		(effects
+			(font
+				(size 1.27 1.27)
+			)
+			(justify right)
+		)
+	)
+	(hierarchical_label "EN_LIDAR"
+		(shape input)
+		(at 130.81 81.28 180)
+		(fields_autoplaced yes)
+		(effects

Commit message: empreinte
Parts:
- C1: value C_Small -> 10p; footprint (none) -> Capacitor_SMD:C_0402_1005Metric
- C2: value C -> 10p; footprint (none) -> Capacitor_SMD:C_0402_1005Metric
- C5, C6, C7: value 100n -> 100nF; footprint (none) -> Capacitor_SMD:C_0402_1005Metric
- C8: value 4.7u -> 4.7uF; footprint (none) -> Capacitor_SMD:C_0603_1608Metric
- L1: value 47n -> 47nH; footprint (none) -> Inductor_SMD:L_0402_1005Metric
- R1: value R_Small -> 10; footprint (none) -> Resistor_SMD:R_0402_1005Metric
- Y1: value Crystal_GND24_Small -> 16 MHz; footprint (none) -> Crystal:Crystal_SMD_0603-4Pin_6.0x3.5mm
Other:
- note added: "Ajouter des leds pour identifier si la led est alimenté ou pas"
- note removed: "A verifier avec le prof"

Commit message: Correction des erreurs évidentes
Changements avant vérification des erreurs :
- Désallocation du pin BTN_RESET
- Réarrangement de certaines sources pour cohérence avec tous les
schémas éléctriques
Connections:
- net BTN_RESET: no longer names the net of U1.46 (PB8)
- no-connect marks 9 -> 10
Changed lines of the file:
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@@
+	)
+	(no_connect
+		(at 130.81 116.84)
 	)
 	(no_connect
@@
 		)
 	)
-	(hierarchical_label "BTN_RESET"
-		(shape input)
-		(at 130.81 116.84 180)
-		(fields_autoplaced yes)
-		(effects
-			(font
-				(size 1.27 1.27)
-			)
-			(justify right)
-		)
-	)

Commit message: point de test et début de placement
Parts:
- added TP201, TP202, TP203, TP204, TP205, TP206, TP207, TP208, TP209, TP210, TP211: TestPoint, TestPoint:TestPoint_Pad_D1.0mm, symbol Connector:TestPoint
Connections:
- net +3.3V: now also TP201.1, TP202.1
- net AG_INT1: now also TP209.1
- net AG_INT2: now also TP210.1
- net EN_LIDAR: now also TP203.1
- net EN_MOT: now also TP204.1
- net LIDAR_RX: now also TP208.1
- net LIDAR_TX: now also TP205.1
- net NRST: now also TP211.1
- net VCP_RX: now also TP207.1
- net VCP_TX: now also TP206.1
Other:
- note removed: "Ajouter des leds pour identifier si la led est alimenté ou pas"

Commit message: maj emplacement
Parts:
- removed TP202, TP203, TP204, TP205, TP206, TP207, TP208, TP209, TP210: TestPoint, TestPoint:TestPoint_Pad_D1.0mm, symbol Connector:TestPoint

Commit message: placement maj
Parts:
- removed TP201, TP211: TestPoint, TestPoint:TestPoint_Pad_D1.0mm, symbol Connector:TestPoint
- added C201: 10nF, Capacitor_SMD:C_0402_1005Metric, symbol Device:C_Small
- added C202: 100nF, Capacitor_SMD:C_0402_1005Metric, symbol Device:C_Small
- L1: value 47nH -> 39nH
- Y1: footprint Crystal:Crystal_SMD_0603-4Pin_6.0x3.5mm -> Crystal:Crystal_SMD_EuroQuartz_MT-4Pin_3.2x2.5mm
Connections:
- net +3.3V: now also C201.1, C202.1
- net GND: now also C201.2, C202.2
