File: Pojet_V-NOM_KiCAD/controle.kicad_sch (KiCad schematic)
At the start: 12 parts, among them U1 STM32G431CBU6, Y1 16 MHz

Commit message: maj final aprés correction du prof + logo ensea
Parts:
- added C203: 100nF, Capacitor_SMD:C_0402_1005Metric, symbol Device:C_Small
Connections:
- net +3.3V: no longer C201.1
- net GND: now also C203.2
- net NRST: now also C203.1
- net at L1.2, U1.21 (VDDA): now also C201.1
Other:
- moved on the sheet: C201, C202, C5, C6, C7, C8, L1

Commit message: final
Connections:
- net TOF1: now also U1.10 (PA2); no longer U1.3 (PC14)
Changed lines of the file:
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@@
+	)
+	(no_connect
+		(at 130.81 101.6)
+	)
+	(no_connect
+		(at 130.81 78.74)
+	)
+	(no_connect
+		(at 130.81 121.92)
+	)
+	(no_connect
+		(at 130.81 124.46)
+	)
+	(no_connect
+		(at 130.81 134.62)
+	)
+	(no_connect
+		(at 130.81 116.84)
 	)
 	(no_connect
@@
 	)
 	(no_connect
-		(at 130.81 101.6)
-	)
-	(no_connect
-		(at 130.81 78.74)
-	)
-	(no_connect
-		(at 130.81 121.92)
-	)
-	(no_connect
-		(at 130.81 124.46)
-	)
-	(no_connect
-		(at 130.81 134.62)
-	)
-	(no_connect
-		(at 130.81 116.84)
-	)
-	(no_connect
-		(at 163.83 63.5)
+		(at 130.81 88.9)
 	)
 	(no_connect
@@
 		)
 	)
+	(hierarchical_label "TOF1"
+		(shape input)
+		(at 163.83 63.5 0)
+		(fields_autoplaced yes)
+		(effects
+			(font
+				(size 1.27 1.27)
+			)
+			(justify left)
+		)
+	)
 	(hierarchical_label "LIDAR_TX"
 		(shape bidirectional)
@@
 		(fields_autoplaced yes)
 		(effects
-			(font
-				(size 1.27 1.27)
-			)
-			(justify right)
-		)
-	)
-	(hierarchical_label "TOF1"
-		(shape input)
-		(at 130.81 88.9 180)
-		(fields_autoplaced yes)
-		(effects
