File: Pojet_V-NOM_KiCAD/acquisition.kicad_sch (KiCad schematic)
At the start: 4 parts, among them U2 ADXL343

Commit message: lidar
rajout du lidar
Parts:
- added J601: Conn_01x08, symbol Connector_Generic:Conn_01x08
Connections:
- net GND: now also J601.4 (Pin_4)
- new net +5V: J601.1 (Pin_1)
- new net PA10: J601.2 (Pin_2)
- new net PA4: J601.5 (Pin_5)
- new net PA5: J601.6 (Pin_6)
- new net PA6: J601.7 (Pin_7)
- new net PA9: J601.3 (Pin_3)
- no-connect marks 2 -> 3
Other:
- note added: "LIDAR"

Commit message: rajout capteur
capteur de bordure
Parts:
- added J602: Conn_01x03, symbol Connector_Generic:Conn_01x03
Connections:
- net +5V: now also J602.3 (Pin_3)
- net GND: now also J602.2 (Pin_2)
- new net Vo: J602.1 (Pin_1)
Other:
- note added: "Capteur de bordure"

Commit message: MAJ Valerian
MAJ Valerian
Connections:
- net PA10 renamed TX_LIDAR
- net PA2 renamed INT1_ACCEL
- net PA3 renamed INT2_ACCEL
- net PA4 renamed M_SCTR
- net PA5 renamed DEV_EN
- net PA6 renamed M_EN
- net PA9 renamed RX_LIDAR
Other:
- moved on the sheet: J601, J602
Changed lines of the file:
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@@
 	)
 	(no_connect
-		(at 158.75 55.88)
+		(at 62.23 156.21)
 	)
 	(wire
@@
 	(wire
 		(pts
-			(xy 228.6 63.5) (xy 240.03 63.5)
+			(xy 205.74 91.44) (xy 217.17 91.44)
 		)
 		(stroke
@@
 		)
 	)
+	(polyline
+		(pts
+			(xy 160.02 12.7) (xy 160.02 198.12)
+		)
+		(stroke
+			(width 0)
+			(type default)
+		)
+	)
 	(wire
 		(pts
@@
 	(wire
 		(pts
-			(xy 176.53 48.26) (xy 176.53 55.88)
-		)
-		(stroke
-			(width 0)
-			(type default)
-		)
-	)
-	(wire
-		(pts
-			(xy 228.6 66.04) (xy 240.03 66.04)
-		)
-		(stroke
-			(width 0)
-			(type default)
-		)
-	)
-	(wire
-		(pts
-			(xy 228.6 60.96) (xy 240.03 60.96)
+			(xy 80.01 148.59) (xy 80.01 156.21)
+		)
+		(stroke
+			(width 0)
+			(type default)
+		)
+	)
+	(wire
+		(pts
+			(xy 205.74 93.98) (xy 217.17 93.98)
+		)
+		(stroke
+			(width 0)
+			(type default)
+		)
+	)
+	(polyline
+		(pts
+			(xy 10.16 110.49) (xy 160.02 110.49)
+		)
+		(stroke
+			(width 0)
+			(type default)
+		)
+	)
+	(wire
+		(pts
+			(xy 205.74 88.9) (xy 217.17 88.9)
 		)
 		(stroke
@@
 	(wire
 		(pts
-			(xy 168.91 48.26) (xy 168.91 55.88)
+			(xy 72.39 148.59) (xy 72.39 156.21)
 		)
 		(stroke
@@
 	(text "LIDAR"
 		(exclude_from_sim no)
-		(at 148.59 33.528 0)
+		(at 52.07 133.858 0)
 		(effects
 			(font
@@
 	(text "Capteur de bordure\n"
 		(exclude_from_sim no)
-		(at 235.204 34.544 0)
+		(at 212.344 62.484 0)
 		(effects
 			(font
@@
 		)
 	)
-	(hierarchical_label "PA2"
+	(hierarchical_label "INT1_ACCEL"
 		(shape passive)
 		(at 81.28 72.39 0)
@@
 		)
 	)
-	(hierarchical_label "PA9"
+	(hierarchical_label "RX_LIDAR"
 		(shape passive)
-		(at 171.45 55.88 90)
+		(at 74.93 156.21 90)
 		(fields_autoplaced yes)
 		(effects
@@
 		)
 	)
-	(hierarchical_label "PA5"
+	(hierarchical_label "DEV_EN"
 		(shape passive)
-		(at 163.83 55.88 90)
+		(at 67.31 156.21 90)
 		(fields_autoplaced yes)
 		(effects
@@
 	(hierarchical_label "Vo"
 		(shape passive)
-		(at 228.6 60.96 180)
+		(at 205.74 88.9 180)
 		(fields_autoplaced yes)
 		(effects
@@
 		)
 	)
-	(hierarchical_label "PA3"
+	(hierarchical_label "INT2_ACCEL"
 		(shape passive)
 		(at 81.28 74.93 0)
@@
 		)
 	)
-	(hierarchical_label "PA6"
+	(hierarchical_label "M_EN"
 		(shape passive)
-		(at 161.29 55.88 90)
+		(at 64.77 156.21 90)
 		(fields_autoplaced yes)
 		(effects
@@
 		)
 	)
-	(hierarchical_label "PA4"
+	(hierarchical_label "M_SCTR"
 		(shape passive)
-		(at 166.37 55.88 90)
+		(at 69.85 156.21 90)
 		(fields_autoplaced yes)
 		(effects
@@
 		)
 	)
-	(hierarchical_label "PA10"
+	(hierarchical_label "TX_LIDAR"
 		(shape passive)
-		(at 173.99 55.88 90)
+		(at 77.47 156.21 90)
 		(fields_autoplaced yes)
 		(effects
@@
 	(symbol
 		(lib_id "power:+5V")
-		(at 176.53 48.26 0)
+		(at 80.01 148.59 0)
 		(unit 1)
 		(exclude_from_sim no)
@@
 		(fields_autoplaced yes)
 		(property "Reference" "#PWR0602"
-			(at 176.53 52.07 0)
+			(at 80.01 152.4 0)
 			(effects
 				(font
@@
 		)
 		(property "Value" "+5V"
-			(at 176.53 43.18 0)
+			(at 80.01 143.51 0)
 			(effects
 				(font
@@
 		)
 		(property "Footprint" ""
-			(at 176.53 48.26 0)
+			(at 80.01 148.59 0)
 			(effects
 				(font
@@
 		)
 		(property "Datasheet" ""
-			(at 176.53 48.26 0)
+			(at 80.01 148.59 0)
 			(effects
 				(font
@@
 		)
 		(property "Description" "Power symbol creates a global label with name \"+5V\""
-			(at 176.53 48.26 0)
+			(at 80.01 148.59 0)
 			(effects
 				(font
@@
 	(symbol
 		(lib_id "power:+5V")
-		(at 228.6 66.04 90)
+		(at 205.74 93.98 90)
 		(unit 1)
 		(exclude_from_sim no)
@@
 		(fields_autoplaced yes)
 		(property "Reference" "#PWR0604"
-			(at 232.41 66.04 0)
+			(at 209.55 93.98 0)
 			(effects
 				(font
@@
 		)
 		(property "Value" "+5V"
-			(at 224.79 66.0399 90)
+			(at 201.93 93.9799 90)
 			(effects
 				(font
@@
 		)
 		(property "Footprint" ""
-			(at 228.6 66.04 0)
+			(at 205.74 93.98 0)
 			(effects
 				(font
@@
 		)
 		(property "Datasheet" ""
-			(at 228.6 66.04 0)
+			(at 205.74 93.98 0)
 			(effects
 				(font
@@
 		)
 		(property "Description" "Power symbol creates a global label with name \"+5V\""
-			(at 228.6 66.04 0)
+			(at 205.74 93.98 0)
 			(effects
 				(font
@@
 	(symbol
 		(lib_id "Connector_Generic:Conn_01x08")
-		(at 168.91 60.96 270)
+		(at 72.39 161.29 270)
 		(unit 1)
 		(exclude_from_sim no)
@@
 		(fields_autoplaced yes)
 		(property "Reference" "J601"
-			(at 167.64 64.77 90)
+			(at 71.12 165.1 90)
 			(effects
 				(font
@@
 		)
 		(property "Value" "Conn_01x08"
-			(at 167.64 67.31 90)
+			(at 71.12 167.64 90)
 			(effects
 				(font
@@
 		)
 		(property "Footprint" ""
-			(at 168.91 60.96 0)
+			(at 72.39 161.29 0)
 			(effects
 				(font
@@
 		)
 		(property "Datasheet" "~"
-			(at 168.91 60.96 0)
+			(at 72.39 161.29 0)
 			(effects
 				(font
@@
 		)
 		(property "Description" "Generic connector, single row, 01x08, script generated (kicad-library-utils/schlib/autogen/connector/)"
-			(at 168.91 60.96 0)
+			(at 72.39 161.29 0)
 			(effects
 				(font
@@
 	(symbol
 		(lib_id "power:GND")
-		(at 228.6 63.5 270)
+		(at 205.74 91.44 270)
 		(unit 1)
 		(exclude_from_sim no)
@@
 		(fields_autoplaced yes)
 		(property "Reference" "#PWR0603"
-			(at 222.25 63.5 0)
+			(at 199.39 91.44 0)
 			(effects
 				(font
@@
 		)
 		(property "Value" "GND"
-			(at 224.79 63.4999 90)
+			(at 201.93 91.4399 90)
 			(effects
 				(font
@@
 		)
 		(property "Footprint" ""
-			(at 228.6 63.5 0)
+			(at 205.74 91.44 0)
 			(effects
 				(font
@@
 		)
 		(property "Datasheet" ""
-			(at 228.6 63.5 0)
+			(at 205.74 91.44 0)
 			(effects
 				(font
@@
 		)
 		(property "Description" "Power symbol creates a global label with name \"GND\" , ground"
-			(at 228.6 63.5 0)
+			(at 205.74 91.44 0)
 			(effects
 				(font
@@
 	(symbol
 		(lib_id "power:GND")
-		(at 168.91 48.26 180)
+		(at 72.39 148.59 180)
 		(unit 1)
 		(exclude_from_sim no)
@@
 		(fields_autoplaced yes)
 		(property "Reference" "#PWR0601"
-			(at 168.91 41.91 0)
+			(at 72.39 142.24 0)
 			(effects
 				(font
@@
 		)
 		(property "Value" "GND"
-			(at 168.91 43.18 0)
+			(at 72.39 143.51 0)
 			(effects
 				(font
@@
 		)
 		(property "Footprint" ""
-			(at 168.91 48.26 0)
+			(at 72.39 148.59 0)
 			(effects
 				(font
@@
 		)
 		(property "Datasheet" ""
-			(at 168.91 48.26 0)
+			(at 72.39 148.59 0)
 			(effects
 				(font
@@
 		)
 		(property "Description" "Power symbol creates a global label with name \"GND\" , ground"
-			(at 168.91 48.26 0)
+			(at 72.39 148.59 0)
 			(effects
 				(font
@@
 	(symbol
 		(lib_id "Connector_Generic:Conn_01x03")
-		(at 245.11 63.5 0)
+		(at 222.25 91.44 0)
 		(unit 1)
 		(exclude_from_sim no)
@@
 		(fields_autoplaced yes)
 		(property "Reference" "J602"
-			(at 247.65 62.2299 0)
+			(at 224.79 90.1699 0)
 			(effects
 				(font
@@
 		)
 		(property "Value" "Conn_01x03"
-			(at 247.65 64.7699 0)
+			(at 224.79 92.7099 0)
 			(effects
 				(font
@@
 		)
 		(property "Footprint" ""
-			(at 245.11 63.5 0)
+			(at 222.25 91.44 0)
 			(effects
 				(font
@@
 		)
 		(property "Datasheet" "~"
-			(at 245.11 63.5 0)
+			(at 222.25 91.44 0)
 			(effects
 				(font
@@
 		)
 		(property "Description" "Generic connector, single row, 01x03, script generated (kicad-library-utils/schlib/autogen/connector/)"
-			(at 245.11 63.5 0)
-			(effects
-				(font
+			(at 222.25 91.44 0)
+			(effects
+				(font

Commit message: modif
Parts:
- removed J601: Conn_01x08, symbol Connector_Generic:Conn_01x08
- removed J602: Conn_01x03, symbol Connector_Generic:Conn_01x03
- added J3: Conn_01x08, symbol Connector_Generic:Conn_01x08
- added J4, J5: Conn_01x03, symbol Connector_Generic:Conn_01x03
Connections:
- net +5V: now also J3.1 (Pin_1), J4.3 (Pin_3), J5.3 (Pin_3)
- net DEV_EN: now also J3.6 (Pin_6)
- net GND: now also J3.4 (Pin_4), J4.2 (Pin_2), J5.2 (Pin_2)
- net M_EN: now also J3.7 (Pin_7)
- net M_SCTR: now also J3.5 (Pin_5)
- net RX_LIDAR: now also J3.3 (Pin_3)
- net TX_LIDAR: now also J3.2 (Pin_2)
- new net Vo_1: J4.1 (Pin_1)
- new net Vo_2: J5.1 (Pin_1)

Commit message: Mise à jour du schéma principal
Connections:
- net CS renamed AG_CSN
- net INT1_ACCEL renamed AG_INT1
- net INT2_ACCEL renamed AG_INT2
- net SDA renamed AG_SDA
- net Vo_1 renamed TOF1
- net Vo_2 renamed TOF2
- net sclk renamed AG_SCLK
Changed lines of the file:
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@@
 		)
 	)
-	(hierarchical_label "SDA"
+	(hierarchical_label "AG_SDA"
 		(shape input)
 		(at 58.42 63.5 180)
@@
 		)
 	)
-	(hierarchical_label "Vo_2"
+	(hierarchical_label "TOF2"
 		(shape output)
 		(at 209.55 97.79 180)
@@
 		)
 	)
-	(hierarchical_label "INT1_ACCEL"
+	(hierarchical_label "AG_INT1"
 		(shape output)
 		(at 83.82 63.5 0)
@@
 		)
 	)
-	(hierarchical_label "sclk"
+	(hierarchical_label "AG_SCLK"
 		(shape input)
 		(at 58.42 66.04 180)
@@
 		)
 	)
-	(hierarchical_label "Vo_1"
+	(hierarchical_label "TOF1"
 		(shape output)
 		(at 208.28 80.01 180)
@@
 		)
 	)
-	(hierarchical_label "CS"
+	(hierarchical_label "AG_CSN"
 		(shape input)
 		(at 58.42 68.58 180)
@@
 		)
 	)
-	(hierarchical_label "INT2_ACCEL"
+	(hierarchical_label "AG_INT2"
 		(shape output)
 		(at 83.82 66.04 0)

Commit message: Maj
Maj lidar et regualteur
Connections:
- net DEV_EN is gone; now on net +3.3V: J3.6 (Pin_6)
- net M_EN is gone; now on net +3.3V: J3.7 (Pin_7)
- net M_SCTR is gone; now on net GND: J3.5 (Pin_5)
Changed lines of the file:
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@@
+		(color 0 0 0 0)
+	)
+	(junction
+		(at 74.93 143.51)
+		(diameter 0)
 		(color 0 0 0 0)
 	)
@@
 	(wire
 		(pts
-			(xy 74.93 139.7) (xy 74.93 147.32)
+			(xy 72.39 143.51) (xy 74.93 143.51)
+		)
+		(stroke
+			(width 0)
+			(type default)
+		)
+	)
+	(wire
+		(pts
+			(xy 74.93 139.7) (xy 74.93 143.51)
 		)
 		(stroke
@@
 	(wire
 		(pts
+			(xy 82.55 143.51) (xy 82.55 147.32)
+		)
+		(stroke
+			(width 0)
+			(type default)
+		)
+	)
+	(wire
+		(pts
 			(xy 52.07 60.96) (xy 58.42 60.96)
 		)
@@
 	(wire
 		(pts
+			(xy 74.93 143.51) (xy 74.93 147.32)
+		)
+		(stroke
+			(width 0)
+			(type default)
+		)
+	)
+	(wire
+		(pts
+			(xy 72.39 147.32) (xy 72.39 143.51)
+		)
+		(stroke
+			(width 0)
+			(type default)
+		)
+	)
+	(wire
+		(pts
 			(xy 208.28 82.55) (xy 219.71 82.55)
 		)
@@
 		(pts
 			(xy 71.12 45.72) (xy 69.85 45.72)
-		)
-		(stroke
-			(width 0)
-			(type default)
-		)
-	)
-	(wire
-		(pts
-			(xy 82.55 139.7) (xy 82.55 147.32)
 		)
 		(stroke
@@
 		)
 	)
+	(hierarchical_label "+3.3V"
+		(shape input)
+		(at 67.31 147.32 90)
+		(fields_autoplaced yes)
+		(effects
+			(font
+				(size 1.27 1.27)
+			)
+			(justify left)
+		)
+	)
 	(hierarchical_label "TOF2"
 		(shape output)
@@
 		)
 	)
-	(hierarchical_label "DEV_EN"
-		(shape passive)
-		(at 69.85 147.32 90)
-		(fields_autoplaced yes)
-		(effects
-			(font
-				(size 1.27 1.27)
-			)
-			(justify left)
-		)
-	)
 	(hierarchical_label "AG_INT1"
 		(shape output)
@@
 		)
 	)
-	(hierarchical_label "M_SCTR"
-		(shape passive)
-		(at 72.39 147.32 90)
-		(fields_autoplaced yes)
-		(effects
-			(font
-				(size 1.27 1.27)
-			)
-			(justify left)
-		)
-	)
-	(hierarchical_label "M_EN"
-		(shape passive)
-		(at 67.31 147.32 90)
-		(fields_autoplaced yes)
-		(effects
-			(font
-				(size 1.27 1.27)
-			)
-			(justify left)
-		)
-	)
 	(hierarchical_label "AG_SCLK"
 		(shape input)
@@
 	)
 	(hierarchical_label "TX_LIDAR"
-		(shape passive)
+		(shape output)
 		(at 80.01 147.32 90)
 		(fields_autoplaced yes)
@@
 	(hierarchical_label "+3.3V"
 		(shape input)
+		(at 69.85 147.32 90)
+		(fields_autoplaced yes)
+		(effects
+			(font
+				(size 1.27 1.27)
+			)
+			(justify left)
+		)
+	)
+	(hierarchical_label "+5V"
+		(shape input)
+		(at 82.55 143.51 90)
+		(fields_autoplaced yes)
+		(effects
+			(font
+				(size 1.27 1.27)
+			)
+			(justify left)
+		)
+	)
+	(hierarchical_label "+3.3V"
+		(shape input)
 		(at 49.53 34.29 180)
 		(fields_autoplaced yes)
@@
 	)
 	(hierarchical_label "RX_LIDAR"
-		(shape passive)
+		(shape input)
 		(at 77.47 147.32 90)
 		(fields_autoplaced yes)
@@
 					(unit 1)
 				)
-			)
-		)
-	)
-	(symbol
-		(lib_id "power:+5V")
-		(at 82.55 139.7 0)
-		(unit 1)
-		(exclude_from_sim no)
-		(in_bom yes)
-		(on_board yes)
-		(dnp no)
-		(fields_autoplaced yes)
-		(property "Reference" "#PWR017"
-			(at 82.55 143.51 0)
-			(effects
-				(font
-					(size 1.27 1.27)
-				)
-				(hide yes)
-			)
-		)
-		(property "Value" "+5V"
-			(at 82.55 134.62 0)
-			(effects
-				(font
-					(size 1.27 1.27)
-				)
-			)
-		)
-		(property "Footprint" ""
-			(at 82.55 139.7 0)
-			(effects
-				(font
-					(size 1.27 1.27)
-				)
-				(hide yes)
-			)
-		)
-		(property "Datasheet" ""
-			(at 82.55 139.7 0)
-			(effects
-				(font
-					(size 1.27 1.27)
-				)
-				(hide yes)
-			)
-		)
-		(property "Description" "Power symbol creates a global label with name \"+5V\""
-			(at 82.55 139.7 0)
-			(effects
-				(font
-					(size 1.27 1.27)
-				)
-				(hide yes)
-			)
-		)
-		(pin "1"
-		)
-		(instances
-			(project "Pojet_V-NOM_KiCAD"
-				(path "/37e0fdad-f3fd-48e0-8377-111662233a91/8a0e1cc3-b8cc-4980-b1ce-7a1b28674574"
-					(reference "#PWR017")
-					(unit 1)
-				)

Commit message: Retouches lisibilité Alim / capteurs
Connections:
- net +3.3V: now also C3.1, C4.1; no longer C3.2, C4.2
- net GND: now also C3.2, C4.2; no longer C3.1, C4.1
Other:
- moved on the sheet: C3, C4, J3, J4, J5, R4, U2

Commit message: maj
Other:
- moved on the sheet: J4, J5
