File: Pojet_V-NOM_KiCAD/acquisition.kicad_sch (KiCad schematic)
At the start: 7 parts, among them J3 Conn_01x08, J4 Conn_01x03, J5 Conn_01x03, U2 ADXL343

Commit message: Correction schéma accéléromètre
Parts:
- removed R4: 10 k, symbol Device:R_Small
Connections:
- net AG_SDO: now reaches U2.12 (SDO/ADDR)
- net AG_SDA renamed AG_SDI
Changed lines of the file:
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@@
 	(wire
 		(pts
-			(xy 55.88 66.04) (xy 55.88 62.23)
+			(xy 88.9 44.45) (xy 72.39 44.45)
 		)
 		(stroke
@@
 	(wire
 		(pts
-			(xy 88.9 44.45) (xy 72.39 44.45)
+			(xy 201.93 102.87) (xy 201.93 91.44)
 		)
 		(stroke
@@
 	(wire
 		(pts
-			(xy 201.93 102.87) (xy 201.93 91.44)
+			(xy 93.98 44.45) (xy 88.9 44.45)
 		)
 		(stroke
@@
 	(wire
 		(pts
-			(xy 93.98 44.45) (xy 88.9 44.45)
+			(xy 227.33 99.06) (xy 227.33 91.44)
 		)
 		(stroke
@@
 	(wire
 		(pts
-			(xy 227.33 99.06) (xy 227.33 91.44)
+			(xy 69.85 50.8) (xy 69.85 52.07)
 		)
 		(stroke
@@
 	(wire
 		(pts
-			(xy 69.85 50.8) (xy 69.85 52.07)
+			(xy 77.47 147.32) (xy 77.47 146.05)
 		)
 		(stroke
@@
 	(wire
 		(pts
-			(xy 77.47 147.32) (xy 77.47 146.05)
+			(xy 72.39 149.86) (xy 72.39 146.05)
 		)
 		(stroke
@@
 	(wire
 		(pts
-			(xy 55.88 62.23) (xy 76.2 62.23)
+			(xy 74.93 146.05) (xy 74.93 149.86)
 		)
 		(stroke
@@
 	(wire
 		(pts
-			(xy 72.39 149.86) (xy 72.39 146.05)
+			(xy 66.04 50.8) (xy 69.85 50.8)
 		)
 		(stroke
@@
 	(wire
 		(pts
-			(xy 74.93 146.05) (xy 74.93 149.86)
+			(xy 66.04 44.45) (xy 72.39 44.45)
+		)
+		(stroke
+			(width 0)
+			(type default)
+		)
+	)
+	(polyline
+		(pts
+			(xy 12.7 101.6) (xy 162.56 101.6)
 		)
 		(stroke
@@
 	(wire
 		(pts
-			(xy 66.04 50.8) (xy 69.85 50.8)
+			(xy 229.87 99.06) (xy 229.87 91.44)
 		)
 		(stroke
@@
 	(wire
 		(pts
-			(xy 66.04 44.45) (xy 72.39 44.45)
-		)
-		(stroke
-			(width 0)
-			(type default)
-		)
-	)
-	(polyline
-		(pts
-			(xy 12.7 101.6) (xy 162.56 101.6)
-		)
-		(stroke
-			(width 0)
-			(type default)
-		)
-	)
-	(wire
-		(pts
-			(xy 229.87 99.06) (xy 229.87 91.44)
-		)
-		(stroke
-			(width 0)
-			(type default)
-		)
-	)
-	(wire
-		(pts
 			(xy 72.39 45.72) (xy 72.39 44.45)
 		)
@@
 		)
 	)
-	(hierarchical_label "AG_SDA"
+	(hierarchical_label "AG_SDI"
 		(shape input)
 		(at 76.2 64.77 180)
@@
 		)
 	)
+	(hierarchical_label "AG_SDO"
+		(shape input)
+		(at 76.2 62.23 180)
+		(fields_autoplaced yes)
+		(effects
+			(font
+				(size 1.27 1.27)
+			)
+			(justify right)
+		)
+	)
 	(hierarchical_label "AG_INT1"
 		(shape output)
@@
 	)
 	(symbol
-		(lib_id "Device:R_Small")
-		(at 55.88 68.58 180)
-		(unit 1)
-		(exclude_from_sim no)
-		(in_bom yes)
-		(on_board yes)
-		(dnp no)
-		(property "Reference" "R4"
-			(at 61.722 70.866 0)
-			(effects
-				(font
-					(size 1.27 1.27)
-				)
-				(justify left)
-			)
-		)
-		(property "Value" "10 k"
-			(at 62.992 68.326 0)
-			(effects
-				(font
-					(size 1.27 1.27)
-				)
-				(justify left)
-			)
-		)
-		(property "Footprint" ""
-			(at 55.88 68.58 0)
-			(effects
-				(font
-					(size 1.27 1.27)
-				)
-				(hide yes)
-			)
-		)
-		(property "Datasheet" "~"
-			(at 55.88 68.58 0)
-			(effects
-				(font
-					(size 1.27 1.27)
-				)
-				(hide yes)
-			)
-		)
-		(property "Description" "Resistor, small symbol"
-			(at 55.88 68.58 0)
-			(effects
-				(font
-					(size 1.27 1.27)
-				)
-				(hide yes)
-			)
-		)
-		(pin "1"
-		)
-		(pin "2"
-		)
-		(instances
-			(project "Pojet_V-NOM_KiCAD"
-				(path "/37e0fdad-f3fd-48e0-8377-111662233a91/8a0e1cc3-b8cc-4980-b1ce-7a1b28674574"
-					(reference "R4")
-					(unit 1)
-				)
-			)
-		)
-	)
-	(symbol
 		(lib_id "Device:C_Small")
 		(at 72.39 48.26 0)
@@
 					(unit 1)
 				)
-			)
-		)
-	)
-	(symbol
-		(lib_id "power:GND")
-		(at 55.88 71.12 0)
-		(unit 1)
-		(exclude_from_sim no)
-		(in_bom yes)
-		(on_board yes)
-		(dnp no)
-		(fields_autoplaced yes)
-		(property "Reference" "#PWR010"
-			(at 55.88 77.47 0)
-			(effects
-				(font
-					(size 1.27 1.27)
-				)
-				(hide yes)
-			)
-		)
-		(property "Value" "GND"
-			(at 55.88 76.2 0)
-			(effects
-				(font
-					(size 1.27 1.27)
-				)
-			)
-		)
-		(property "Footprint" ""
-			(at 55.88 71.12 0)
-			(effects
-				(font
-					(size 1.27 1.27)
-				)
-				(hide yes)
-			)
-		)
-		(property "Datasheet" ""
-			(at 55.88 71.12 0)
-			(effects
-				(font
-					(size 1.27 1.27)
-				)
-				(hide yes)
-			)
-		)
-		(property "Description" "Power symbol creates a global label with name \"GND\" , ground"
-			(at 55.88 71.12 0)
-			(effects
-				(font
-					(size 1.27 1.27)
-				)
-				(hide yes)
-			)
-		)
-		(pin "1"
-		)
-		(instances
-			(project "Pojet_V-NOM_KiCAD"
-				(path "/37e0fdad-f3fd-48e0-8377-111662233a91/8a0e1cc3-b8cc-4980-b1ce-7a1b28674574"
-					(reference "#PWR010")
-					(unit 1)
-				)

Commit message: maj regulateur 5V
Changed lines of the file:
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@@
 	)
 	(hierarchical_label "AG_SDO"
-		(shape input)
+		(shape output)
 		(at 76.2 62.23 180)
 		(fields_autoplaced yes)

Commit message: Modifications conseillés par l'enseignant
Connections:
- net +3.3V: no longer J3.6 (Pin_6), J3.7 (Pin_7)
- net GND: no longer J3.5 (Pin_5)
- net AG_SDI renamed AG_MOSI
- net AG_SDO renamed AG_MISO
- new net EN_LIDAR: J3.6 (Pin_6)
- new net EN_MOT: J3.5 (Pin_5)
- new net VIT_MOT_LIDAR: J3.7 (Pin_7)
Changed lines of the file:
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@@
-	)
-	(junction
-		(at 72.39 149.86)
-		(diameter 0)
-		(color 0 0 0 0)
 	)
 	(junction
@@
 		(color 0 0 0 0)
 	)
-	(junction
-		(at 77.47 147.32)
-		(diameter 0)
-		(color 0 0 0 0)
-	)
 	(no_connect
 		(at 83.82 52.07)
@@
 	(wire
 		(pts
-			(xy 80.01 146.05) (xy 80.01 147.32)
-		)
-		(stroke
-			(width 0)
-			(type default)
-		)
-	)
-	(wire
-		(pts
-			(xy 74.93 149.86) (xy 72.39 149.86)
-		)
-		(stroke
-			(width 0)
-			(type default)
-		)
-	)
-	(wire
-		(pts
-			(xy 77.47 154.94) (xy 77.47 147.32)
-		)
-		(stroke
-			(width 0)
-			(type default)
-		)
-	)
-	(wire
-		(pts
 			(xy 224.79 100.33) (xy 224.79 91.44)
 		)
@@
 	(wire
 		(pts
-			(xy 80.01 147.32) (xy 77.47 147.32)
-		)
-		(stroke
-			(width 0)
-			(type default)
-		)
-	)
-	(wire
-		(pts
 			(xy 88.9 77.47) (xy 88.9 81.28)
 		)
@@
 	(wire
 		(pts
-			(xy 72.39 154.94) (xy 72.39 149.86)
+			(xy 72.39 146.05) (xy 72.39 154.94)
 		)
 		(stroke
@@
 		(pts
 			(xy 69.85 50.8) (xy 69.85 52.07)
-		)
-		(stroke
-			(width 0)
-			(type default)
-		)
-	)
-	(wire
-		(pts
-			(xy 77.47 147.32) (xy 77.47 146.05)
-		)
-		(stroke
-			(width 0)
-			(type default)
-		)
-	)
-	(wire
-		(pts
-			(xy 72.39 149.86) (xy 72.39 146.05)
-		)
-		(stroke
-			(width 0)
-			(type default)
-		)
-	)
-	(wire
-		(pts
-			(xy 74.93 146.05) (xy 74.93 149.86)
 		)
 		(stroke
@@
 		)
 	)
-	(hierarchical_label "AG_SDI"
+	(hierarchical_label "AG_MOSI"
 		(shape input)
 		(at 76.2 64.77 180)
@@
 		)
 	)
-	(hierarchical_label "AG_SDO"
+	(hierarchical_label "AG_MISO"
 		(shape output)
 		(at 76.2 62.23 180)
@@
 		)
 	)
+	(hierarchical_label "EN_MOT"
+		(shape input)
+		(at 74.93 146.05 270)
+		(fields_autoplaced yes)
+		(effects
+			(font
+				(size 1.27 1.27)
+			)
+			(justify right)
+		)
+	)
 	(hierarchical_label "AG_INT1"
 		(shape output)
@@
 		)
 	)
+	(hierarchical_label "EN_LIDAR"
+		(shape input)
+		(at 77.47 146.05 270)
+		(fields_autoplaced yes)
+		(effects
+			(font
+				(size 1.27 1.27)
+			)
+			(justify right)
+		)
+	)
 	(hierarchical_label "AG_SCLK"
 		(shape input)
@@
 		(shape output)
 		(at 201.93 102.87 270)
+		(fields_autoplaced yes)
+		(effects
+			(font
+				(size 1.27 1.27)
+			)
+			(justify right)
+		)
+	)
+	(hierarchical_label "VIT_MOT_LIDAR"
+		(shape input)
+		(at 80.01 146.05 270)
 		(fields_autoplaced yes)
 		(effects
@@
 					(unit 1)
 				)
-			)
-		)
-	)
-	(symbol
-		(lib_id "power:+3.3V")
-		(at 77.47 154.94 180)
-		(unit 1)
-		(exclude_from_sim no)
-		(in_bom yes)
-		(on_board yes)
-		(dnp no)
-		(fields_autoplaced yes)
-		(property "Reference" "#PWR0601"
-			(at 77.47 151.13 0)
-			(effects
-				(font
-					(size 1.27 1.27)
-				)
-				(hide yes)
-			)
-		)
-		(property "Value" "+3.3V"
-			(at 77.47 160.02 0)
-			(effects
-				(font
-					(size 1.27 1.27)
-				)
-			)
-		)
-		(property "Footprint" ""
-			(at 77.47 154.94 0)
-			(effects
-				(font
-					(size 1.27 1.27)
-				)
-				(hide yes)
-			)
-		)
-		(property "Datasheet" ""
-			(at 77.47 154.94 0)
-			(effects
-				(font
-					(size 1.27 1.27)
-				)
-				(hide yes)
-			)
-		)
-		(property "Description" "Power symbol creates a global label with name \"+3.3V\""
-			(at 77.47 154.94 0)
-			(effects
-				(font
-					(size 1.27 1.27)
-				)
-				(hide yes)
-			)
-		)
-		(pin "1"
-		)
-		(instances
-			(project ""
-				(path "/37e0fdad-f3fd-48e0-8377-111662233a91/8a0e1cc3-b8cc-4980-b1ce-7a1b28674574"
-					(reference "#PWR0601")
-					(unit 1)
-				)

Commit message: empreinte
Parts:
- C3: footprint (none) -> Capacitor_SMD:C_0603_1608Metric
- C4: footprint (none) -> Capacitor_SMD:C_0402_1005Metric
- J3: footprint (none) -> Connector_JST:JST_XH_S8B-XH-A-1_1x08_P2.50mm_Horizontal
- J4, J5: footprint (none) -> Connector_JST:JST_XH_S3B-XH-A-1_1x03_P2.50mm_Horizontal
Changed lines of the file:
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@@
-	(wire
-		(pts
-			(xy 64.77 154.94) (xy 64.77 146.05)
-		)
-		(stroke
-			(width 0)
-			(type default)
-		)
-	)
 	(wire
 		(pts
@@
 			)
 		)
-		(property "Footprint" ""
+		(property "Footprint" "Capacitor_SMD:C_0402_1005Metric"
 			(at 72.39 48.26 0)
 			(effects
@@
 	)
 	(symbol
-		(lib_id "power:+5V")
-		(at 64.77 154.94 180)
-		(unit 1)
-		(exclude_from_sim no)
-		(in_bom yes)
-		(on_board yes)
-		(dnp no)
-		(fields_autoplaced yes)
-		(property "Reference" "#PWR0602"
-			(at 64.77 151.13 0)
-			(effects
-				(font
-					(size 1.27 1.27)
-				)
-				(hide yes)
-			)
-		)
-		(property "Value" "+5V"
-			(at 64.77 160.02 0)
-			(effects
-				(font
-					(size 1.27 1.27)
-				)
-			)
-		)
-		(property "Footprint" ""
-			(at 64.77 154.94 0)
-			(effects
-				(font
-					(size 1.27 1.27)
-				)
-				(hide yes)
-			)
-		)
-		(property "Datasheet" ""
-			(at 64.77 154.94 0)
-			(effects
-				(font
-					(size 1.27 1.27)
-				)
-				(hide yes)
-			)
-		)
-		(property "Description" "Power symbol creates a global label with name \"+5V\""
-			(at 64.77 154.94 0)
-			(effects
-				(font
-					(size 1.27 1.27)
-				)
-				(hide yes)
-			)
-		)
-		(pin "1"
-		)
-		(instances
-			(project ""
-				(path "/37e0fdad-f3fd-48e0-8377-111662233a91/8a0e1cc3-b8cc-4980-b1ce-7a1b28674574"
-					(reference "#PWR0602")
-					(unit 1)
-				)
-			)
-		)
-	)
-	(symbol
 		(lib_id "Device:C_Small")
 		(at 66.04 48.26 0)
@@
 			)
 		)
-		(property "Footprint" ""
+		(property "Footprint" "Capacitor_SMD:C_0603_1608Metric"
 			(at 66.04 48.26 0)
 			(effects
@@
 			)
 		)
-		(property "Footprint" ""
+		(property "Footprint" "Connector_JST:JST_XH_S3B-XH-A-1_1x03_P2.50mm_Horizontal"
 			(at 204.47 86.36 0)
 			(effects
@@
 	)
 	(symbol
+		(lib_id "power:+5V")
+		(at 64.77 146.05 180)
+		(unit 1)
+		(exclude_from_sim no)
+		(in_bom yes)
+		(on_board yes)
+		(dnp no)
+		(fields_autoplaced yes)
+		(property "Reference" "#PWR06"
+			(at 64.77 142.24 0)
+			(effects
+				(font
+					(size 1.27 1.27)
+				)
+				(hide yes)
+			)
+		)
+		(property "Value" "+5V"
+			(at 64.77 151.13 0)
+			(effects
+				(font
+					(size 1.27 1.27)
+				)
+			)
+		)
+		(property "Footprint" ""
+			(at 64.77 146.05 0)
+			(effects
+				(font
+					(size 1.27 1.27)
+				)
+				(hide yes)
+			)
+		)
+		(property "Datasheet" ""
+			(at 64.77 146.05 0)
+			(effects
+				(font
+					(size 1.27 1.27)
+				)
+				(hide yes)
+			)
+		)
+		(property "Description" "Power symbol creates a global label with name \"+5V\""
+			(at 64.77 146.05 0)
+			(effects
+				(font
+					(size 1.27 1.27)
+				)
+				(hide yes)
+			)
+		)
+		(pin "1"
+		)
+		(instances
+			(project ""
+				(path "/37e0fdad-f3fd-48e0-8377-111662233a91/8a0e1cc3-b8cc-4980-b1ce-7a1b28674574"
+					(reference "#PWR06")
+					(unit 1)
+				)
+			)
+		)
+	)
+	(symbol
 		(lib_id "Connector_Generic:Conn_01x08")
 		(at 72.39 140.97 90)
@@
 			)
 		)
-		(property "Footprint" ""
+		(property "Footprint" "Connector_JST:JST_XH_S8B-XH-A-1_1x08_P2.50mm_Horizontal"
 			(at 72.39 140.97 0)
 			(effects
@@
 			)
 		)
-		(property "Footprint" ""
+		(property "Footprint" "Connector_JST:JST_XH_S3B-XH-A-1_1x03_P2.50mm_Horizontal"
 			(at 227.33 86.36 0)
 			(effects

Commit message: Correction des erreurs évidentes
Changements avant vérification des erreurs :
- Désallocation du pin BTN_RESET
- Réarrangement de certaines sources pour cohérence avec tous les
schémas éléctriques
Other:
- note added: "Capteurs de bordure"
- note removed: "Capteur de bordure"
- moved on the sheet: C3, C4, J3, J4, J5, U2

Commit message: point de test et début de placement
Parts:
- added TP601, TP602, TP603, TP604, TP605, TP606, TP607, TP608, TP609, TP610, TP611, TP612, TP613, TP614, TP615, TP616, TP617: TestPoint, TestPoint:TestPoint_Pad_D1.0mm, symbol Connector:TestPoint
Connections:
- net +3.3V: now also TP614.1
- net +5V: now also TP615.1, TP616.1, TP617.1
- net AG_CSN: now also TP612.1
- net AG_INT1: now also TP601.1
- net AG_INT2: now also TP602.1
- net AG_MISO: now also TP603.1
- net AG_MOSI: now also TP604.1
- net AG_SCLK: now also TP611.1
- net EN_LIDAR: now also TP610.1
- net EN_MOT: now also TP609.1
- net RX_LIDAR: now also TP608.1
- net TOF1: now also TP605.1
- net TOF2: now also TP606.1
- net TX_LIDAR: now also TP607.1
- net VIT_MOT_LIDAR: now also TP613.1

Commit message: maj emplacement
Parts:
- removed TP605, TP606, TP609, TP610, TP615, TP616, TP617: TestPoint, TestPoint:TestPoint_Pad_D1.0mm, symbol Connector:TestPoint

Commit message: placement maj
Parts:
- removed TP607, TP608, TP613, TP614: TestPoint, TestPoint:TestPoint_Pad_D1.0mm, symbol Connector:TestPoint
- TP601, TP602, TP603, TP604, TP611, TP612: footprint TestPoint:TestPoint_Pad_D1.0mm -> TestPoint:TestPoint_Pad_D1.5mm
Other:
- moved on the sheet: TP604
