File: Pojet_V-NOM_KiCAD/Régulateur_5V.kicad_sch (KiCad schematic)
At the start: 30 parts, among them IC1001 MP1475SGJ-P, IC1002 MP1475SGJ-P

Commit message: Fix Librairie STM32G410CBU6 mode project
Parts:
- removed C1001: 15 p, symbol Device:C_Small
- removed C1002, C1003, C1005: 22 u, symbol Device:C_Small
- removed C1004, C1006, C1007: 0.1 u, symbol Device:C_Small
- removed L1001: 4.7 u, symbol Device:L
- removed R1001: 16 k, symbol Device:R_Small
- removed R1002: 40.2 k, symbol Device:R_Small
- removed R1003: 7.68 k, symbol Device:R_Small
- removed R1004: 100 k, symbol Device:R_Small
- removed R1005: 20, symbol Device:R_Small
- removed R1006: 100k, symbol Device:R_Small
- C1008: value 15 pF -> 15 p
- C1009, C1010: value 22 uF -> 22 u
- C1011: value 0.1 uF -> 22 u
- C1012: value 22 uF -> 0.1 u
- C1013, C1014: value 0.1 uF -> 0.1 u
- L1002: value 4.7 uH -> 4.7 u
Connections:
- net +5V: now also C1011.1, IC1002.1 (PG), R1010.2; no longer C1012.1
- net +7.2V: now also C1012.2; no longer C1011.2, IC1001.2 (IN)
- net GND: now also C1011.2, C1012.1; no longer C1011.1, C1012.2, IC1001.4 (GND)
