File: Pojet_V-NOM_KiCAD/Régulateur_5V.kicad_sch (KiCad schematic)
At the start: 15 parts, among them IC1 MP1475SGJ-P

Commit message: Maj
Maj lidar et regualteur
Parts:
- removed C10, C11, C9: 0.1 uF, symbol Device:C_Small
- removed C5: 15 pF, symbol Device:C_Small
- removed C6, C7, C8: 22 uF, symbol Device:C_Small
- removed IC1: MP1475SGJ-P, SOT65P280X100-8N, symbol MP1475SGJ-P:MP1475SGJ-P
- removed L2: 4.7 uH, symbol Device:L
- removed R10: 100k, symbol Device:R_Small
- removed R5: 40.2 k, symbol Device:R_Small
- removed R6: 7.68 k, symbol Device:R_Small
- removed R7: 100 k, symbol Device:R_Small
- removed R8: 20, symbol Device:R_Small
- removed R9: 16 k, symbol Device:R_Small
- added C1001: 15 pF, symbol Device:C_Small
- added C1002, C1003, C1005: 22 uF, symbol Device:C_Small
- added C1004, C1006, C1007: 0.1 uF, symbol Device:C_Small
- added IC1001: MP1475SGJ-P, SOT65P280X100-8N, symbol MP1475SGJ-P:MP1475SGJ-P
- added L1001: 4.7 uH, symbol Device:L
- added R1001: 16 k, symbol Device:R_Small
- added R1002: 40.2 k, symbol Device:R_Small
- added R1003: 7.68 k, symbol Device:R_Small
- added R1004: 100 k, symbol Device:R_Small
- added R1005: 20, symbol Device:R_Small
- added R1006: 100k, symbol Device:R_Small
Connections:
- net +5V: now also C1001.1, C1002.1, C1005.1, L1001.1, R1002.2
- net +7.2V: now also C1003.2, C1004.2, IC1001.2 (IN), R1006.2
- net GND: now also C1002.2, C1003.1, C1004.1, C1005.2, C1007.2, IC1001.4 (GND), R1003.2
- new net: C1001.2, R1001.1, R1002.1, R1003.1
- new net: IC1001.8 (FB), R1001.2
- new net: C1006.1, IC1001.3 (SW), L1001.2
- new net: C1006.2, R1005.2
- new net: IC1001.5 (BST), R1005.1
- new net: IC1001.1 (PG), R1004.2
- new net: IC1001.6 (EN/SYNC), R1006.1
- new net: C1007.1, IC1001.7 (VCC), R1004.1

Commit message: Retouches lisibilité Alim / capteurs
Parts:
- added C1008: 15 pF, symbol Device:C_Small
- added C1009, C1010, C1012: 22 uF, symbol Device:C_Small
- added C1011, C1013, C1014: 0.1 uF, symbol Device:C_Small
- added IC1002: MP1475SGJ-P, SOT65P280X100-8N, symbol MP1475SGJ-P:MP1475SGJ-P
- added L1002: 4.7 uH, symbol Device:L
- added R1007: 16 k, symbol Device:R_Small
- added R1008: 40.2 k, symbol Device:R_Small
- added R1009: 7.68 k, symbol Device:R_Small
- added R1010: 100 k, symbol Device:R_Small
- added R1011: 20, symbol Device:R_Small
- added R1012: 100k, symbol Device:R_Small
- C1001: value 15 pF -> 15 p
- C1002, C1003, C1005: value 22 uF -> 22 u
- C1004, C1006, C1007: value 0.1 uF -> 0.1 u
- L1001: value 4.7 uH -> 4.7 u
Connections:
- net +5V: now also C1008.1, C1009.1, C1012.1, L1002.1, R1008.2
- net +7.2V: now also C1010.2, C1011.2, IC1002.2 (IN), R1012.2
- net GND: now also C1009.2, C1010.1, C1011.1, C1012.2, C1014.2, IC1002.4 (GND), R1009.2
- new net: IC1002.5 (BST), R1011.1
- new net: C1013.2, R1011.2
- new net: C1008.2, R1007.1, R1008.1, R1009.1
- new net: C1013.1, IC1002.3 (SW), L1002.2
- new net: IC1002.6 (EN/SYNC), R1012.1
- new net: IC1002.8 (FB), R1007.2
- new net: C1014.1, IC1002.7 (VCC), R1010.1
- new net: IC1002.1 (PG), R1010.2
Other:
- note added: "Régulateur 5V"
- moved on the sheet: C1001, C1002, C1005, C1006, C1007, IC1001, L1001, R1001, R1002, R1003, R1004, R1005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

Commit message: maj regulateur 5V
Parts:
- removed C1001: 15 p, symbol Device:C_Small
- removed C1002, C1003, C1005: 22 u, symbol Device:C_Small
- removed C1004, C1006, C1007: 0.1 u, symbol Device:C_Small
- removed IC1001: MP1475SGJ-P, SOT65P280X100-8N, symbol MP1475SGJ-P:MP1475SGJ-P
- removed L1001: 4.7 u, symbol Device:L
- removed R1001: 16 k, symbol Device:R_Small
- removed R1002: 40.2 k, symbol Device:R_Small
- removed R1003: 7.68 k, symbol Device:R_Small
- removed R1004: 100 k, symbol Device:R_Small
- removed R1005: 20, symbol Device:R_Small
- removed R1006: 100k, symbol Device:R_Small
Connections:
- net +5V: now also R1008.1; no longer R1008.2
- net at R1011.2: now also C1013.1; no longer C1013.2
- net at C1008.2, R1007.1, R1009.1: now also R1008.2; no longer R1008.1
- net at IC1002.3 (SW), L1002.2: now also C1013.2; no longer C1013.1
- net at C1014.1, IC1002.7 (VCC): now also R1010.2; no longer R1010.1
- net at IC1002.1 (PG): now also R1010.1; no longer R1010.2
Other:
- moved on the sheet: C1008, C1009, C1012, C1013, C1014, IC1002, L1002, R1007, R1008, R1009, R1010, R1011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

Commit message: DERNIER MODIF Alim
Connections:
- net +7.2V renamed +BATT
Changed lines of the file:
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@@
-		)
-	)
-	(hierarchical_label "+7.2V"
-		(shape input)
-		(at 77.47 80.01 180)
-		(fields_autoplaced yes)
-		(effects
-			(font
-				(size 1.27 1.27)
-			)
-			(justify right)
-		)
-	)
-	(hierarchical_label "+5V"
-		(shape input)
-		(at 208.28 91.44 0)
-		(fields_autoplaced yes)
-		(effects
-			(font
-				(size 1.27 1.27)
-			)
-			(justify left)
 		)
 	)
@@
 				(path "/37e0fdad-f3fd-48e0-8377-111662233a91/aef3d9b2-029f-4338-91be-d4af664a9426/8d105b4f-1ef8-4d0d-b5ad-377f3bebef1c"
 					(reference "C1008")
+					(unit 1)
+				)
+			)
+		)
+	)
+	(symbol
+		(lib_id "power:+BATT")
+		(at 77.47 80.01 0)
+		(unit 1)
+		(exclude_from_sim no)
+		(in_bom yes)
+		(on_board yes)
+		(dnp no)
+		(fields_autoplaced yes)
+		(property "Reference" "#PWR01001"
+			(at 77.47 83.82 0)
+			(effects
+				(font
+					(size 1.27 1.27)
+				)
+				(hide yes)
+			)
+		)
+		(property "Value" "+BATT"
+			(at 77.47 74.93 0)
+			(effects
+				(font
+					(size 1.27 1.27)
+				)
+			)
+		)
+		(property "Footprint" ""
+			(at 77.47 80.01 0)
+			(effects
+				(font
+					(size 1.27 1.27)
+				)
+				(hide yes)
+			)
+		)
+		(property "Datasheet" ""
+			(at 77.47 80.01 0)
+			(effects
+				(font
+					(size 1.27 1.27)
+				)
+				(hide yes)
+			)
+		)
+		(property "Description" "Power symbol creates a global label with name \"+BATT\""
+			(at 77.47 80.01 0)
+			(effects
+				(font
+					(size 1.27 1.27)
+				)
+				(hide yes)
+			)
+		)
+		(pin "1"
+		)
+		(instances
+			(project "Pojet_V-NOM_KiCAD"
+				(path "/37e0fdad-f3fd-48e0-8377-111662233a91/aef3d9b2-029f-4338-91be-d4af664a9426/8d105b4f-1ef8-4d0d-b5ad-377f3bebef1c"
+					(reference "#PWR01001")
 					(unit 1)
 				)
@@
 					(unit 1)
 				)
+			)
+		)
+	)
+	(symbol
+		(lib_id "power:+5V")
+		(at 208.28 91.44 0)
+		(unit 1)
+		(exclude_from_sim no)
+		(in_bom yes)
+		(on_board yes)
+		(dnp no)
+		(fields_autoplaced yes)
+		(property "Reference" "#PWR01002"
+			(at 208.28 95.25 0)
+			(effects
+				(font
+					(size 1.27 1.27)
+				)
+				(hide yes)
+			)
+		)
+		(property "Value" "+5V"
+			(at 208.28 86.36 0)
+			(effects
+				(font
+					(size 1.27 1.27)
+				)
+			)
+		)
+		(property "Footprint" ""
+			(at 208.28 91.44 0)
+			(effects
+				(font
+					(size 1.27 1.27)
+				)
+				(hide yes)
+			)
+		)
+		(property "Datasheet" ""
+			(at 208.28 91.44 0)
+			(effects
+				(font
+					(size 1.27 1.27)
+				)
+				(hide yes)
+			)
+		)
+		(property "Description" "Power symbol creates a global label with name \"+5V\""
+			(at 208.28 91.44 0)
+			(effects
+				(font
+					(size 1.27 1.27)
+				)
+				(hide yes)
+			)
+		)
+		(pin "1"
+		)
+		(instances
+			(project ""
+				(path "/37e0fdad-f3fd-48e0-8377-111662233a91/aef3d9b2-029f-4338-91be-d4af664a9426/8d105b4f-1ef8-4d0d-b5ad-377f3bebef1c"
+					(reference "#PWR01002")
+					(unit 1)
+				)

Commit message: empreinte
Parts:
- C1008, C1011, C1013, C1014: footprint (none) -> Capacitor_SMD:C_0402_1005Metric
- C1009, C1010, C1012: footprint (none) -> Capacitor_SMD:C_0805_2012Metric
- IC1002: footprint SOT65P280X100-8N -> KiCad:SOT65P280X100-8N
- L1002: footprint (none) -> Capacitor_SMD:C_0603_1608Metric
- R1007, R1008, R1009, R1010, R1011, R1012: footprint (none) -> Resistor_SMD:R_0402_1005Metric
Changed lines of the file:
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@@
 			)
 		)
-		(property "Footprint" ""
+		(property "Footprint" "Resistor_SMD:R_0402_1005Metric"
 			(at 149.86 80.01 0)
 			(effects
@@
 			)
 		)
-		(property "Footprint" ""
+		(property "Footprint" "Capacitor_SMD:C_0402_1005Metric"
 			(at 187.96 107.95 0)
 			(effects
@@
 			)
 		)
-		(property "Footprint" ""
+		(property "Footprint" "Resistor_SMD:R_0402_1005Metric"
 			(at 166.37 118.11 0)
 			(effects
@@
 			)
 		)
-		(property "Footprint" ""
+		(property "Footprint" "Capacitor_SMD:C_0402_1005Metric"
 			(at 157.48 83.82 0)
 			(effects
@@
 			)
 		)
-		(property "Footprint" ""
+		(property "Footprint" "Capacitor_SMD:C_0603_1608Metric"
 			(at 173.99 91.44 0)
 			(effects
@@
 			)
 		)
-		(property "Footprint" ""
+		(property "Footprint" "Capacitor_SMD:C_0805_2012Metric"
 			(at 196.85 93.98 0)
 			(effects
@@
 			)
 		)
-		(property "Footprint" ""
+		(property "Footprint" "Capacitor_SMD:C_0402_1005Metric"
 			(at 96.52 82.55 0)
 			(effects
@@
 			)
 		)
-		(property "Footprint" ""
+		(property "Footprint" "Resistor_SMD:R_0402_1005Metric"
 			(at 186.69 115.57 0)
 			(effects
@@
 			)
 		)
-		(property "Footprint" ""
+		(property "Footprint" "Resistor_SMD:R_0402_1005Metric"
 			(at 107.95 115.57 0)
 			(effects
@@
 			)
 		)
-		(property "Footprint" ""
+		(property "Footprint" "Resistor_SMD:R_0402_1005Metric"
 			(at 152.4 115.57 0)
 			(effects
@@
 			)
 		)
-		(property "Footprint" ""
+		(property "Footprint" "Resistor_SMD:R_0402_1005Metric"
 			(at 87.63 96.52 0)
 			(effects
@@
 			)
 		)
-		(property "Footprint" ""
+		(property "Footprint" "Capacitor_SMD:C_0805_2012Metric"
 			(at 102.87 82.55 0)
 			(effects
@@
 			)
 		)
-		(property "Footprint" ""
+		(property "Footprint" "Capacitor_SMD:C_0805_2012Metric"
 			(at 182.88 93.98 0)
 			(effects
@@
 			)
 		)
-		(property "Footprint" "SOT65P280X100-8N"
+		(property "Footprint" "KiCad:SOT65P280X100-8N"
 			(at 139.7 174.93 0)
 			(effects
@@
 			)
 		)
-		(property "Footprint" ""
+		(property "Footprint" "Capacitor_SMD:C_0402_1005Metric"
 			(at 105.41 96.52 0)
 			(effects

Commit message: point de test et début de placement
Parts:
- added TP1001, TP1002, TP1003: TestPoint, TestPoint:TestPoint_Pad_D1.0mm, symbol Connector:TestPoint
- IC1002: footprint KiCad:SOT65P280X100-8N -> Package_TO_SOT_SMD:SOT-23-8
Connections:
- net +5V: now also TP1001.1
- net +BATT: now also TP1002.1
- net at C1014.1, IC1002.7 (VCC), R1010.2: now also TP1003.1

Commit message: placement maj
Parts:
- L1002: footprint Capacitor_SMD:C_0603_1608Metric -> Inductor_SMD:L_0402_1005Metric
- TP1001, TP1002, TP1003: footprint TestPoint:TestPoint_Pad_D1.0mm -> TestPoint:TestPoint_Pad_D1.5mm
Changed lines of the file:
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@@
 			)
 		)
-		(property "Footprint" "TestPoint:TestPoint_Pad_D1.0mm"
+		(property "Footprint" "TestPoint:TestPoint_Pad_D1.5mm"
 			(at 92.71 91.44 0)
 			(effects
@@
 			)
 		)
-		(property "Footprint" "Capacitor_SMD:C_0603_1608Metric"
+		(property "Footprint" "Inductor_SMD:L_0402_1005Metric"
 			(at 173.99 91.44 0)
 			(effects
@@
 			)
 		)
-		(property "Footprint" "TestPoint:TestPoint_Pad_D1.0mm"
+		(property "Footprint" "TestPoint:TestPoint_Pad_D1.5mm"
 			(at 80.01 80.01 0)
 			(effects
@@
 			)
 		)
-		(property "Footprint" "TestPoint:TestPoint_Pad_D1.0mm"
+		(property "Footprint" "TestPoint:TestPoint_Pad_D1.5mm"
 			(at 212.09 91.44 0)
 			(effects

Commit message: maj routage
Parts:
- L1002: footprint Inductor_SMD:L_0402_1005Metric -> Library:Inductance L1
Changed lines of the file:
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@@
 			)
 		)
-		(property "Footprint" "Inductor_SMD:L_0402_1005Metric"
+		(property "Footprint" "Library:Inductance L1"
 			(at 173.99 91.44 0)
 			(effects
