File: Pojet_V-NOM_KiCAD/alimentation.kicad_sch (KiCad schematic)
At the start: 21 parts, among them IC401 MP1475SGJ-P, U401 ADXL343

Commit message: Ajout de toutes les feuilles au projet principal
Parts:
- removed C404: 10 uF, symbol Device:C_Small
- removed C405: 0.1 uF, symbol Device:C_Small
- removed R403: 10 k, symbol Device:R_Small
- removed U401: ADXL343, Package_LGA:LGA-14_3x5mm_P0.8mm_LayoutBorder1x6y, symbol Sensor_Motion:ADXL343
Connections:
- no-connect marks 2 -> 0
Other:
- note removed: "Accéléromètre"

Commit message: rajout capteur
capteur de bordure
Connections:
- net +7.5V: now also C406.1, IC401.3 (SW), L401.2
Other:
- moved on the sheet: C403
Changed lines of the file:
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@@
+	)
+	(junction
+		(at 58.42 62.23)
+		(diameter 0)
+		(color 0 0 0 0)
 	)
 	(junction
@@
 	(wire
 		(pts
+			(xy 58.42 62.23) (xy 60.96 62.23)
+		)
+		(stroke
+			(width 0)
+			(type default)
+		)
+	)
+	(wire
+		(pts
 			(xy 113.03 59.69) (xy 113.03 82.55)
 		)
@@
 	(wire
 		(pts
+			(xy 58.42 73.66) (xy 58.42 62.23)
+		)
+		(stroke
+			(width 0)
+			(type default)
+		)
+	)
+	(wire
+		(pts
 			(xy 170.18 58.42) (xy 170.18 59.69)
 		)
@@
 	(wire
 		(pts
-			(xy 58.42 64.77) (xy 58.42 59.69)
-		)
-		(stroke
-			(width 0)
-			(type default)
-		)
-	)
-	(wire
-		(pts
-			(xy 58.42 71.12) (xy 58.42 69.85)
-		)
-		(stroke
-			(width 0)
-			(type default)
-		)
-	)
-	(wire
-		(pts
-			(xy 53.34 62.23) (xy 60.96 62.23)
+			(xy 58.42 62.23) (xy 58.42 59.69)
+		)
+		(stroke
+			(width 0)
+			(type default)
+		)
+	)
+	(wire
+		(pts
+			(xy 58.42 87.63) (xy 58.42 78.74)
+		)
+		(stroke
+			(width 0)
+			(type default)
+		)
+	)
+	(wire
+		(pts
+			(xy 53.34 62.23) (xy 58.42 62.23)
 		)
 		(stroke
@@
 		(dnp no)
 		(property "Reference" "R402"
-			(at 33.02 71.12 0)
+			(at 33.02 70.358 0)
 			(effects
 				(font
@@
 		)
 		(property "Value" "13 k"
-			(at 32.258 72.898 0)
+			(at 33.02 72.39 0)
 			(effects
 				(font
@@
 	(symbol
 		(lib_id "Device:C_Small")
-		(at 58.42 67.31 0)
+		(at 58.42 76.2 0)
 		(unit 1)
 		(exclude_from_sim no)
@@
 		(dnp no)
 		(property "Reference" "C403"
-			(at 54.61 68.072 0)
+			(at 52.578 74.676 0)
 			(effects
 				(font
@@
 		)
 		(property "Value" "22 uF"
-			(at 52.832 69.85 0)
+			(at 55.372 78.486 0)
 			(effects
 				(font
@@
 		)
 		(property "Footprint" ""
-			(at 58.42 67.31 0)
+			(at 58.42 76.2 0)
 			(effects
 				(font
@@
 		)
 		(property "Datasheet" "~"
-			(at 58.42 67.31 0)
+			(at 58.42 76.2 0)
 			(effects
 				(font
@@
 		)
 		(property "Description" "Unpolarized capacitor, small symbol"
-			(at 58.42 67.31 0)
+			(at 58.42 76.2 0)
 			(effects
 				(font
@@
 	(symbol
 		(lib_id "power:GND")
-		(at 58.42 71.12 0)
+		(at 58.42 87.63 0)
 		(unit 1)
 		(exclude_from_sim no)
@@
 		(fields_autoplaced yes)
 		(property "Reference" "#PWR0408"
-			(at 58.42 77.47 0)
+			(at 58.42 93.98 0)
 			(effects
 				(font
@@
 		)
 		(property "Value" "GND"
-			(at 58.42 76.2 0)
-			(effects
-				(font
-					(size 1.27 1.27)
-				)
-			)
-		)
-		(property "Footprint" ""
-			(at 58.42 71.12 0)
+			(at 58.42 92.71 0)
+			(effects
+				(font
+					(size 1.27 1.27)
+				)
+			)
+		)
+		(property "Footprint" ""
+			(at 58.42 87.63 0)
 			(effects
 				(font
@@
 		)
 		(property "Datasheet" ""
-			(at 58.42 71.12 0)
+			(at 58.42 87.63 0)
 			(effects
 				(font
@@
 		)
 		(property "Description" "Power symbol creates a global label with name \"GND\" , ground"
-			(at 58.42 71.12 0)
+			(at 58.42 87.63 0)
 			(effects
 				(font
@@
 		(dnp no)
 		(property "Reference" "R401"
-			(at 32.512 65.024 0)
+			(at 32.766 64.262 0)
 			(effects
 				(font
@@
 		)
 		(property "Value" "40.2 k"
-			(at 31.242 66.802 0)
-			(effects
-				(font
+			(at 32.004 66.04 0)
+			(effects
+				(font

Commit message: regulateur 5 V
Regulateur 5V maj
Parts:
- removed R407: 100k, symbol Device:R_Small
- added C404: 22 uF, symbol Device:C_Small
- added C405, C409: 0.1 uF, symbol Device:C_Small
- added R403: 100 k, symbol Device:R_Small
- C401: value 47 uF -> 15 pF
- C402: value 0.1 uF -> 22 uF
- R402: value 13 k -> 7.68 k
- R404: value 100 k -> 20
- R405: value 20 -> 16 k
- R406: value 16 k -> 100k
Connections:
- net +5V: now also C402.1, C404.1
- net +7.5V: now also C403.2, R406.2, C405.2; no longer C403.1, C406.1, IC401.3 (SW), L401.2
- net GND: now also C403.1, C404.2, C405.1, C409.2; no longer C401.2, C403.2
- net at R401.1, R402.1: now also C401.2, R405.2; no longer R406.2
- net at IC401.5 (BST): now also R404.1; no longer R405.1
- net at IC401.6 (EN/SYNC): now also R406.1
- net at IC401.7 (VCC): now also C409.1, R403.1; no longer R404.1
- net at IC401.8 (FB): now also R405.1; no longer R406.1
- net at C406.2: now also R404.2; no longer R405.2
- new net: C406.1, IC401.3 (SW), L401.2
- new net: IC401.1 (PG), R403.2

Commit message: MAJ Valerian
MAJ Valerian
Other:
- note added: "Batterie"
- moved on the sheet: BT401, C407, C408, PS401, R408

Commit message: modif
Parts:
- removed BT401: Battery, symbol Device:Battery
- removed C401: 15 pF, symbol Device:C_Small
- removed C402, C403, C404: 22 uF, symbol Device:C_Small
- removed C405, C406, C409: 0.1 uF, symbol Device:C_Small
- removed C407, C408: 0.47 uF, symbol Device:C_Small
- removed IC401: MP1475SGJ-P, SOT65P280X100-8N, symbol MP1475SGJ-P:MP1475SGJ-P
- removed L401: 4.7 uH, symbol Device:L
- removed PS401: BU33SD5WG-TR, SOT95P280X125-5N, symbol BU33SD5WG-TR:BU33SD5WG-TR
- removed R401: 40.2 k, symbol Device:R_Small
- removed R402: 7.68 k, symbol Device:R_Small
- removed R403: 100 k, symbol Device:R_Small
- removed R404: 20, symbol Device:R_Small
- removed R405: 16 k, symbol Device:R_Small
- removed R406: 100k, symbol Device:R_Small
- removed R408: 10 k, symbol Device:R_Small
- added BT1: Battery, symbol Device:Battery
Connections:
- net GND: now also BT1.2 (-)
- new net +7.2V: BT1.1 (+)
Other:
- added sheet Régulateur_3.3V (Régulateur_3.3V.kicad_sch)
- added sheet Régulateur_5V (Régulateur_5V.kicad_sch)
- note removed: "Régulateur 3.3v"
- note removed: "Régulateur 5V"

Commit message: maj
Changed lines of the file:
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@@
 	(paper "A4")
-	(junction
-		(at 149.86 85.09)
-		(diameter 0)
-		(color 0 0 0 0)
-	)
 	(junction
 		(at 68.58 83.82)
@@
 	(wire
 		(pts
-			(xy 143.51 85.09) (xy 149.86 85.09)
-		)
-		(stroke
-			(width 0)
-			(type default)
-		)
-	)
-	(wire
-		(pts
-			(xy 149.86 85.09) (xy 186.69 85.09)
-		)
-		(stroke
-			(width 0)
-			(type default)
-		)
-	)
-	(wire
-		(pts
-			(xy 149.86 78.74) (xy 149.86 85.09)
+			(xy 143.51 85.09) (xy 186.69 85.09)
 		)
 		(stroke
@@
 		(fields_autoplaced yes)
 		(effects
-			(font
-				(size 1.27 1.27)
-			)
-			(justify left)
-		)
-	)
-	(hierarchical_label "+5V"
-		(shape output)
-		(at 149.86 78.74 90)
-		(fields_autoplaced yes)
-		(effects

Commit message: Corrections sonde et switch
Parts:
- added J6: Conn_01x02, Connector_JST:JST_XH_S2B-XH-A_1x02_P2.50mm_Horizontal, symbol Connector_Generic:Conn_01x02
Connections:
- net +7.2V: now also J6.2 (Pin_2); no longer BT1.1 (+)
- new net: BT1.1 (+), J6.1 (Pin_1)
Other:
- moved on the sheet: BT1
Changed lines of the file:
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@@
 	(paper "A4")
 	(junction
-		(at 68.58 83.82)
+		(at 71.12 83.82)
 		(diameter 0)
 		(color 0 0 0 0)
@@
 	(wire
 		(pts
-			(xy 62.23 83.82) (xy 68.58 83.82)
-		)
-		(stroke
-			(width 0)
-			(type default)
-		)
-	)
-	(wire
-		(pts
-			(xy 52.07 83.82) (xy 49.53 83.82)
-		)
-		(stroke
-			(width 0)
-			(type default)
-		)
-	)
-	(wire
-		(pts
-			(xy 68.58 80.01) (xy 68.58 83.82)
+			(xy 35.56 93.98) (xy 35.56 96.52)
+		)
+		(stroke
+			(width 0)
+			(type default)
+		)
+	)
+	(wire
+		(pts
+			(xy 71.12 80.01) (xy 71.12 83.82)
+		)
+		(stroke
+			(width 0)
+			(type default)
+		)
+	)
+	(wire
+		(pts
+			(xy 53.34 83.82) (xy 71.12 83.82)
+		)
+		(stroke
+			(width 0)
+			(type default)
+		)
+	)
+	(wire
+		(pts
+			(xy 35.56 83.82) (xy 50.8 83.82)
+		)
+		(stroke
+			(width 0)
+			(type default)
+		)
+	)
+	(wire
+		(pts
+			(xy 71.12 83.82) (xy 76.2 83.82)
 		)
 		(stroke
@@
 		(pts
 			(xy 143.51 85.09) (xy 186.69 85.09)
-		)
-		(stroke
-			(width 0)
-			(type default)
-		)
-	)
-	(wire
-		(pts
-			(xy 68.58 83.82) (xy 76.2 83.82)
 		)
 		(stroke
@@
 	(hierarchical_label "+7.2V"
 		(shape output)
-		(at 68.58 80.01 90)
+		(at 71.12 80.01 90)
 		(fields_autoplaced yes)
 		(effects
@@
 	(symbol
 		(lib_id "power:GND")
-		(at 49.53 83.82 270)
+		(at 35.56 96.52 0)
 		(unit 1)
 		(exclude_from_sim no)
@@
 		(fields_autoplaced yes)
 		(property "Reference" "#PWR05"
-			(at 43.18 83.82 0)
+			(at 35.56 102.87 0)
 			(effects
 				(font
@@
 		)
 		(property "Value" "GND"
-			(at 45.72 83.8199 90)
+			(at 35.5599 100.33 90)
 			(effects
 				(font
@@
 		)
 		(property "Footprint" ""
-			(at 49.53 83.82 0)
+			(at 35.56 96.52 0)
 			(effects
 				(font
@@
 		)
 		(property "Datasheet" ""
-			(at 49.53 83.82 0)
+			(at 35.56 96.52 0)
 			(effects
 				(font
@@
 		)
 		(property "Description" "Power symbol creates a global label with name \"GND\" , ground"
-			(at 49.53 83.82 0)
+			(at 35.56 96.52 0)
 			(effects
 				(font
@@
 	)
 	(symbol
-		(lib_id "Device:Battery")
-		(at 57.15 83.82 270)
+		(lib_id "Connector_Generic:Conn_01x02")
+		(at 50.8 78.74 90)
 		(unit 1)
 		(exclude_from_sim no)
@@
 		(dnp no)
 		(fields_autoplaced yes)
+		(property "Reference" "J6"
+			(at 55.88 77.4699 90)
+			(effects
+				(font
+					(size 1.27 1.27)
+				)
+				(justify right)
+			)
+		)
+		(property "Value" "Conn_01x02"
+			(at 55.88 80.0099 90)
+			(effects
+				(font
+					(size 1.27 1.27)
+				)
+				(justify right)
+			)
+		)
+		(property "Footprint" "Connector_JST:JST_XH_S2B-XH-A_1x02_P2.50mm_Horizontal"
+			(at 50.8 78.74 0)
+			(effects
+				(font
+					(size 1.27 1.27)
+				)
+				(hide yes)
+			)
+		)
+		(property "Datasheet" "~"
+			(at 50.8 78.74 0)
+			(effects
+				(font
+					(size 1.27 1.27)
+				)
+				(hide yes)
+			)
+		)
+		(property "Description" "Generic connector, single row, 01x02, script generated (kicad-library-utils/schlib/autogen/connector/)"
+			(at 50.8 78.74 0)
+			(effects
+				(font
+					(size 1.27 1.27)
+				)
+				(hide yes)
+			)
+		)
+		(pin "2"
+		)
+		(pin "1"
+		)
+		(instances
+			(project ""
+				(path "/37e0fdad-f3fd-48e0-8377-111662233a91/aef3d9b2-029f-4338-91be-d4af664a9426"
+					(reference "J6")
+					(unit 1)
+				)
+			)
+		)
+	)
+	(symbol
+		(lib_id "Device:Battery")
+		(at 35.56 88.9 0)
+		(unit 1)
+		(exclude_from_sim no)
+		(in_bom yes)
+		(on_board yes)
+		(dnp no)
+		(fields_autoplaced yes)
 		(property "Reference" "BT1"
-			(at 57.7215 76.2 90)
+			(at 27.94 88.3285 90)
 			(effects
 				(font
@@
 		)
 		(property "Value" "Battery"
-			(at 57.7215 78.74 90)
+			(at 30.48 88.3285 90)
 			(effects
 				(font
@@
 		)
 		(property "Footprint" ""
-			(at 58.674 83.82 90)
+			(at 35.56 87.376 90)
 			(effects
 				(font
@@
 		)
 		(property "Datasheet" "~"
-			(at 58.674 83.82 90)
+			(at 35.56 87.376 90)
 			(effects
 				(font
@@
 		)
 		(property "Description" "Multiple-cell battery"
-			(at 57.15 83.82 0)
-			(effects
-				(font
+			(at 35.56 88.9 0)
+			(effects
+				(font

Commit message: DERNIER MODIF Alim
Parts:
- BT1: value Battery -> +7.2V
Connections:
- net +7.2V renamed +BATT
Other:
- sheet Régulateur_3.3V ports: added none; removed +3.3V, +5V
- sheet Régulateur_5V ports: added none; removed +5V, +7.2V
Changed lines of the file:
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@@
 	(generator_version "8.0")
 	(paper "A4")
-	(junction
-		(at 71.12 83.82)
-		(diameter 0)
-		(color 0 0 0 0)
-	)
 	(wire
 		(pts
-			(xy 241.3 85.09) (xy 247.65 85.09)
+			(xy 53.34 83.82) (xy 72.39 83.82)
 		)
 		(stroke
@@
 	(wire
 		(pts
-			(xy 71.12 80.01) (xy 71.12 83.82)
-		)
-		(stroke
-			(width 0)
-			(type default)
-		)
-	)
-	(wire
-		(pts
-			(xy 53.34 83.82) (xy 71.12 83.82)
-		)
-		(stroke
-			(width 0)
-			(type default)
-		)
-	)
-	(wire
-		(pts
 			(xy 35.56 83.82) (xy 50.8 83.82)
-		)
-		(stroke
-			(width 0)
-			(type default)
-		)
-	)
-	(wire
-		(pts
-			(xy 71.12 83.82) (xy 76.2 83.82)
-		)
-		(stroke
-			(width 0)
-			(type default)
-		)
-	)
-	(wire
-		(pts
-			(xy 143.51 85.09) (xy 186.69 85.09)
 		)
 		(stroke
@@
 		)
 	)
-	(hierarchical_label "+3.3V"
-		(shape output)
-		(at 247.65 85.09 0)
-		(fields_autoplaced yes)
-		(effects
-			(font
-				(size 1.27 1.27)
-			)
-			(justify left)
-		)
-	)
-	(hierarchical_label "+7.2V"
-		(shape output)
-		(at 71.12 80.01 90)
-		(fields_autoplaced yes)
-		(effects
-			(font
-				(size 1.27 1.27)
-			)
-			(justify left)
-		)
-	)
 	(symbol
 		(lib_id "power:GND")
@@
 	)
 	(symbol
+		(lib_id "power:+BATT")
+		(at 72.39 83.82 0)
+		(unit 1)
+		(exclude_from_sim no)
+		(in_bom yes)
+		(on_board yes)
+		(dnp no)
+		(fields_autoplaced yes)
+		(property "Reference" "#PWR0401"
+			(at 72.39 87.63 0)
+			(effects
+				(font
+					(size 1.27 1.27)
+				)
+				(hide yes)
+			)
+		)
+		(property "Value" "+BATT"
+			(at 72.39 78.74 0)
+			(effects
+				(font
+					(size 1.27 1.27)
+				)
+			)
+		)
+		(property "Footprint" ""
+			(at 72.39 83.82 0)
+			(effects
+				(font
+					(size 1.27 1.27)
+				)
+				(hide yes)
+			)
+		)
+		(property "Datasheet" ""
+			(at 72.39 83.82 0)
+			(effects
+				(font
+					(size 1.27 1.27)
+				)
+				(hide yes)
+			)
+		)
+		(property "Description" "Power symbol creates a global label with name \"+BATT\""
+			(at 72.39 83.82 0)
+			(effects
+				(font
+					(size 1.27 1.27)
+				)
+				(hide yes)
+			)
+		)
+		(pin "1"
+		)
+		(instances
+			(project "Pojet_V-NOM_KiCAD"
+				(path "/37e0fdad-f3fd-48e0-8377-111662233a91/aef3d9b2-029f-4338-91be-d4af664a9426"
+					(reference "#PWR0401")
+					(unit 1)
+				)
+			)
+		)
+	)
+	(symbol
 		(lib_id "Device:Battery")
 		(at 35.56 88.9 0)
@@
 			)
 		)
-		(property "Value" "Battery"
+		(property "Value" "+7.2V"
 			(at 30.48 88.3285 90)
 			(effects
@@
 	)
 	(sheet
-		(at 76.2 63.5)
+		(at 91.44 66.04)
 		(size 67.31 44.45)
 		(fields_autoplaced yes)
@@
 		)
 		(property "Sheetname" "Régulateur_5V"
-			(at 76.2 62.1534 0)
+			(at 91.44 64.6934 0)
 			(effects
 				(font
@@
 		)
 		(property "Sheetfile" "Régulateur_5V.kicad_sch"
-			(at 76.2 108.5346 0)
+			(at 91.44 111.0746 0)
 			(effects
 				(font
@@
 				)
 				(justify left top)
-			)
-		)
-		(pin "+5V" output
-			(at 143.51 85.09 0)
-			(effects
-				(font
-					(size 1.27 1.27)
-				)
-				(justify right)
-			)
-		)
-		(pin "+7.2V" input
-			(at 76.2 83.82 180)
-			(effects
-				(font
-					(size 1.27 1.27)
-				)
-				(justify left)
 			)
 		)
@@
 			)
 		)
-		(pin "+3.3V" output
-			(at 241.3 85.09 0)
-			(effects
-				(font
-					(size 1.27 1.27)
-				)
-				(justify right)
-			)
-		)
-		(pin "+5V" input
-			(at 186.69 85.09 180)
-			(effects
-				(font
-					(size 1.27 1.27)
-				)
-				(justify left)
-			)
-		)
