File: Pojet_V-NOM_KiCAD/Régulateur_3.3V.kicad_sch (KiCad schematic)
At the start: 3 parts

Commit message: Maj
Maj lidar et regualteur
Parts:
- removed C12, C13: 1uF, symbol Device:C_Small
- removed PS1: BU33SD5WG-TR, SOT95P280X125-5N, symbol BU33SD5WG-TR:BU33SD5WG-TR
- added C901, C902: 1uF, symbol Device:C_Small
- added PS901: BU33SD5WG-TR, SOT95P280X125-5N, symbol BU33SD5WG-TR:BU33SD5WG-TR
Connections:
- net +3.3V: now also C902.1, PS901.5 (VOUT)
- net +5V: now also C901.1, PS901.1 (VIN), PS901.3 (STBY)
- net GND: now also C901.2, C902.2, PS901.2 (GND)

Commit message: Retouches lisibilité Alim / capteurs
Other:
- note added: "Régulateur 3.3V"
- moved on the sheet: C901, C902, PS901
Changed lines of the file:
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@@
 	(paper "A4")
 	(junction
-		(at 128.27 92.71)
+		(at 119.38 101.6)
 		(diameter 0)
 		(color 0 0 0 0)
 	)
 	(junction
-		(at 172.72 95.25)
+		(at 163.83 104.14)
 		(diameter 0)
 		(color 0 0 0 0)
@@
 	(wire
 		(pts
-			(xy 139.7 95.25) (xy 142.24 95.25)
-		)
-		(stroke
-			(width 0)
-			(type default)
-		)
-	)
-	(wire
-		(pts
-			(xy 172.72 95.25) (xy 172.72 99.06)
-		)
-		(stroke
-			(width 0)
-			(type default)
-		)
-	)
-	(wire
-		(pts
-			(xy 170.18 95.25) (xy 172.72 95.25)
-		)
-		(stroke
-			(width 0)
-			(type default)
-		)
-	)
-	(wire
-		(pts
-			(xy 121.92 92.71) (xy 128.27 92.71)
-		)
-		(stroke
-			(width 0)
-			(type default)
-		)
-	)
-	(wire
-		(pts
-			(xy 128.27 92.71) (xy 142.24 92.71)
-		)
-		(stroke
-			(width 0)
-			(type default)
-		)
-	)
-	(wire
-		(pts
-			(xy 172.72 95.25) (xy 179.07 95.25)
-		)
-		(stroke
-			(width 0)
-			(type default)
-		)
-	)
-	(wire
-		(pts
-			(xy 172.72 106.68) (xy 172.72 104.14)
-		)
-		(stroke
-			(width 0)
-			(type default)
+			(xy 163.83 104.14) (xy 163.83 107.95)
+		)
+		(stroke
+			(width 0)
+			(type default)
+		)
+	)
+	(wire
+		(pts
+			(xy 127 104.14) (xy 133.35 104.14)
+		)
+		(stroke
+			(width 0)
+			(type default)
+		)
+	)
+	(wire
+		(pts
+			(xy 161.29 104.14) (xy 163.83 104.14)
+		)
+		(stroke
+			(width 0)
+			(type default)
+		)
+	)
+	(wire
+		(pts
+			(xy 113.03 101.6) (xy 119.38 101.6)
+		)
+		(stroke
+			(width 0)
+			(type default)
+		)
+	)
+	(wire
+		(pts
+			(xy 119.38 101.6) (xy 133.35 101.6)
+		)
+		(stroke
+			(width 0)
+			(type default)
+		)
+	)
+	(wire
+		(pts
+			(xy 163.83 104.14) (xy 170.18 104.14)
+		)
+		(stroke
+			(width 0)
+			(type default)
+		)
+	)
+	(wire
+		(pts
+			(xy 127 113.03) (xy 127 104.14)
+		)
+		(stroke
+			(width 0)
+			(type default)
+		)
+	)
+	(wire
+		(pts
+			(xy 163.83 115.57) (xy 163.83 113.03)
+		)
+		(stroke
+			(width 0)
+			(type default)
+		)
+	)
+	(text "Régulateur 3.3V"
+		(exclude_from_sim no)
+		(at 34.036 19.812 0)
+		(effects
+			(font
+				(size 2.54 2.54)
+			)
 		)
 	)
 	(hierarchical_label "+5V"
 		(shape input)
-		(at 121.92 92.71 180)
+		(at 113.03 101.6 180)
 		(fields_autoplaced yes)
 		(effects
@@
 	(hierarchical_label "+3.3V"
 		(shape output)
-		(at 179.07 95.25 0)
+		(at 170.18 104.14 0)
 		(fields_autoplaced yes)
 		(effects
@@
 	(hierarchical_label "+5V"
 		(shape input)
-		(at 142.24 97.79 180)
+		(at 133.35 106.68 180)
 		(fields_autoplaced yes)
 		(effects
@@
 	(symbol
 		(lib_id "power:GND")
-		(at 139.7 95.25 270)
+		(at 127 113.03 0)
 		(unit 1)
 		(exclude_from_sim no)
@@
 		(dnp no)
 		(property "Reference" "#PWR0902"
-			(at 133.35 95.25 0)
+			(at 127 119.38 0)
 			(effects
 				(font
@@
 		)
 		(property "Value" "GND"
-			(at 141.478 93.726 90)
+			(at 125.476 111.252 90)
 			(effects
 				(font
@@
 		)
 		(property "Footprint" ""
-			(at 139.7 95.25 0)
+			(at 127 113.03 0)
 			(effects
 				(font
@@
 		)
 		(property "Datasheet" ""
-			(at 139.7 95.25 0)
+			(at 127 113.03 0)
 			(effects
 				(font
@@
 		)
 		(property "Description" "Power symbol creates a global label with name \"GND\" , ground"
-			(at 139.7 95.25 0)
+			(at 127 113.03 0)
 			(effects
 				(font
@@
 	(symbol
 		(lib_id "Device:C_Small")
-		(at 172.72 101.6 0)
+		(at 163.83 110.49 0)
 		(unit 1)
 		(exclude_from_sim no)
@@
 		(fields_autoplaced yes)
 		(property "Reference" "C902"
-			(at 175.26 100.3362 0)
+			(at 166.37 109.2262 0)
 			(effects
 				(font
@@
 		)
 		(property "Value" "1uF"
-			(at 175.26 102.8762 0)
+			(at 166.37 111.7662 0)
 			(effects
 				(font
@@
 		)
 		(property "Footprint" ""
-			(at 172.72 101.6 0)
+			(at 163.83 110.49 0)
 			(effects
 				(font
@@
 		)
 		(property "Datasheet" "~"
-			(at 172.72 101.6 0)
+			(at 163.83 110.49 0)
 			(effects
 				(font
@@
 		)
 		(property "Description" "Unpolarized capacitor, small symbol"
-			(at 172.72 101.6 0)
+			(at 163.83 110.49 0)
 			(effects
 				(font
@@
 	(symbol
 		(lib_id "BU33SD5WG-TR:BU33SD5WG-TR")
-		(at 142.24 92.71 0)
+		(at 133.35 101.6 0)
 		(unit 1)
 		(exclude_from_sim no)
@@
 		(fields_autoplaced yes)
 		(property "Reference" "PS901"
-			(at 156.21 85.09 0)
+			(at 147.32 93.98 0)
 			(effects
 				(font
@@
 		)
 		(property "Value" "BU33SD5WG-TR"
-			(at 156.21 87.63 0)
+			(at 147.32 96.52 0)
 			(effects
 				(font
@@
 		)
 		(property "Footprint" "SOT95P280X125-5N"
-			(at 166.37 187.63 0)
+			(at 157.48 196.52 0)
 			(effects
 				(font
@@
 		)
 		(property "Datasheet" "https://componentsearchengine.com/Datasheets/1/BU33SD5WG-TR.pdf"
-			(at 166.37 287.63 0)
+			(at 157.48 296.52 0)
 			(effects
 				(font
@@
 		)
 		(property "Description" "LDO regulator,3.3V,0.5A,standby,SSOP5 ROHM BU33SD5WG-TR, LDO Voltage Regulator, 0.5A, 3.3 V +/-2%, 1.7  6 Vin, 5-Pin SSOP"
-			(at 142.24 92.71 0)
+			(at 133.35 101.6 0)
 			(effects
 				(font
@@
 		)
 		(property "Height" "1.25"
-			(at 166.37 487.63 0)
+			(at 157.48 496.52 0)
 			(effects
 				(font
@@
 		)
 		(property "Manufacturer_Name" "ROHM Semiconductor"
-			(at 166.37 587.63 0)
+			(at 157.48 596.52 0)
 			(effects
 				(font
@@
 		)
 		(property "Manufacturer_Part_Number" "BU33SD5WG-TR"
-			(at 166.37 687.63 0)
+			(at 157.48 696.52 0)
 			(effects
 				(font
@@
 		)
 		(property "Mouser Part Number" "755-BU33SD5WG-TR"
-			(at 166.37 787.63 0)
+			(at 157.48 796.52 0)
 			(effects
 				(font
@@
 		)
 		(property "Mouser Price/Stock" "https://www.mouser.co.uk/ProductDetail/ROHM-Semiconductor/BU33SD5WG-TR?qs=%2FKR40Cd6GUrQDzRkUEt69Q%3D%3D"
-			(at 166.37 887.63 0)
+			(at 157.48 896.52 0)
 			(effects
 				(font
@@
 		)
 		(property "Arrow Part Number" ""
-			(at 166.37 987.63 0)
+			(at 157.48 996.52 0)
 			(effects
 				(font
@@
 		)
 		(property "Arrow Price/Stock" ""
-			(at 166.37 1087.63 0)
+			(at 157.48 1096.52 0)
 			(effects
 				(font
@@
 	(symbol
 		(lib_id "Device:C_Small")
-		(at 128.27 95.25 0)
+		(at 119.38 104.14 0)
 		(unit 1)
 		(exclude_from_sim no)
@@
 		(fields_autoplaced yes)
 		(property "Reference" "C901"
-			(at 130.81 93.9862 0)
+			(at 121.92 102.8762 0)
 			(effects
 				(font
@@
 		)
 		(property "Value" "1uF"
-			(at 130.81 96.5262 0)
+			(at 121.92 105.4162 0)
 			(effects
 				(font
@@
 		)
 		(property "Footprint" ""
-			(at 128.27 95.25 0)
+			(at 119.38 104.14 0)
 			(effects
 				(font
@@
 		)
 		(property "Datasheet" "~"
-			(at 128.27 95.25 0)
+			(at 119.38 104.14 0)
 			(effects
 				(font
@@
 		)
 		(property "Description" "Unpolarized capacitor, small symbol"
-			(at 128.27 95.25 0)
+			(at 119.38 104.14 0)
 			(effects
 				(font
@@
 	(symbol
 		(lib_id "power:GND")
-		(at 128.27 97.79 0)
+		(at 119.38 106.68 0)
 		(unit 1)
 		(exclude_from_sim no)
@@
 		(fields_autoplaced yes)
 		(property "Reference" "#PWR0901"
-			(at 128.27 104.14 0)
+			(at 119.38 113.03 0)
 			(effects
 				(font
@@
 		)
 		(property "Value" "GND"
-			(at 128.27 102.87 0)
+			(at 119.38 111.76 0)
 			(effects
 				(font
@@
 		)
 		(property "Footprint" ""
-			(at 128.27 97.79 0)
+			(at 119.38 106.68 0)
 			(effects
 				(font
@@
 		)
 		(property "Datasheet" ""
-			(at 128.27 97.79 0)
+			(at 119.38 106.68 0)
 			(effects
 				(font
@@
 		)
 		(property "Description" "Power symbol creates a global label with name \"GND\" , ground"
-			(at 128.27 97.79 0)
+			(at 119.38 106.68 0)
 			(effects
 				(font
@@
 	(symbol
 		(lib_id "power:GND")
-		(at 172.72 106.68 0)
+		(at 163.83 115.57 0)
 		(unit 1)
 		(exclude_from_sim no)
@@
 		(fields_autoplaced yes)
 		(property "Reference" "#PWR0903"
-			(at 172.72 113.03 0)
+			(at 163.83 121.92 0)
 			(effects
 				(font
@@
 		)
 		(property "Value" "GND"
-			(at 172.72 111.76 0)
+			(at 163.83 120.65 0)
 			(effects
 				(font
@@
 		)
 		(property "Footprint" ""
-			(at 172.72 106.68 0)
+			(at 163.83 115.57 0)
 			(effects
 				(font
@@
 		)
 		(property "Datasheet" ""
-			(at 172.72 106.68 0)
+			(at 163.83 115.57 0)
 			(effects
 				(font
@@
 		)
 		(property "Description" "Power symbol creates a global label with name \"GND\" , ground"
-			(at 172.72 106.68 0)
-			(effects
-				(font
+			(at 163.83 115.57 0)
+			(effects
+				(font

Commit message: DERNIER MODIF Alim
Changed lines of the file:
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@@
 		)
 	)
-	(hierarchical_label "+5V"
-		(shape input)
-		(at 113.03 101.6 180)
+	(symbol
+		(lib_id "power:+3.3V")
+		(at 170.18 104.14 0)
+		(unit 1)
+		(exclude_from_sim no)
+		(in_bom yes)
+		(on_board yes)
+		(dnp no)
 		(fields_autoplaced yes)
-		(effects
-			(font
-				(size 1.27 1.27)
-			)
-			(justify right)
-		)
-	)
-	(hierarchical_label "+3.3V"
-		(shape output)
-		(at 170.18 104.14 0)
-		(fields_autoplaced yes)
-		(effects
-			(font
-				(size 1.27 1.27)
-			)
-			(justify left)
-		)
-	)
-	(hierarchical_label "+5V"
-		(shape input)
-		(at 133.35 106.68 180)
-		(fields_autoplaced yes)
-		(effects
-			(font
-				(size 1.27 1.27)
-			)
-			(justify right)
+		(property "Reference" "#PWR0905"
+			(at 170.18 107.95 0)
+			(effects
+				(font
+					(size 1.27 1.27)
+				)
+				(hide yes)
+			)
+		)
+		(property "Value" "+3.3V"
+			(at 170.18 99.06 0)
+			(effects
+				(font
+					(size 1.27 1.27)
+				)
+			)
+		)
+		(property "Footprint" ""
+			(at 170.18 104.14 0)
+			(effects
+				(font
+					(size 1.27 1.27)
+				)
+				(hide yes)
+			)
+		)
+		(property "Datasheet" ""
+			(at 170.18 104.14 0)
+			(effects
+				(font
+					(size 1.27 1.27)
+				)
+				(hide yes)
+			)
+		)
+		(property "Description" "Power symbol creates a global label with name \"+3.3V\""
+			(at 170.18 104.14 0)
+			(effects
+				(font
+					(size 1.27 1.27)
+				)
+				(hide yes)
+			)
+		)
+		(pin "1"
+		)
+		(instances
+			(project ""
+				(path "/37e0fdad-f3fd-48e0-8377-111662233a91/aef3d9b2-029f-4338-91be-d4af664a9426/a5848076-92cd-4e99-9706-01c7593ded28"
+					(reference "#PWR0905")
+					(unit 1)
+				)
+			)
 		)
 	)
@@
 				(path "/37e0fdad-f3fd-48e0-8377-111662233a91/aef3d9b2-029f-4338-91be-d4af664a9426/a5848076-92cd-4e99-9706-01c7593ded28"
 					(reference "#PWR0902")
+					(unit 1)
+				)
+			)
+		)
+	)
+	(symbol
+		(lib_id "power:+5V")
+		(at 133.35 106.68 90)
+		(unit 1)
+		(exclude_from_sim no)
+		(in_bom yes)
+		(on_board yes)
+		(dnp no)
+		(property "Reference" "#PWR0906"
+			(at 137.16 106.68 0)
+			(effects
+				(font
+					(size 1.27 1.27)
+				)
+				(hide yes)
+			)
+		)
+		(property "Value" "+5V"
+			(at 134.112 108.712 90)
+			(effects
+				(font
+					(size 1.27 1.27)
+				)
+				(justify left)
+			)
+		)
+		(property "Footprint" ""
+			(at 133.35 106.68 0)
+			(effects
+				(font
+					(size 1.27 1.27)
+				)
+				(hide yes)
+			)
+		)
+		(property "Datasheet" ""
+			(at 133.35 106.68 0)
+			(effects
+				(font
+					(size 1.27 1.27)
+				)
+				(hide yes)
+			)
+		)
+		(property "Description" "Power symbol creates a global label with name \"+5V\""
+			(at 133.35 106.68 0)
+			(effects
+				(font
+					(size 1.27 1.27)
+				)
+				(hide yes)
+			)
+		)
+		(pin "1"
+		)
+		(instances
+			(project "Pojet_V-NOM_KiCAD"
+				(path "/37e0fdad-f3fd-48e0-8377-111662233a91/aef3d9b2-029f-4338-91be-d4af664a9426/a5848076-92cd-4e99-9706-01c7593ded28"
+					(reference "#PWR0906")
 					(unit 1)
 				)
@@
 					(unit 1)
 				)
+			)
+		)
+	)
+	(symbol
+		(lib_id "power:+5V")
+		(at 113.03 101.6 0)
+		(unit 1)
+		(exclude_from_sim no)
+		(in_bom yes)
+		(on_board yes)
+		(dnp no)
+		(fields_autoplaced yes)
+		(property "Reference" "#PWR0904"
+			(at 113.03 105.41 0)
+			(effects
+				(font
+					(size 1.27 1.27)
+				)
+				(hide yes)
+			)
+		)
+		(property "Value" "+5V"
+			(at 113.03 96.52 0)
+			(effects
+				(font
+					(size 1.27 1.27)
+				)
+			)
+		)
+		(property "Footprint" ""
+			(at 113.03 101.6 0)
+			(effects
+				(font
+					(size 1.27 1.27)
+				)
+				(hide yes)
+			)
+		)
+		(property "Datasheet" ""
+			(at 113.03 101.6 0)
+			(effects
+				(font
+					(size 1.27 1.27)
+				)
+				(hide yes)
+			)
+		)
+		(property "Description" "Power symbol creates a global label with name \"+5V\""
+			(at 113.03 101.6 0)
+			(effects
+				(font
+					(size 1.27 1.27)
+				)
+				(hide yes)
+			)
+		)
+		(pin "1"
+		)
+		(instances
+			(project ""
+				(path "/37e0fdad-f3fd-48e0-8377-111662233a91/aef3d9b2-029f-4338-91be-d4af664a9426/a5848076-92cd-4e99-9706-01c7593ded28"
+					(reference "#PWR0904")
+					(unit 1)
+				)

Commit message: empreinte
Parts:
- C901, C902: footprint (none) -> Capacitor_SMD:C_0603_1608Metric
- PS901: footprint SOT95P280X125-5N -> Package_TO_SOT_SMD:SOT-23-5
Changed lines of the file:
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@@
 			)
 		)
-		(property "Footprint" ""
+		(property "Footprint" "Capacitor_SMD:C_0603_1608Metric"
 			(at 163.83 110.49 0)
 			(effects
@@
 			)
 		)
-		(property "Footprint" "SOT95P280X125-5N"
+		(property "Footprint" "Package_TO_SOT_SMD:SOT-23-5"
 			(at 157.48 196.52 0)
 			(effects
@@
 			)
 		)
-		(property "Footprint" ""
+		(property "Footprint" "Capacitor_SMD:C_0603_1608Metric"
 			(at 119.38 104.14 0)
 			(effects

Commit message: point de test et début de placement
Parts:
- added TP901, TP902: TestPoint, TestPoint:TestPoint_Pad_D1.0mm, symbol Connector:TestPoint
Connections:
- net +3.3V: now also TP901.1
- net +5V: now also TP902.1
Other:
- moved on the sheet: PS901
Changed lines of the file:
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@@
+	)
+	(junction
+		(at 171.45 104.14)
+		(diameter 0)
+		(color 0 0 0 0)
+	)
+	(junction
+		(at 127 101.6)
+		(diameter 0)
+		(color 0 0 0 0)
 	)
 	(junction
@@
 	(wire
 		(pts
-			(xy 127 104.14) (xy 133.35 104.14)
-		)
-		(stroke
-			(width 0)
-			(type default)
-		)
-	)
-	(wire
-		(pts
-			(xy 161.29 104.14) (xy 163.83 104.14)
-		)
-		(stroke
-			(width 0)
-			(type default)
-		)
-	)
-	(wire
-		(pts
-			(xy 113.03 101.6) (xy 119.38 101.6)
-		)
-		(stroke
-			(width 0)
-			(type default)
-		)
-	)
-	(wire
-		(pts
-			(xy 119.38 101.6) (xy 133.35 101.6)
-		)
-		(stroke
-			(width 0)
-			(type default)
-		)
-	)
-	(wire
-		(pts
-			(xy 163.83 104.14) (xy 170.18 104.14)
+			(xy 127 101.6) (xy 134.62 101.6)
+		)
+		(stroke
+			(width 0)
+			(type default)
+		)
+	)
+	(wire
+		(pts
+			(xy 134.62 106.68) (xy 133.35 106.68)
+		)
+		(stroke
+			(width 0)
+			(type default)
+		)
+	)
+	(wire
+		(pts
+			(xy 127 104.14) (xy 134.62 104.14)
+		)
+		(stroke
+			(width 0)
+			(type default)
+		)
+	)
+	(wire
+		(pts
+			(xy 127 99.06) (xy 127 101.6)
+		)
+		(stroke
+			(width 0)
+			(type default)
+		)
+	)
+	(wire
+		(pts
+			(xy 162.56 104.14) (xy 163.83 104.14)
+		)
+		(stroke
+			(width 0)
+			(type default)
+		)
+	)
+	(wire
+		(pts
+			(xy 171.45 104.14) (xy 185.42 104.14)
+		)
+		(stroke
+			(width 0)
+			(type default)
+		)
+	)
+	(wire
+		(pts
+			(xy 107.95 101.6) (xy 119.38 101.6)
+		)
+		(stroke
+			(width 0)
+			(type default)
+		)
+	)
+	(wire
+		(pts
+			(xy 119.38 101.6) (xy 127 101.6)
+		)
+		(stroke
+			(width 0)
+			(type default)
+		)
+	)
+	(wire
+		(pts
+			(xy 163.83 104.14) (xy 171.45 104.14)
 		)
 		(stroke
@@
 	(symbol
 		(lib_id "power:+3.3V")
-		(at 170.18 104.14 0)
+		(at 185.42 104.14 0)
 		(unit 1)
 		(exclude_from_sim no)
@@
 		(fields_autoplaced yes)
 		(property "Reference" "#PWR0905"
-			(at 170.18 107.95 0)
+			(at 185.42 107.95 0)
 			(effects
 				(font
@@
 		)
 		(property "Value" "+3.3V"
-			(at 170.18 99.06 0)
+			(at 185.42 99.06 0)
 			(effects
 				(font
@@
 		)
 		(property "Footprint" ""
-			(at 170.18 104.14 0)
+			(at 185.42 104.14 0)
 			(effects
 				(font
@@
 		)
 		(property "Datasheet" ""
-			(at 170.18 104.14 0)
+			(at 185.42 104.14 0)
 			(effects
 				(font
@@
 		)
 		(property "Description" "Power symbol creates a global label with name \"+3.3V\""
-			(at 170.18 104.14 0)
+			(at 185.42 104.14 0)
 			(effects
 				(font
@@
 				(path "/37e0fdad-f3fd-48e0-8377-111662233a91/aef3d9b2-029f-4338-91be-d4af664a9426/a5848076-92cd-4e99-9706-01c7593ded28"
 					(reference "#PWR0902")
+					(unit 1)
+				)
+			)
+		)
+	)
+	(symbol
+		(lib_id "Connector:TestPoint")
+		(at 171.45 104.14 0)
+		(unit 1)
+		(exclude_from_sim no)
+		(in_bom yes)
+		(on_board yes)
+		(dnp no)
+		(fields_autoplaced yes)
+		(property "Reference" "TP901"
+			(at 173.99 99.5679 0)
+			(effects
+				(font
+					(size 1.27 1.27)
+				)
+				(justify left)
+			)
+		)
+		(property "Value" "TestPoint"
+			(at 173.99 102.1079 0)
+			(effects
+				(font
+					(size 1.27 1.27)
+				)
+				(justify left)
+			)
+		)
+		(property "Footprint" "TestPoint:TestPoint_Pad_D1.0mm"
+			(at 176.53 104.14 0)
+			(effects
+				(font
+					(size 1.27 1.27)
+				)
+				(hide yes)
+			)
+		)
+		(property "Datasheet" "~"
+			(at 176.53 104.14 0)
+			(effects
+				(font
+					(size 1.27 1.27)
+				)
+				(hide yes)
+			)
+		)
+		(property "Description" "test point"
+			(at 171.45 104.14 0)
+			(effects
+				(font
+					(size 1.27 1.27)
+				)
+				(hide yes)
+			)
+		)
+		(pin "1"
+		)
+		(instances
+			(project ""
+				(path "/37e0fdad-f3fd-48e0-8377-111662233a91/aef3d9b2-029f-4338-91be-d4af664a9426/a5848076-92cd-4e99-9706-01c7593ded28"
+					(reference "TP901")
 					(unit 1)
 				)
@@
 	(symbol
 		(lib_id "BU33SD5WG-TR:BU33SD5WG-TR")
-		(at 133.35 101.6 0)
+		(at 134.62 101.6 0)
 		(unit 1)
 		(exclude_from_sim no)
@@
 		(fields_autoplaced yes)
 		(property "Reference" "PS901"
-			(at 147.32 93.98 0)
+			(at 148.59 93.98 0)
 			(effects
 				(font
@@
 		)
 		(property "Value" "BU33SD5WG-TR"
-			(at 147.32 96.52 0)
+			(at 148.59 96.52 0)
 			(effects
 				(font
@@
 		)
 		(property "Footprint" "Package_TO_SOT_SMD:SOT-23-5"
-			(at 157.48 196.52 0)
+			(at 158.75 196.52 0)
 			(effects
 				(font
@@
 		)
 		(property "Datasheet" "https://componentsearchengine.com/Datasheets/1/BU33SD5WG-TR.pdf"
-			(at 157.48 296.52 0)
+			(at 158.75 296.52 0)
 			(effects
 				(font
@@
 		)
 		(property "Description" "LDO regulator,3.3V,0.5A,standby,SSOP5 ROHM BU33SD5WG-TR, LDO Voltage Regulator, 0.5A, 3.3 V +/-2%, 1.7  6 Vin, 5-Pin SSOP"
-			(at 133.35 101.6 0)
+			(at 134.62 101.6 0)
 			(effects
 				(font
@@
 		)
 		(property "Height" "1.25"
-			(at 157.48 496.52 0)
+			(at 158.75 496.52 0)
 			(effects
 				(font
@@
 		)
 		(property "Manufacturer_Name" "ROHM Semiconductor"
-			(at 157.48 596.52 0)
+			(at 158.75 596.52 0)
 			(effects
 				(font
@@
 		)
 		(property "Manufacturer_Part_Number" "BU33SD5WG-TR"
-			(at 157.48 696.52 0)
+			(at 158.75 696.52 0)
 			(effects
 				(font
@@
 		)
 		(property "Mouser Part Number" "755-BU33SD5WG-TR"
-			(at 157.48 796.52 0)
+			(at 158.75 796.52 0)
 			(effects
 				(font
@@
 		)
 		(property "Mouser Price/Stock" "https://www.mouser.co.uk/ProductDetail/ROHM-Semiconductor/BU33SD5WG-TR?qs=%2FKR40Cd6GUrQDzRkUEt69Q%3D%3D"
-			(at 157.48 896.52 0)
+			(at 158.75 896.52 0)
 			(effects
 				(font
@@
 		)
 		(property "Arrow Part Number" ""
-			(at 157.48 996.52 0)
+			(at 158.75 996.52 0)
 			(effects
 				(font
@@
 		)
 		(property "Arrow Price/Stock" ""
-			(at 157.48 1096.52 0)
+			(at 158.75 1096.52 0)
 			(effects
 				(font
@@
 	(symbol
 		(lib_id "power:+5V")
-		(at 113.03 101.6 0)
+		(at 107.95 101.6 0)
 		(unit 1)
 		(exclude_from_sim no)
@@
 		(fields_autoplaced yes)
 		(property "Reference" "#PWR0904"
-			(at 113.03 105.41 0)
+			(at 107.95 105.41 0)
 			(effects
 				(font
@@
 		)
 		(property "Value" "+5V"
-			(at 113.03 96.52 0)
+			(at 107.95 96.52 0)
 			(effects
 				(font
@@
 		)
 		(property "Footprint" ""
-			(at 113.03 101.6 0)
+			(at 107.95 101.6 0)
 			(effects
 				(font
@@
 		)
 		(property "Datasheet" ""
-			(at 113.03 101.6 0)
+			(at 107.95 101.6 0)
 			(effects
 				(font
@@
 		)
 		(property "Description" "Power symbol creates a global label with name \"+5V\""
-			(at 113.03 101.6 0)
+			(at 107.95 101.6 0)
 			(effects
 				(font
@@
 					(unit 1)
 				)
+			)
+		)
+	)
+	(symbol
+		(lib_id "Connector:TestPoint")
+		(at 127 99.06 0)
+		(unit 1)
+		(exclude_from_sim no)
+		(in_bom yes)
+		(on_board yes)
+		(dnp no)
+		(fields_autoplaced yes)
+		(property "Reference" "TP902"
+			(at 129.54 94.4879 0)
+			(effects
+				(font
+					(size 1.27 1.27)
+				)
+				(justify left)
+			)
+		)
+		(property "Value" "TestPoint"
+			(at 129.54 97.0279 0)
+			(effects
+				(font
+					(size 1.27 1.27)
+				)
+				(justify left)
+			)
+		)
+		(property "Footprint" "TestPoint:TestPoint_Pad_D1.0mm"
+			(at 132.08 99.06 0)
+			(effects
+				(font
+					(size 1.27 1.27)
+				)
+				(hide yes)
+			)
+		)
+		(property "Datasheet" "~"
+			(at 132.08 99.06 0)
+			(effects
+				(font
+					(size 1.27 1.27)
+				)
+				(hide yes)
+			)
+		)
+		(property "Description" "test point"
+			(at 127 99.06 0)
+			(effects
+				(font
+					(size 1.27 1.27)
+				)
+				(hide yes)
+			)
+		)
+		(pin "1"
+		)
+		(instances
+			(project "Pojet_V-NOM_KiCAD"
+				(path "/37e0fdad-f3fd-48e0-8377-111662233a91/aef3d9b2-029f-4338-91be-d4af664a9426/a5848076-92cd-4e99-9706-01c7593ded28"
+					(reference "TP902")
+					(unit 1)
+				)
