File: Pojet_V-NOM_KiCAD/deplacement.kicad_sch (KiCad schematic)
At the start: 8 parts, among them J301 Conn_01x06, J302 Conn_01x06, U301 ZXBM5210-SP, U302 ZXBM5210-SP

Commit message: rajout capteur
capteur de bordure
Connections:
- net GND: now also J301.2 (Pin_2), J302.2 (Pin_2)
- net PB6: now also J302.4 (Pin_4)
- net at J302.1 (Pin_1): now also U302.7 (OUT2); no longer U302.1 (OUT1)
- net PB5: now reaches J302.3 (Pin_3)
- net +5V: now reaches J302.5 (Pin_5)
- net +5V: now also J301.5 (Pin_5)
- net at J302.6 (Pin_6): now also U302.1 (OUT1); no longer U302.7 (OUT2)
- net at U301.1 (OUT1): now also J301.6 (Pin_6); no longer J301.1 (Pin_1)
- net at U301.7 (OUT2): now also J301.1 (Pin_1); no longer J301.6 (Pin_6)
- net PA5: now reaches J301.3 (Pin_3)
- net PA6: now reaches J301.4 (Pin_4)

Commit message: MAJ Valerian
MAJ Valerian
Connections:
- net PA0 renamed FWD1
- net PA1 renamed REV1
- net PA5 renamed Encoder B phase 1 
- net PA6 renamed Encoder A phase 1 
- net PA8 renamed VREF1
- net PB0 renamed FWD2
- net PB1 renamed REV2
- net PB5 renamed Encoder B phase 2
- net PB6 renamed VREF2
- net VREF2: no longer J302.4 (Pin_4)
- new net Encoder A phase 2: J302.4 (Pin_4)
Changed lines of the file:
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@@
 	(wire
 		(pts
-			(xy 220.98 72.39) (xy 220.98 86.36)
+			(xy 219.71 77.47) (xy 219.71 78.74)
 		)
 		(stroke
@@
 	(wire
 		(pts
+			(xy 228.6 77.47) (xy 228.6 86.36)
+		)
+		(stroke
+			(width 0)
+			(type default)
+		)
+	)
+	(wire
+		(pts
 			(xy 77.47 33.02) (xy 81.28 33.02)
 		)
@@
 	(wire
 		(pts
+			(xy 220.98 78.74) (xy 220.98 86.36)
+		)
+		(stroke
+			(width 0)
+			(type default)
+		)
+	)
+	(wire
+		(pts
 			(xy 104.14 71.12) (xy 104.14 82.55)
 		)
@@
 	(wire
 		(pts
-			(xy 228.6 72.39) (xy 228.6 86.36)
-		)
-		(stroke
-			(width 0)
-			(type default)
-		)
-	)
-	(hierarchical_label "PA5"
+			(xy 219.71 78.74) (xy 220.98 78.74)
+		)
+		(stroke
+			(width 0)
+			(type default)
+		)
+	)
+	(hierarchical_label "Encoder B phase 1 "
 		(shape passive)
 		(at 109.22 77.47 90)
@@
 		)
 	)
-	(hierarchical_label "PA0"
+	(hierarchical_label "FWD1"
 		(shape passive)
 		(at 69.85 52.07 180)
@@
 		)
 	)
-	(hierarchical_label "PB0"
+	(hierarchical_label "FWD2"
 		(shape passive)
 		(at 186.69 55.88 180)
@@
 		)
 	)
-	(hierarchical_label "PA8"
+	(hierarchical_label "VREF1"
 		(shape passive)
 		(at 39.37 27.94 90)
@@
 		)
 	)
-	(hierarchical_label "PB5"
+	(hierarchical_label "Encoder B phase 2"
 		(shape passive)
 		(at 226.06 80.01 90)
@@
 		)
 	)
-	(hierarchical_label "PA1"
+	(hierarchical_label "REV1"
 		(shape passive)
 		(at 69.85 54.61 180)
@@
 		)
 	)
-	(hierarchical_label "PA6"
+	(hierarchical_label "Encoder A phase 1 "
 		(shape passive)
 		(at 106.68 77.47 90)
@@
 		)
 	)
-	(hierarchical_label "PB6"
+	(hierarchical_label "VREF2"
 		(shape passive)
 		(at 166.37 33.02 90)
@@
 		)
 	)
-	(hierarchical_label "PB6"
+	(hierarchical_label "Encoder A phase 2"
 		(shape passive)
 		(at 223.52 80.01 90)
@@
 		)
 	)
-	(hierarchical_label "PB1"
+	(hierarchical_label "REV2"
 		(shape passive)
 		(at 186.69 58.42 180)
@@
 		(on_board yes)
 		(dnp no)
-		(fields_autoplaced yes)
 		(property "Reference" "#PWR0308"
 			(at 104.14 74.93 0)
@@
 		)
 		(property "Value" "+5V"
-			(at 104.14 66.04 0)
+			(at 103.124 65.786 0)
 			(effects
 				(font
@@
 	(symbol
 		(lib_id "power:GND")
-		(at 228.6 72.39 180)
+		(at 228.6 77.47 180)
 		(unit 1)
 		(exclude_from_sim no)
@@
 		(on_board yes)
 		(dnp no)
-		(fields_autoplaced yes)
 		(property "Reference" "#PWR0310"
-			(at 228.6 66.04 0)
+			(at 228.6 71.12 0)
 			(effects
 				(font
@@
 		)
 		(property "Value" "GND"
-			(at 228.6 67.31 0)
+			(at 229.108 72.39 0)
 			(effects
 				(font
@@
 		)
 		(property "Footprint" ""
-			(at 228.6 72.39 0)
+			(at 228.6 77.47 0)
 			(effects
 				(font
@@
 		)
 		(property "Datasheet" ""
-			(at 228.6 72.39 0)
+			(at 228.6 77.47 0)
 			(effects
 				(font
@@
 		)
 		(property "Description" "Power symbol creates a global label with name \"GND\" , ground"
-			(at 228.6 72.39 0)
+			(at 228.6 77.47 0)
 			(effects
 				(font
@@
 	(symbol
 		(lib_id "power:+5V")
-		(at 220.98 72.39 0)
+		(at 219.71 77.47 0)
 		(unit 1)
 		(exclude_from_sim no)
@@
 		(dnp no)
 		(property "Reference" "#PWR0309"
-			(at 220.98 76.2 0)
+			(at 219.71 81.28 0)
 			(effects
 				(font
@@
 		)
 		(property "Value" "+5V"
-			(at 220.726 67.818 0)
+			(at 219.456 72.898 0)
 			(effects
 				(font
@@
 		)
 		(property "Footprint" ""
-			(at 220.98 72.39 0)
+			(at 219.71 77.47 0)
 			(effects
 				(font
@@
 		)
 		(property "Datasheet" ""
-			(at 220.98 72.39 0)
+			(at 219.71 77.47 0)
 			(effects
 				(font
@@
 		)
 		(property "Description" "Power symbol creates a global label with name \"+5V\""
-			(at 220.98 72.39 0)
+			(at 219.71 77.47 0)
 			(effects
 				(font
@@
 		(on_board yes)
 		(dnp no)
-		(fields_autoplaced yes)
 		(property "Reference" "#PWR0307"
 			(at 111.76 64.77 0)
@@
 		)
 		(property "Value" "GND"
-			(at 111.76 66.04 0)
-			(effects
-				(font
+			(at 112.268 66.04 0)
+			(effects
+				(font

Commit message: Maj Deplacement
Maj Deplacement
Parts:
- removed C301, C303: 1uF, Capacitor_SMD:C_0402_1005Metric, symbol Device:C_Small
- removed C302, C304: 10uF, Capacitor_SMD:C_0402_1005Metric, symbol Device:C_Small
- removed U301, U302: ZXBM5210-SP, Package_SO:Diodes_SO-8EP, symbol Driver_Motor:ZXBM5210-SP
Connections:
- net Driver_Motor1/OUT1: now reaches J301.6 (Pin_6)
- net Driver_Motor1/OUT2: now reaches J301.1 (Pin_1)
- net Driver_Motor2/OUT2: now reaches J302.1 (Pin_1)
- net Driver_Motor2/OUT1: now reaches J302.6 (Pin_6)
- net Encoder A phase 1  renamed Encoder A phase 1
- net Encoder B phase 1  renamed Encoder B phase 1
Other:
- added sheet Driver_Motor1 (Driver_Moter.kicad_sch)
- added sheet Driver_Motor2 (Driver_Moter.kicad_sch)
- note added: "Driver motor 1"
- note added: "Driver motor 2"

Commit message: Maj
Maj lidar et regualteur
Connections:
- net +5V is gone; now on net +7.2V: J301.5 (Pin_5), J302.5 (Pin_5)
Changed lines of the file:
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@@
+		)
+	)
+	(hierarchical_label "+7.2V"
+		(shape input)
+		(at 130.81 90.17 180)
+		(fields_autoplaced yes)
+		(effects
+			(font
+				(size 1.27 1.27)
+			)
+			(justify right)
 		)
 	)
@@
 		(shape output)
 		(at 130.81 85.09 180)
+		(fields_autoplaced yes)
+		(effects
+			(font
+				(size 1.27 1.27)
+			)
+			(justify right)
+		)
+	)
+	(hierarchical_label "+7.2V"
+		(shape input)
+		(at 265.43 88.9 180)
 		(fields_autoplaced yes)
 		(effects
@@
 					(unit 1)
 				)
-			)
-		)
-	)
-	(symbol
-		(lib_id "power:+5V")
-		(at 265.43 88.9 90)
-		(unit 1)
-		(exclude_from_sim no)
-		(in_bom yes)
-		(on_board yes)
-		(dnp no)
-		(property "Reference" "#PWR0304"
-			(at 269.24 88.9 0)
-			(effects
-				(font
-					(size 1.27 1.27)
-				)
-				(hide yes)
-			)
-		)
-		(property "Value" "+5V"
-			(at 260.096 89.916 0)
-			(effects
-				(font
-					(size 1.27 1.27)
-				)
-			)
-		)
-		(property "Footprint" ""
-			(at 265.43 88.9 0)
-			(effects
-				(font
-					(size 1.27 1.27)
-				)
-				(hide yes)
-			)
-		)
-		(property "Datasheet" ""
-			(at 265.43 88.9 0)
-			(effects
-				(font
-					(size 1.27 1.27)
-				)
-				(hide yes)
-			)
-		)
-		(property "Description" "Power symbol creates a global label with name \"+5V\""
-			(at 265.43 88.9 0)
-			(effects
-				(font
-					(size 1.27 1.27)
-				)
-				(hide yes)
-			)
-		)
-		(pin "1"
-		)
-		(instances
-			(project "Pojet_V-NOM_KiCAD"
-				(path "/37e0fdad-f3fd-48e0-8377-111662233a91/778527cd-4ba2-44a7-9be0-e348ce68e304"
-					(reference "#PWR0304")
-					(unit 1)
-				)
-			)
-		)
-	)
-	(symbol
-		(lib_id "power:+5V")
-		(at 130.81 90.17 90)
-		(unit 1)
-		(exclude_from_sim no)
-		(in_bom yes)
-		(on_board yes)
-		(dnp no)
-		(property "Reference" "#PWR0302"
-			(at 134.62 90.17 0)
-			(effects
-				(font
-					(size 1.27 1.27)
-				)
-				(hide yes)
-			)
-		)
-		(property "Value" "+5V"
-			(at 125.476 91.186 0)
-			(effects
-				(font
-					(size 1.27 1.27)
-				)
-			)
-		)
-		(property "Footprint" ""
-			(at 130.81 90.17 0)
-			(effects
-				(font
-					(size 1.27 1.27)
-				)
-				(hide yes)
-			)
-		)
-		(property "Datasheet" ""
-			(at 130.81 90.17 0)
-			(effects
-				(font
-					(size 1.27 1.27)
-				)
-				(hide yes)
-			)
-		)
-		(property "Description" "Power symbol creates a global label with name \"+5V\""
-			(at 130.81 90.17 0)
-			(effects
-				(font
-					(size 1.27 1.27)
-				)
-				(hide yes)
-			)
-		)
-		(pin "1"
-		)
-		(instances
-			(project "Pojet_V-NOM_KiCAD"
-				(path "/37e0fdad-f3fd-48e0-8377-111662233a91/778527cd-4ba2-44a7-9be0-e348ce68e304"
-					(reference "#PWR0302")
-					(unit 1)
-				)

Commit message: DERNIER MODIF Alim
Connections:
- net +7.2V renamed +BATT
Other:
- sheet Driver_Motor1 ports: added none; removed +7.2V
- sheet Driver_Motor2 ports: added none; removed +7.2V
Changed lines of the file:
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@@
-	(wire
-		(pts
-			(xy 63.5 54.61) (xy 63.5 60.96)
-		)
-		(stroke
-			(width 0)
-			(type default)
-		)
-	)
 	(wire
 		(pts
@@
 		)
 	)
-	(wire
-		(pts
-			(xy 208.28 55.88) (xy 208.28 60.96)
-		)
-		(stroke
-			(width 0)
-			(type default)
-		)
-	)
 	(polyline
 		(pts
@@
 		)
 	)
-	(hierarchical_label "+7.2V"
-		(shape input)
-		(at 130.81 90.17 180)
-		(fields_autoplaced yes)
-		(effects
-			(font
-				(size 1.27 1.27)
-			)
-			(justify right)
-		)
-	)
 	(hierarchical_label "Encoder A phase 1"
 		(shape output)
@@
 		)
 	)
-	(hierarchical_label "+7.2V"
-		(shape input)
-		(at 265.43 88.9 180)
-		(fields_autoplaced yes)
-		(effects
-			(font
-				(size 1.27 1.27)
-			)
-			(justify right)
-		)
-	)
 	(hierarchical_label "VREF2"
 		(shape input)
@@
 		)
 	)
-	(hierarchical_label "+7.2V"
-		(shape input)
-		(at 208.28 55.88 90)
-		(fields_autoplaced yes)
-		(effects
-			(font
-				(size 1.27 1.27)
-			)
-			(justify left)
-		)
-	)
 	(hierarchical_label "FWD2"
 		(shape input)
@@
 			)
 			(justify right)
-		)
-	)
-	(hierarchical_label "+7.2V"
-		(shape input)
-		(at 63.5 54.61 90)
-		(fields_autoplaced yes)
-		(effects
-			(font
-				(size 1.27 1.27)
-			)
-			(justify left)
 		)
 	)
@@
 	)
 	(symbol
+		(lib_id "power:+BATT")
+		(at 265.43 88.9 90)
+		(unit 1)
+		(exclude_from_sim no)
+		(in_bom yes)
+		(on_board yes)
+		(dnp no)
+		(fields_autoplaced yes)
+		(property "Reference" "#PWR0304"
+			(at 269.24 88.9 0)
+			(effects
+				(font
+					(size 1.27 1.27)
+				)
+				(hide yes)
+			)
+		)
+		(property "Value" "+BATT"
+			(at 261.62 88.8999 90)
+			(effects
+				(font
+					(size 1.27 1.27)
+				)
+				(justify left)
+			)
+		)
+		(property "Footprint" ""
+			(at 265.43 88.9 0)
+			(effects
+				(font
+					(size 1.27 1.27)
+				)
+				(hide yes)
+			)
+		)
+		(property "Datasheet" ""
+			(at 265.43 88.9 0)
+			(effects
+				(font
+					(size 1.27 1.27)
+				)
+				(hide yes)
+			)
+		)
+		(property "Description" "Power symbol creates a global label with name \"+BATT\""
+			(at 265.43 88.9 0)
+			(effects
+				(font
+					(size 1.27 1.27)
+				)
+				(hide yes)
+			)
+		)
+		(pin "1"
+		)
+		(instances
+			(project "Pojet_V-NOM_KiCAD"
+				(path "/37e0fdad-f3fd-48e0-8377-111662233a91/778527cd-4ba2-44a7-9be0-e348ce68e304"
+					(reference "#PWR0304")
+					(unit 1)
+				)
+			)
+		)
+	)
+	(symbol
+		(lib_id "power:+BATT")
+		(at 130.81 90.17 90)
+		(unit 1)
+		(exclude_from_sim no)
+		(in_bom yes)
+		(on_board yes)
+		(dnp no)
+		(fields_autoplaced yes)
+		(property "Reference" "#PWR0302"
+			(at 134.62 90.17 0)
+			(effects
+				(font
+					(size 1.27 1.27)
+				)
+				(hide yes)
+			)
+		)
+		(property "Value" "+BATT"
+			(at 127 90.1699 90)
+			(effects
+				(font
+					(size 1.27 1.27)
+				)
+				(justify left)
+			)
+		)
+		(property "Footprint" ""
+			(at 130.81 90.17 0)
+			(effects
+				(font
+					(size 1.27 1.27)
+				)
+				(hide yes)
+			)
+		)
+		(property "Datasheet" ""
+			(at 130.81 90.17 0)
+			(effects
+				(font
+					(size 1.27 1.27)
+				)
+				(hide yes)
+			)
+		)
+		(property "Description" "Power symbol creates a global label with name \"+BATT\""
+			(at 130.81 90.17 0)
+			(effects
+				(font
+					(size 1.27 1.27)
+				)
+				(hide yes)
+			)
+		)
+		(pin "1"
+		)
+		(instances
+			(project ""
+				(path "/37e0fdad-f3fd-48e0-8377-111662233a91/778527cd-4ba2-44a7-9be0-e348ce68e304"
+					(reference "#PWR0302")
+					(unit 1)
+				)
+			)
+		)
+	)
+	(symbol
 		(lib_id "power:GND")
 		(at 265.43 81.28 270)
@@
 			)
 		)
-		(pin "+7.2V" input
-			(at 63.5 60.96 90)
-			(effects
-				(font
-					(size 1.27 1.27)
-				)
-				(justify right)
-			)
-		)
 		(pin "OUT1" output
 			(at 96.52 92.71 0)
@@
 			)
 		)
-		(pin "+7.2V" input
-			(at 208.28 60.96 90)
-			(effects
-				(font
-					(size 1.27 1.27)
-				)
-				(justify right)
-			)
-		)

Commit message: Correction des erreurs évidentes
Changements avant vérification des erreurs :
- Désallocation du pin BTN_RESET
- Réarrangement de certaines sources pour cohérence avec tous les
schémas éléctriques
Other:
- note added: "Driver moteur 1"
- note added: "Driver moteur 2"
- note removed: "Driver motor 1"
- note removed: "Driver motor 2"
- moved on the sheet: J301, J302
Changed lines of the file:
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@@
 	(wire
 		(pts
-			(xy 22.86 78.74) (xy 30.48 78.74)
+			(xy 30.48 81.28) (xy 38.1 81.28)
 		)
 		(stroke
@@
 	(wire
 		(pts
-			(xy 96.52 92.71) (xy 130.81 92.71)
+			(xy 104.14 95.25) (xy 128.27 95.25)
 		)
 		(stroke
@@
 	(wire
 		(pts
-			(xy 166.37 90.17) (xy 177.8 90.17)
+			(xy 165.1 93.98) (xy 176.53 93.98)
 		)
 		(stroke
@@
 	(wire
 		(pts
-			(xy 238.76 78.74) (xy 265.43 78.74)
+			(xy 237.49 82.55) (xy 264.16 82.55)
 		)
 		(stroke
@@
 	(wire
 		(pts
-			(xy 238.76 91.44) (xy 265.43 91.44)
+			(xy 237.49 95.25) (xy 264.16 95.25)
 		)
 		(stroke
@@
 	(wire
 		(pts
-			(xy 96.52 80.01) (xy 130.81 80.01)
+			(xy 104.14 82.55) (xy 128.27 82.55)
 		)
 		(stroke
@@
 	(wire
 		(pts
-			(xy 22.86 91.44) (xy 30.48 91.44)
+			(xy 30.48 93.98) (xy 38.1 93.98)
 		)
 		(stroke
@@
 	(wire
 		(pts
-			(xy 167.64 76.2) (xy 177.8 76.2)
+			(xy 166.37 80.01) (xy 176.53 80.01)
 		)
 		(stroke
@@
 		)
 	)
-	(text "Driver motor 2\n"
+	(text "Driver moteur 2\n"
 		(exclude_from_sim no)
 		(at 169.672 18.034 0)
@@
 		)
 	)
-	(text "Driver motor 1\n"
+	(text "Driver moteur 1\n"
 		(exclude_from_sim no)
 		(at 36.322 18.288 0)
@@
 	(hierarchical_label "Encoder A phase 1"
 		(shape output)
-		(at 130.81 87.63 180)
+		(at 128.27 90.17 180)
 		(fields_autoplaced yes)
 		(effects
@@
 	(hierarchical_label "VREF1"
 		(shape input)
-		(at 22.86 78.74 180)
+		(at 30.48 81.28 180)
 		(fields_autoplaced yes)
 		(effects
@@
 	(hierarchical_label "FWD1"
 		(shape input)
-		(at 22.86 91.44 180)
+		(at 30.48 93.98 180)
 		(fields_autoplaced yes)
 		(effects
@@
 	(hierarchical_label "Encoder B phase 2"
 		(shape output)
-		(at 265.43 83.82 180)
+		(at 264.16 87.63 180)
 		(fields_autoplaced yes)
 		(effects
@@
 	(hierarchical_label "Encoder A phase 2"
 		(shape output)
-		(at 265.43 86.36 180)
+		(at 264.16 90.17 180)
 		(fields_autoplaced yes)
 		(effects
@@
 	(hierarchical_label "Encoder B phase 1"
 		(shape output)
-		(at 130.81 85.09 180)
+		(at 128.27 87.63 180)
 		(fields_autoplaced yes)
 		(effects
@@
 	(hierarchical_label "VREF2"
 		(shape input)
-		(at 167.64 76.2 180)
+		(at 166.37 80.01 180)
 		(fields_autoplaced yes)
 		(effects
@@
 	(hierarchical_label "FWD2"
 		(shape input)
-		(at 166.37 90.17 180)
+		(at 165.1 93.98 180)
 		(fields_autoplaced yes)
 		(effects
@@
 	(symbol
 		(lib_id "Connector_Generic:Conn_01x06")
-		(at 135.89 85.09 0)
+		(at 133.35 87.63 0)
 		(unit 1)
 		(exclude_from_sim no)
@@
 		(fields_autoplaced yes)
 		(property "Reference" "J301"
-			(at 138.43 85.0899 0)
+			(at 135.89 87.6299 0)
 			(effects
 				(font
@@
 		)
 		(property "Value" "Conn_01x06"
-			(at 138.43 87.6299 0)
+			(at 135.89 90.1699 0)
 			(effects
 				(font
@@
 		)
 		(property "Footprint" "Connector_JST:JST_XH_S6B-XH-A_1x06_P2.50mm_Horizontal"
-			(at 135.89 85.09 0)
+			(at 133.35 87.63 0)
 			(effects
 				(font
@@
 		)
 		(property "Datasheet" "~"
-			(at 135.89 85.09 0)
+			(at 133.35 87.63 0)
 			(effects
 				(font
@@
 		)
 		(property "Description" "Generic connector, single row, 01x06, script generated (kicad-library-utils/schlib/autogen/connector/)"
-			(at 135.89 85.09 0)
+			(at 133.35 87.63 0)
 			(effects
 				(font
@@
 	(symbol
 		(lib_id "Connector_Generic:Conn_01x06")
-		(at 270.51 83.82 0)
+		(at 269.24 87.63 0)
 		(unit 1)
 		(exclude_from_sim no)
@@
 		(fields_autoplaced yes)
 		(property "Reference" "J302"
-			(at 273.05 83.8199 0)
+			(at 271.78 87.6299 0)
 			(effects
 				(font
@@
 		)
 		(property "Value" "Conn_01x06"
-			(at 273.05 86.3599 0)
+			(at 271.78 90.1699 0)
 			(effects
 				(font
@@
 		)
 		(property "Footprint" "Connector_JST:JST_XH_S6B-XH-A_1x06_P2.50mm_Horizontal"
-			(at 270.51 83.82 0)
+			(at 269.24 87.63 0)
 			(effects
 				(font
@@
 		)
 		(property "Datasheet" "~"
-			(at 270.51 83.82 0)
+			(at 269.24 87.63 0)
 			(effects
 				(font
@@
 		)
 		(property "Description" "Generic connector, single row, 01x06, script generated (kicad-library-utils/schlib/autogen/connector/)"
-			(at 270.51 83.82 0)
+			(at 269.24 87.63 0)
 			(effects
 				(font
@@
 	(symbol
 		(lib_id "power:+BATT")
-		(at 265.43 88.9 90)
+		(at 264.16 92.71 90)
 		(unit 1)
 		(exclude_from_sim no)
@@
 		(fields_autoplaced yes)
 		(property "Reference" "#PWR0304"
-			(at 269.24 88.9 0)
+			(at 267.97 92.71 0)
 			(effects
 				(font
@@
 		)
 		(property "Value" "+BATT"
-			(at 261.62 88.8999 90)
+			(at 260.35 92.7099 90)
 			(effects
 				(font
@@
 		)
 		(property "Footprint" ""
-			(at 265.43 88.9 0)
+			(at 264.16 92.71 0)
 			(effects
 				(font
@@
 		)
 		(property "Datasheet" ""
-			(at 265.43 88.9 0)
+			(at 264.16 92.71 0)
 			(effects
 				(font
@@
 		)
 		(property "Description" "Power symbol creates a global label with name \"+BATT\""
-			(at 265.43 88.9 0)
+			(at 264.16 92.71 0)
 			(effects
 				(font
@@
 	(symbol
 		(lib_id "power:+BATT")
-		(at 130.81 90.17 90)
+		(at 128.27 92.71 90)
 		(unit 1)
 		(exclude_from_sim no)
@@
 		(fields_autoplaced yes)
 		(property "Reference" "#PWR0302"
-			(at 134.62 90.17 0)
+			(at 132.08 92.71 0)
 			(effects
 				(font
@@
 		)
 		(property "Value" "+BATT"
-			(at 127 90.1699 90)
+			(at 124.46 92.7099 90)
 			(effects
 				(font
@@
 		)
 		(property "Footprint" ""
-			(at 130.81 90.17 0)
+			(at 128.27 92.71 0)
 			(effects
 				(font
@@
 		)
 		(property "Datasheet" ""
-			(at 130.81 90.17 0)
+			(at 128.27 92.71 0)
 			(effects
 				(font
@@
 		)
 		(property "Description" "Power symbol creates a global label with name \"+BATT\""
-			(at 130.81 90.17 0)
+			(at 128.27 92.71 0)
 			(effects
 				(font
@@
 	(symbol
 		(lib_id "power:GND")
-		(at 265.43 81.28 270)
+		(at 264.16 85.09 270)
 		(unit 1)
 		(exclude_from_sim no)
@@
 		(dnp no)
 		(property "Reference" "#PWR0303"
-			(at 259.08 81.28 0)
+			(at 257.81 85.09 0)
 			(effects
 				(font
@@
 		)
 		(property "Value" "GND"
-			(at 260.35 80.772 0)
+			(at 259.08 84.582 0)
 			(effects
 				(font
@@
 		)
 		(property "Footprint" ""
-			(at 265.43 81.28 0)
+			(at 264.16 85.09 0)
 			(effects
 				(font
@@
 		)
 		(property "Datasheet" ""
-			(at 265.43 81.28 0)
+			(at 264.16 85.09 0)
 			(effects
 				(font
@@
 		)
 		(property "Description" "Power symbol creates a global label with name \"GND\" , ground"
-			(at 265.43 81.28 0)
+			(at 264.16 85.09 0)
 			(effects
 				(font
@@
 	(symbol
 		(lib_id "power:GND")
-		(at 130.81 82.55 270)
+		(at 128.27 85.09 270)
 		(unit 1)
 		(exclude_from_sim no)
@@
 		(dnp no)
 		(property "Reference" "#PWR0301"
-			(at 124.46 82.55 0)
+			(at 121.92 85.09 0)
 			(effects
 				(font
@@
 		)
 		(property "Value" "GND"
-			(at 125.73 82.042 0)
+			(at 123.19 84.582 0)
 			(effects
 				(font
@@
 		)
 		(property "Footprint" ""
-			(at 130.81 82.55 0)
+			(at 128.27 85.09 0)
 			(effects
 				(font
@@
 		)
 		(property "Datasheet" ""
-			(at 130.81 82.55 0)
+			(at 128.27 85.09 0)
 			(effects
 				(font
@@
 		)
 		(property "Description" "Power symbol creates a global label with name \"GND\" , ground"
-			(at 130.81 82.55 0)
+			(at 128.27 85.09 0)
 			(effects
 				(font
@@
 	)
 	(sheet
-		(at 30.48 60.96)
+		(at 38.1 63.5)
 		(size 66.04 50.8)
 		(fields_autoplaced yes)
@@
 		)
 		(property "Sheetname" "Driver_Motor1"
-			(at 30.48 60.2484 0)
+			(at 38.1 62.7884 0)
 			(effects
 				(font
@@
 		)
 		(property "Sheetfile" "Driver_Moter.kicad_sch"
-			(at 30.48 112.3446 0)
+			(at 38.1 114.8846 0)
 			(effects
 				(font
@@
 		)
 		(pin "OUT1" output
-			(at 96.52 92.71 0)
+			(at 104.14 95.25 0)
 			(effects
 				(font
@@
 		)
 		(pin "OUT2" output
-			(at 96.52 80.01 0)
+			(at 104.14 82.55 0)
 			(effects
 				(font
@@
 		)
 		(pin "REV" input
-			(at 30.48 78.74 180)
+			(at 38.1 81.28 180)
 			(effects
 				(font
@@
 		)
 		(pin "FWD" input
-			(at 30.48 91.44 180)
+			(at 38.1 93.98 180)
 			(effects
 				(font
@@
 	)
 	(sheet
-		(at 177.8 60.96)
+		(at 176.53 64.77)
 		(size 60.96 46.99)
 		(fields_autoplaced yes)
@@
 		)
 		(property "Sheetname" "Driver_Motor2"
-			(at 177.8 60.2484 0)
+			(at 176.53 64.0584 0)
 			(effects
 				(font
@@
 		)
 		(property "Sheetfile" "Driver_Moter.kicad_sch"
-			(at 177.8 108.5346 0)
+			(at 176.53 112.3446 0)
 			(effects
 				(font
@@
 		)
 		(pin "OUT1" output
-			(at 238.76 91.44 0)
+			(at 237.49 95.25 0)
 			(effects
 				(font
@@
 		)
 		(pin "OUT2" output
-			(at 238.76 78.74 0)
+			(at 237.49 82.55 0)
 			(effects
 				(font
@@
 		)
 		(pin "REV" input
-			(at 177.8 76.2 180)
+			(at 176.53 80.01 180)
 			(effects
 				(font
@@
 		)
 		(pin "FWD" input
-			(at 177.8 90.17 180)
-			(effects
-				(font
+			(at 176.53 93.98 180)
+			(effects
+				(font

Commit message: point de test et début de placement
Parts:
- added TP301, TP302, TP303, TP304: TestPoint, TestPoint:TestPoint_Pad_D1.0mm, symbol Connector:TestPoint
Connections:
- net Encoder A phase 1: now also TP302.1
- net Encoder A phase 2: now also TP304.1
- net Encoder B phase 1: now also TP301.1
- net Encoder B phase 2: now also TP303.1
Other:
- moved on the sheet: J301

Commit message: placement maj
Parts:
- removed TP301, TP302, TP303, TP304: TestPoint, TestPoint:TestPoint_Pad_D1.0mm, symbol Connector:TestPoint
Connections:
- net +BATT renamed +3.3V
