File: Pojet_V-NOM_KiCAD/deplacement.kicad_sch (KiCad schematic)
At the start: 2 parts, among them J301 Conn_01x06, J302 Conn_01x06

Commit message: grande partie de routage
Changed lines of the file:
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@@
 	(paper "A4")
-	(junction
-		(at 132.08 90.17)
-		(diameter 0)
-		(color 0 0 0 0)
-	)
 	(junction
 		(at 121.92 92.71)
@@
 	(wire
 		(pts
-			(xy 132.08 90.17) (xy 113.03 90.17)
-		)
-		(stroke
-			(width 0)
-			(type default)
-		)
-	)
-	(wire
-		(pts
-			(xy 137.16 90.17) (xy 132.08 90.17)
+			(xy 113.03 90.17) (xy 137.16 90.17)
 		)
 		(stroke
@@
 		)
 		(stroke
-			(width 0)
-			(type default)
-		)
-	)
-	(wire
-		(pts
-			(xy 132.08 96.52) (xy 132.08 90.17)
-		)
-		(stroke
