File: Pojet_V-NOM_KiCAD/interface_utilisateur.kicad_sch (KiCad schematic)
At the start: 6 parts, among them J1 Conn_ST_STDC14, J2 Conn_01x02

Commit message: Corrections sonde et switch
Connections:
- net SWO: no longer names the net of J1.8 (JTDO/SWO)
- no-connect marks 2 -> 3
Changed lines of the file:
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@@
+	)
+	(no_connect
+		(at 57.15 100.33)
 	)
 	(no_connect
@@
 		)
 	)
-	(hierarchical_label "SWO"
-		(shape output)
-		(at 57.15 100.33 0)
-		(fields_autoplaced yes)
-		(effects
-			(font
-				(size 1.27 1.27)
-			)
-			(justify left)
-		)
-	)

Commit message: Fix boutons poussoirs + BTN_START
Parts:
- removed J2: Conn_01x02, Connector_JST:JST_XH_S2B-XH-A_1x02_P2.50mm_Horizontal, symbol Connector_Generic:Conn_01x02
- added SW501, SW502: SW_Push, symbol Switch:SW_Push
Connections:
- net GND: now also SW501.2, SW502.2
- net Switch_Mode: now also SW502.1
- new net BTN_START: SW501.1
Other:
- note added: "Boutons poussoirs"
- note removed: "Switch (connector)"
Changed lines of the file:
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@@
 	(wire
 		(pts
-			(xy 220.98 91.44) (xy 220.98 95.25)
+			(xy 237.49 64.77) (xy 237.49 68.58)
+		)
+		(stroke
+			(width 0)
+			(type default)
+		)
+	)
+	(wire
+		(pts
+			(xy 232.41 64.77) (xy 237.49 64.77)
+		)
+		(stroke
+			(width 0)
+			(type default)
+		)
+	)
+	(wire
+		(pts
+			(xy 215.9 64.77) (xy 222.25 64.77)
+		)
+		(stroke
+			(width 0)
+			(type default)
+		)
+	)
+	(wire
+		(pts
+			(xy 232.41 81.28) (xy 237.49 81.28)
 		)
 		(stroke
@@
 	(wire
 		(pts
-			(xy 223.52 91.44) (xy 220.98 91.44)
-		)
-		(stroke
-			(width 0)
-			(type default)
-		)
-	)
-	(wire
-		(pts
 			(xy 134.62 110.49) (xy 134.62 123.19)
 		)
@@
 	(wire
 		(pts
+			(xy 237.49 81.28) (xy 237.49 85.09)
+		)
+		(stroke
+			(width 0)
+			(type default)
+		)
+	)
+	(wire
+		(pts
 			(xy 44.45 125.73) (xy 44.45 120.65)
 		)
@@
 		)
 	)
+	(wire
+		(pts
+			(xy 215.9 81.28) (xy 222.25 81.28)
+		)
+		(stroke
+			(width 0)
+			(type default)
+		)
+	)
 	(text "ST LINK / SWD Connector\n"
 		(exclude_from_sim no)
@@
 		)
 	)
-	(text "Switch (connector)\n"
+	(text "Boutons poussoirs"
 		(exclude_from_sim no)
 		(at 198.628 17.018 0)
@@
 		)
 	)
+	(hierarchical_label "BTN_START"
+		(shape output)
+		(at 215.9 64.77 180)
+		(fields_autoplaced yes)
+		(effects
+			(font
+				(size 1.27 1.27)
+			)
+			(justify right)
+		)
+	)
 	(hierarchical_label "NRST"
 		(shape output)
@@
 	(hierarchical_label "Switch_Mode"
 		(shape output)
-		(at 223.52 88.9 180)
+		(at 215.9 81.28 180)
 		(fields_autoplaced yes)
 		(effects
@@
 	)
 	(symbol
-		(lib_id "Connector_Generic:Conn_01x02")
-		(at 228.6 88.9 0)
+		(lib_id "Switch:SW_Push")
+		(at 227.33 81.28 0)
 		(unit 1)
 		(exclude_from_sim no)
@@
 		(dnp no)
 		(fields_autoplaced yes)
-		(property "Reference" "J2"
-			(at 231.14 88.8999 0)
-			(effects
-				(font
-					(size 1.27 1.27)
-				)
-				(justify left)
-			)
-		)
-		(property "Value" "Conn_01x02"
-			(at 231.14 91.4399 0)
-			(effects
-				(font
-					(size 1.27 1.27)
-				)
-				(justify left)
-			)
-		)
-		(property "Footprint" "Connector_JST:JST_XH_S2B-XH-A_1x02_P2.50mm_Horizontal"
-			(at 228.6 88.9 0)
+		(property "Reference" "SW502"
+			(at 227.33 73.66 0)
+			(effects
+				(font
+					(size 1.27 1.27)
+				)
+			)
+		)
+		(property "Value" "SW_Push"
+			(at 227.33 76.2 0)
+			(effects
+				(font
+					(size 1.27 1.27)
+				)
+			)
+		)
+		(property "Footprint" ""
+			(at 227.33 76.2 0)
 			(effects
 				(font
@@
 		)
 		(property "Datasheet" "~"
-			(at 228.6 88.9 0)
-			(effects
-				(font
-					(size 1.27 1.27)
-				)
-				(hide yes)
-			)
-		)
-		(property "Description" "Generic connector, single row, 01x02, script generated (kicad-library-utils/schlib/autogen/connector/)"
-			(at 228.6 88.9 0)
-			(effects
-				(font
-					(size 1.27 1.27)
-				)
-				(hide yes)
-			)
+			(at 227.33 76.2 0)
+			(effects
+				(font
+					(size 1.27 1.27)
+				)
+				(hide yes)
+			)
+		)
+		(property "Description" "Push button switch, generic, two pins"
+			(at 227.33 81.28 0)
+			(effects
+				(font
+					(size 1.27 1.27)
+				)
+				(hide yes)
+			)
+		)
+		(pin "2"
 		)
 		(pin "1"
-		)
-		(pin "2"
 		)
 		(instances
 			(project "Pojet_V-NOM_KiCAD"
 				(path "/37e0fdad-f3fd-48e0-8377-111662233a91/e3530ec7-9c0b-4af7-af62-470ecf12c871"
-					(reference "J2")
+					(reference "SW502")
 					(unit 1)
 				)
@@
 	)
 	(symbol
+		(lib_id "Switch:SW_Push")
+		(at 227.33 64.77 0)
+		(unit 1)
+		(exclude_from_sim no)
+		(in_bom yes)
+		(on_board yes)
+		(dnp no)
+		(fields_autoplaced yes)
+		(property "Reference" "SW501"
+			(at 227.33 57.15 0)
+			(effects
+				(font
+					(size 1.27 1.27)
+				)
+			)
+		)
+		(property "Value" "SW_Push"
+			(at 227.33 59.69 0)
+			(effects
+				(font
+					(size 1.27 1.27)
+				)
+			)
+		)
+		(property "Footprint" ""
+			(at 227.33 59.69 0)
+			(effects
+				(font
+					(size 1.27 1.27)
+				)
+				(hide yes)
+			)
+		)
+		(property "Datasheet" "~"
+			(at 227.33 59.69 0)
+			(effects
+				(font
+					(size 1.27 1.27)
+				)
+				(hide yes)
+			)
+		)
+		(property "Description" "Push button switch, generic, two pins"
+			(at 227.33 64.77 0)
+			(effects
+				(font
+					(size 1.27 1.27)
+				)
+				(hide yes)
+			)
+		)
+		(pin "2"
+		)
+		(pin "1"
+		)
+		(instances
+			(project ""
+				(path "/37e0fdad-f3fd-48e0-8377-111662233a91/e3530ec7-9c0b-4af7-af62-470ecf12c871"
+					(reference "SW501")
+					(unit 1)
+				)
+			)
+		)
+	)
+	(symbol
 		(lib_id "power:GND")
 		(at 43.18 132.08 0)
@@
 	)
 	(symbol
+		(lib_id "power:GND")
+		(at 237.49 68.58 0)
+		(unit 1)
+		(exclude_from_sim no)
+		(in_bom yes)
+		(on_board yes)
+		(dnp no)
+		(fields_autoplaced yes)
+		(property "Reference" "#PWR0506"
+			(at 237.49 74.93 0)
+			(effects
+				(font
+					(size 1.27 1.27)
+				)
+				(hide yes)
+			)
+		)
+		(property "Value" "GND"
+			(at 237.49 73.66 0)
+			(effects
+				(font
+					(size 1.27 1.27)
+				)
+			)
+		)
+		(property "Footprint" ""
+			(at 237.49 68.58 0)
+			(effects
+				(font
+					(size 1.27 1.27)
+				)
+				(hide yes)
+			)
+		)
+		(property "Datasheet" ""
+			(at 237.49 68.58 0)
+			(effects
+				(font
+					(size 1.27 1.27)
+				)
+				(hide yes)
+			)
+		)
+		(property "Description" "Power symbol creates a global label with name \"GND\" , ground"
+			(at 237.49 68.58 0)
+			(effects
+				(font
+					(size 1.27 1.27)
+				)
+				(hide yes)
+			)
+		)
+		(pin "1"
+		)
+		(instances
+			(project ""
+				(path "/37e0fdad-f3fd-48e0-8377-111662233a91/e3530ec7-9c0b-4af7-af62-470ecf12c871"
+					(reference "#PWR0506")
+					(unit 1)
+				)
+			)
+		)
+	)
+	(symbol
 		(lib_id "Device:R_Small")
 		(at 134.62 107.95 0)
@@
 	(symbol
 		(lib_id "power:GND")
-		(at 220.98 95.25 0)
+		(at 237.49 85.09 0)
 		(unit 1)
 		(exclude_from_sim no)
@@
 		(fields_autoplaced yes)
 		(property "Reference" "#PWR0505"
-			(at 220.98 101.6 0)
+			(at 237.49 91.44 0)
 			(effects
 				(font
@@
 		)
 		(property "Value" "GND"
-			(at 220.98 100.33 0)
+			(at 237.49 90.17 0)
 			(effects
 				(font
@@
 		)
 		(property "Footprint" ""
-			(at 220.98 95.25 0)
+			(at 237.49 85.09 0)
 			(effects
 				(font
@@
 		)
 		(property "Datasheet" ""
-			(at 220.98 95.25 0)
+			(at 237.49 85.09 0)
 			(effects
 				(font
@@
 		)
 		(property "Description" "Power symbol creates a global label with name \"GND\" , ground"
-			(at 220.98 95.25 0)
-			(effects
-				(font
+			(at 237.49 85.09 0)
+			(effects
+				(font

Commit message: Empreinte boutons
Parts:
- SW501, SW502: footprint (none) -> Button_Switch_SMD:SW_Push_1P1T_NO_6x6mm_H9.5mm

Commit message: empreinte
Parts:
- R2, R3: footprint Resistor_SMD:R_0603_1608Metric_Pad0.98x0.95mm_HandSolder -> Resistor_SMD:R_0402_1005Metric
Changed lines of the file:
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@@
 			)
 		)
-		(property "Footprint" "Resistor_SMD:R_0603_1608Metric_Pad0.98x0.95mm_HandSolder"
+		(property "Footprint" "Resistor_SMD:R_0402_1005Metric"
 			(at 154.94 107.95 0)
 			(effects
@@
 			)
 		)
-		(property "Footprint" "Resistor_SMD:R_0603_1608Metric_Pad0.98x0.95mm_HandSolder"
+		(property "Footprint" "Resistor_SMD:R_0402_1005Metric"
 			(at 134.62 107.95 0)
 			(effects

Commit message: Correction des erreurs évidentes
Changements avant vérification des erreurs :
- Désallocation du pin BTN_RESET
- Réarrangement de certaines sources pour cohérence avec tous les
schémas éléctriques
Other:
- moved on the sheet: D1, D2, J1, R2, R3, SW501, SW502

Commit message: point de test et début de placement
Parts:
- added TP501, TP502, TP503, TP504, TP505, TP506: TestPoint, TestPoint:TestPoint_Pad_D1.0mm, symbol Connector:TestPoint
Connections:
- net +3.3V: now also TP505.1
- net NRST: now also TP506.1
- net SWCLK: now also TP504.1
- net SWDIO: now also TP503.1
- net VCP_RX: now also TP501.1
- net VCP_TX: now also TP502.1

Commit message: maj emplacement
Parts:
- removed TP501, TP502, TP504, TP506: TestPoint, TestPoint:TestPoint_Pad_D1.0mm, symbol Connector:TestPoint

Commit message: placement maj
Parts:
- added TP501, TP502, TP504: TestPoint, TestPoint:TestPoint_Pad_D1.5mm, symbol Connector:TestPoint
- TP503, TP505: footprint TestPoint:TestPoint_Pad_D1.0mm -> TestPoint:TestPoint_Pad_D1.5mm
Connections:
- net +3.3V: no longer TP505.1
- net NRST: now also TP502.1
- net SWCLK: now also TP501.1
- net VCP_RX: now also TP505.1
- net VCP_TX: now also TP504.1
