File: Pojet_V-NOM_KiCAD/_autosave-Pojet_V-NOM_KiCAD.kicad_pcb (KiCad board)
At the start: 4 copper layers, 57 x 54 mm, 75 parts, among them IC1002 MP1475SGJ-P, J1 Conn_ST_STDC14, J3 Conn_01x08, J301 Conn_01x06, J302 Conn_01x06, J4 Conn_01x03, J5 Conn_01x03, J6 Switch ON/OFF, SW501 SW_Push, SW502 SW_Push, U1 STM32G431CBU6, U2 ADXL343, U701 ZXBM5210-SP, U801 ZXBM5210-SP, Y1 16 MHz

Commit message: maj routage
Parts:
- moved C1008 62.2 mm to (90.1, 77.5)
- moved C1009 62.2 mm to (83.1, 85.0)
- moved C1010 62.2 mm to (82.6, 78.0)
- moved C1011 62.2 mm to (80.5, 79.1)
- moved C1012 62.2 mm to (80.6, 85.0)
- moved C1013 62.2 mm to (85.1, 82.5)
- moved C1014 62.2 mm to (89.1, 79.5)
- moved IC1002 62.2 mm to (86.0, 80.0)
- moved L1002 62.2 mm to (83.1, 81.5)
- moved R1007 62.2 mm to (87.1, 77.5)
- moved R1008 62.2 mm to (89.1, 76.5)
- moved R1009 62.2 mm to (88.6, 78.0)
- moved R1010 62.2 mm to (84.6, 77.5)
- moved R1011 62.2 mm to (87.1, 82.5)
- moved R1012 62.2 mm to (89.1, 80.5)
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Routing:
- net /acquisition/RX_LIDAR: track 46.2 -> 49.0 mm
- net /acquisition/TX_LIDAR: track 47.0 -> 49.7 mm

Commit message: retouche routage
Parts:
- moved C1008 0.99 mm to (90.6, 76.6)
- moved C1009 0.99 mm to (83.6, 84.1)
- moved C1010 0.99 mm to (83.1, 77.1)
- moved C1011 0.99 mm to (81.0, 78.2)
- moved C1012 0.99 mm to (81.1, 84.1), turned to 90 degrees
- moved C1013 0.99 mm to (85.6, 81.6)
- moved C1014 0.99 mm to (89.6, 78.6)
- moved IC1002 0.99 mm to (86.5, 79.1)
- moved L1002 0.99 mm to (83.6, 80.6)
- moved R1007 0.99 mm to (87.6, 76.6)
- moved R1008 0.99 mm to (89.6, 75.6)
- moved R1009 0.99 mm to (89.1, 77.1)
- moved R1010 0.99 mm to (85.1, 76.6)
- moved R1011 0.99 mm to (87.6, 81.6)
- moved R1012 0.99 mm to (89.6, 79.6)
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Routing:
- net +5V: track 0.00 -> 13.0 mm, vias 0 -> 10
- net /acquisition/AG_MISO: track 13.3 -> 18.1 mm, vias 0 -> 2
- net /acquisition/VIT_MOT_LIDAR: track 56.0 -> 51.7 mm
- net /acquisition/RX_LIDAR: track 49.0 -> 46.1 mm, vias 3 -> 2
- net /controle/SWDIO: track 46.6 -> 43.8 mm
- net /controle/SWCLK: track 45.3 -> 42.8 mm
- net /acquisition/EN_MOT: track 45.0 -> 42.5 mm
- net /acquisition/EN_LIDAR: track 44.5 -> 42.1 mm
- net /Deplacement/Encoder A phase 1: track 50.4 -> 52.6 mm
- net /acquisition/TX_LIDAR: track 49.7 -> 48.0 mm
- net /acquisition/AG_INT2: track 25.2 -> 24.1 mm
- net /acquisition/AG_INT1: track 24.4 -> 23.4 mm
- net /Deplacement/FWD1: track 23.2 -> 22.3 mm
- net /Deplacement/FWD2: track 9.13 -> 8.32 mm
- net /acquisition/AG_MOSI: track 18.2 -> 17.6 mm
