File: Pojet_V-NOM_KiCAD/Pojet_V-NOM_KiCAD.kicad_pcb (KiCad board)
At the start: 2 copper layers, 55 parts, among them IC1002 MP1475SGJ-P, J1 Conn_ST_STDC14, J3 Conn_01x08, J301 Conn_01x06, J302 Conn_01x06, J4 Conn_01x03, J5 Conn_01x03, J6 Switch ON/OFF, SW501 SW_Push, SW502 SW_Push, U1 STM32G431CBU6, U2 ADXL343, U701 ZXBM5210-SP, U801 ZXBM5210-SP, Y1 16 MHz

Commit message: point de test et début de placement
Parts:
- added TP1001: TestPoint, TestPoint:TestPoint_Pad_D1.0mm, F.Cu at (268.8, 95.6)
- added TP1002: TestPoint, TestPoint:TestPoint_Pad_D1.0mm, F.Cu at (268.8, 100.3)
- added TP1003: TestPoint, TestPoint:TestPoint_Pad_D1.0mm, F.Cu at (218.9, 89.3)
- added TP201: TestPoint, TestPoint:TestPoint_Pad_D1.0mm, F.Cu at (268.8, 106.9)
- added TP202: TestPoint, TestPoint:TestPoint_Pad_D1.0mm, F.Cu at (201.0, 68.7)
- added TP203: TestPoint, TestPoint:TestPoint_Pad_D1.0mm, F.Cu at (201.0, 73.3)
- added TP204: TestPoint, TestPoint:TestPoint_Pad_D1.0mm, F.Cu at (201.0, 78.0)
- added TP205: TestPoint, TestPoint:TestPoint_Pad_D1.0mm, F.Cu at (201.0, 82.6)
- added TP206: TestPoint, TestPoint:TestPoint_Pad_D1.0mm, F.Cu at (201.0, 87.3)
- added TP207: TestPoint, TestPoint:TestPoint_Pad_D1.0mm, F.Cu at (205.6, 68.7)
- added TP208: TestPoint, TestPoint:TestPoint_Pad_D1.0mm, F.Cu at (205.6, 73.3)
- added TP209: TestPoint, TestPoint:TestPoint_Pad_D1.0mm, F.Cu at (205.6, 78.0)
- added TP210: TestPoint, TestPoint:TestPoint_Pad_D1.0mm, F.Cu at (205.6, 82.6)
- added TP211: TestPoint, TestPoint:TestPoint_Pad_D1.0mm, F.Cu at (205.6, 87.3)
- added TP301: TestPoint, TestPoint:TestPoint_Pad_D1.0mm, F.Cu at (262.1, 75.0)
- added TP302: TestPoint, TestPoint:TestPoint_Pad_D1.0mm, F.Cu at (262.1, 79.7)
- added TP303: TestPoint, TestPoint:TestPoint_Pad_D1.0mm, F.Cu at (262.1, 84.3)
- added TP304: TestPoint, TestPoint:TestPoint_Pad_D1.0mm, F.Cu at (262.1, 89.0)
- added TP501: TestPoint, TestPoint:TestPoint_Pad_D1.0mm, F.Cu at (262.1, 95.6)
- added TP502: TestPoint, TestPoint:TestPoint_Pad_D1.0mm, F.Cu at (262.1, 100.3)
- added TP503: TestPoint, TestPoint:TestPoint_Pad_D1.0mm, F.Cu at (262.1, 104.9)
- added TP504: TestPoint, TestPoint:TestPoint_Pad_D1.0mm, F.Cu at (262.1, 109.6)
- added TP505: TestPoint, TestPoint:TestPoint_Pad_D1.0mm, F.Cu at (218.9, 68.7)
- added TP506: TestPoint, TestPoint:TestPoint_Pad_D1.0mm, F.Cu at (218.9, 73.3)
- added TP601: TestPoint, TestPoint:TestPoint_Pad_D1.0mm, F.Cu at (246.2, 75.0)
- added TP602: TestPoint, TestPoint:TestPoint_Pad_D1.0mm, F.Cu at (246.2, 79.7)
- added TP603: TestPoint, TestPoint:TestPoint_Pad_D1.0mm, F.Cu at (246.2, 84.3)
- added TP604: TestPoint, TestPoint:TestPoint_Pad_D1.0mm, F.Cu at (246.2, 89.0)
- added TP605: TestPoint, TestPoint:TestPoint_Pad_D1.0mm, F.Cu at (246.2, 93.6)
- added TP606: TestPoint, TestPoint:TestPoint_Pad_D1.0mm, F.Cu at (250.8, 75.0)
- added TP607: TestPoint, TestPoint:TestPoint_Pad_D1.0mm, F.Cu at (250.8, 79.7)
- added TP608: TestPoint, TestPoint:TestPoint_Pad_D1.0mm, F.Cu at (250.8, 84.3)
- added TP609: TestPoint, TestPoint:TestPoint_Pad_D1.0mm, F.Cu at (250.8, 89.0)
- added TP610: TestPoint, TestPoint:TestPoint_Pad_D1.0mm, F.Cu at (250.8, 93.6)
- added TP611: TestPoint, TestPoint:TestPoint_Pad_D1.0mm, F.Cu at (255.5, 75.0)
- added TP612: TestPoint, TestPoint:TestPoint_Pad_D1.0mm, F.Cu at (255.5, 79.7)
- added TP613: TestPoint, TestPoint:TestPoint_Pad_D1.0mm, F.Cu at (255.5, 84.3)
- added TP614: TestPoint, TestPoint:TestPoint_Pad_D1.0mm, F.Cu at (212.3, 68.7)
- added TP615: TestPoint, TestPoint:TestPoint_Pad_D1.0mm, F.Cu at (212.3, 73.3)
- added TP616: TestPoint, TestPoint:TestPoint_Pad_D1.0mm, F.Cu at (212.3, 78.0)
- added TP617: TestPoint, TestPoint:TestPoint_Pad_D1.0mm, F.Cu at (212.3, 82.6)
- added TP701: TestPoint, TestPoint:TestPoint_Pad_D1.0mm, F.Cu at (268.8, 75.0)
- added TP702: TestPoint, TestPoint:TestPoint_Pad_D1.0mm, F.Cu at (268.8, 79.7)
- added TP703: TestPoint, TestPoint:TestPoint_Pad_D1.0mm, F.Cu at (268.8, 84.3)
- added TP704: TestPoint, TestPoint:TestPoint_Pad_D1.0mm, F.Cu at (268.8, 89.0)
- added TP705: TestPoint, TestPoint:TestPoint_Pad_D1.0mm, F.Cu at (218.9, 80.0)
- added TP801: TestPoint, TestPoint:TestPoint_Pad_D1.0mm, F.Cu at (275.4, 75.0)
- added TP802: TestPoint, TestPoint:TestPoint_Pad_D1.0mm, F.Cu at (275.4, 79.7)
- added TP803: TestPoint, TestPoint:TestPoint_Pad_D1.0mm, F.Cu at (275.4, 84.3)
- added TP804: TestPoint, TestPoint:TestPoint_Pad_D1.0mm, F.Cu at (275.4, 89.0)
- added TP805: TestPoint, TestPoint:TestPoint_Pad_D1.0mm, F.Cu at (212.3, 89.3)
- added TP901: TestPoint, TestPoint:TestPoint_Pad_D1.0mm, F.Cu at (275.4, 95.6)
- added TP902: TestPoint, TestPoint:TestPoint_Pad_D1.0mm, F.Cu at (275.4, 100.3)
- IC1002: footprint KiCad:SOT65P280X100-8N -> Package_TO_SOT_SMD:SOT-23-8
- moved BT1 100.0 mm to (231.5, 131.5)
- moved C1 100.0 mm to (229.5, 143.1)
- moved C1009 100.0 mm to (250.2, 143.6)
- moved C1010 100.0 mm to (250.2, 146.6)
- moved C1012 100.0 mm to (250.2, 149.7)
- moved C2 100.0 mm to (229.5, 145.1)
- moved C5 100.0 mm to (229.5, 147.1)
- moved C6 100.0 mm to (229.5, 149.0)
- moved C7 100.0 mm to (229.5, 151.0)
- moved C701 100.0 mm to (250.4, 134.2)
- moved C702 100.0 mm to (250.4, 136.1)
- moved IC1002 100.0 mm to (255.1, 152.3)
- moved J3 100.0 mm to (208.8, 102.4)
- moved J301 100.0 mm to (239.3, 100.8)
- moved J302 100.0 mm to (239.3, 114.3)
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Connections:
- U1 pad 39: /controle/EN_LIDAR -> /acquisition/EN_LIDAR
- U1 pad 40: /controle/EN_MOT -> /acquisition/EN_MOT
- U1 pad 46: /controle/BTN_RESET -> unconnected-(U1-PB8-Pad46)
Other:
- board outline added: 57 x 54 mm
- copper layers 2 -> 4

Commit message: maj emplacement
Parts:
- removed TP202, TP203, TP204, TP205, TP206, TP207, TP208, TP209, TP210, TP501, TP502, TP504, TP506, TP605, TP606, TP609, TP610, TP615, TP616, TP617, TP701, TP702, TP705, TP801, TP802, TP805: TestPoint, TestPoint:TestPoint_Pad_D1.0mm

Commit message: placement des compo dans la pcb
Parts:
- moved TP804 225.7 mm to (52.5, 53.6)
- moved TP803 225.5 mm to (52.5, 50.5)
- moved TP901 220.3 mm to (56.5, 70.8)
- moved TP902 212.9 mm to (63.5, 79.5)
- moved TP704 206.9 mm to (63.5, 63.0)
- moved TP703 206.7 mm to (63.5, 59.9)
- moved U701 206.2 mm to (59.0, 60.0), turned to 90 degrees
- moved C701 205.2 mm to (57.5, 64.0)
- moved C702 203.6 mm to (60.0, 64.0)
- moved TP302 199.9 mm to (63.5, 57.5)
- moved J302 198.9 mm to (45.0, 71.5), turned to 90 degrees
- moved IC1002 198.6 mm to (71.4, 77.0)
- moved TP304 198.5 mm to (64.5, 70.3)
- moved C1013 198.2 mm to (68.5, 77.0), turned to -90 degrees
- moved TP301 196.9 mm to (66.0, 57.5)
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
Commit message: placement maj
Parts:
- removed TP201, TP211, TP301, TP302, TP303, TP304, TP607, TP608, TP613, TP614, TP902: TestPoint, TestPoint:TestPoint_Pad_D1.0mm
- added C201: 10nF, Capacitor_SMD:C_0402_1005Metric, F.Cu at (76.3, 61.8)
- added C202: 100nF, Capacitor_SMD:C_0402_1005Metric, F.Cu at (64.8, 65.3)
- added TP501: TestPoint, TestPoint:TestPoint_Pad_D1.5mm, F.Cu at (87.0, 58.0)
- added TP502: TestPoint, TestPoint:TestPoint_Pad_D1.5mm, F.Cu at (87.0, 54.0)
- added TP504: TestPoint, TestPoint:TestPoint_Pad_D1.5mm, F.Cu at (87.0, 51.0)
- C701, C702, C801, C802: footprint Capacitor_SMD:C_0402_1005Metric -> Capacitor_SMD:C_0603_1608Metric
- L1: value 47nH -> 39nH
- L1002: footprint Capacitor_SMD:C_0603_1608Metric -> Inductor_SMD:L_0402_1005Metric
- TP1001, TP1002, TP1003, TP503, TP505, TP601, TP602, TP603, TP604, TP611, TP612, TP703, TP704, TP803, TP804, TP901: footprint TestPoint:TestPoint_Pad_D1.0mm -> TestPoint:TestPoint_Pad_D1.5mm
- Y1: footprint Crystal:Crystal_SMD_0603-4Pin_6.0x3.5mm -> Crystal:Crystal_SMD_EuroQuartz_MT-4Pin_3.2x2.5mm
- moved D1 43.8 mm to (87.1, 68.0)
- moved R2 42.4 mm to (86.6, 69.5)
- moved TP612 35.2 mm to (55.0, 83.5)
- moved TP611 26.6 mm to (54.0, 75.0)
- moved R3 23.2 mm to (59.8, 62.3), turned to 180 degrees
- moved R1009 19.6 mm to (87.6, 79.0), turned to -90 degrees
- moved R1011 19.6 mm to (86.1, 83.5), turned to 180 degrees
- moved R1012 19.4 mm to (88.1, 81.5), turned to 0 degrees
- moved D2 19.0 mm to (62.8, 62.3), turned to 0 degrees
- moved C1013 17.0 mm to (84.1, 83.5), turned to 180 degrees
- moved R1007 16.8 mm to (86.1, 78.5), turned to 180 degrees
- moved C6 16.5 mm to (62.8, 64.3), turned to 180 degrees
- moved C1008 14.6 mm to (89.1, 78.5), turned to 180 degrees
- moved TP901 14.6 mm to (66.5, 81.5)
- moved C1014 14.5 mm to (88.1, 80.5), turned to 0 degrees
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Connections:
- J301 pad 5: +BATT -> +3.3V
- J302 pad 5: +BATT -> +3.3V
- TP505 pad 1: +3.3V -> /controle/VCP_RX
Routing:
- net Net-(U1-PF0): track 0.00 -> 1.46 mm
- net Net-(C2-Pad2): track 0.00 -> 1.43 mm
- net Net-(U1-VDDA): track 0.00 -> 1.30 mm
- net +3.3V: track 0.00 -> 1.20 mm, vias 0 -> 1
- net GND: vias 0 -> 17
- added copper zone on In2.Cu, net +3.3V

Commit message: routage
Parts:
- moved TP601 35.2 mm to (75.3, 52.3), turned to 90 degrees
- moved TP612 35.0 mm to (75.8, 55.3), turned to 90 degrees
- moved TP602 31.4 mm to (72.3, 51.8), turned to 90 degrees
- moved C4 31.3 mm to (72.9, 58.2), turned to 180 degrees
- moved U2 29.5 mm to (71.8, 55.3), turned to 90 degrees
- moved TP603 27.8 mm to (69.8, 52.3), turned to 90 degrees
- moved C3 27.1 mm to (69.9, 58.2), turned to 0 degrees
- moved R2 26.8 mm to (62.5, 57.8), turned to 90 degrees
- moved D1 25.4 mm to (62.8, 60.8), turned to -90 degrees
- moved TP604 24.0 mm to (67.3, 53.3), turned to 90 degrees
- moved C701 23.0 mm to (54.0, 48.0), turned to -90 degrees
- moved TP611 22.9 mm to (67.3, 56.3), turned to 90 degrees
- moved C702 19.6 mm to (54.0, 51.0), turned to 90 degrees
- moved U701 18.7 mm to (58.5, 49.5), turned to 0 degrees
- moved C7 16.9 mm to (65.5, 73.5)
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Routing:
- net /acquisition/TOF2: track 0.00 -> 40.8 mm
- net /controle/BTN_MODE: track 0.00 -> 32.1 mm
- net /acquisition/TOF1: track 0.00 -> 26.5 mm
- net /Deplacement/Encoder A phase 2: track 0.00 -> 22.6 mm
- net /Deplacement/Encoder B phase 2: track 0.00 -> 18.3 mm
- net /Deplacement/VREF2: track 0.00 -> 17.1 mm
- net /Deplacement/VREF1: track 0.00 -> 17.1 mm
- net /Deplacement/Driver_Motor2/OUT1: track 0.00 -> 16.8 mm
- net /Deplacement/FWD2: track 0.00 -> 14.0 mm
- net /Deplacement/Driver_Motor1/OUT2: track 0.00 -> 12.5 mm
- net Net-(BT1-+): track 0.00 -> 9.66 mm
- net /Deplacement/Driver_Motor2/OUT2: track 0.00 -> 9.36 mm
- net /controle/BTN_START: track 0.00 -> 7.95 mm
- net /controle/VCP_RX: track 0.00 -> 7.09 mm
- net Net-(IC1002-VCC): track 0.00 -> 6.97 mm
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
Commit message: grande partie de routage
Parts:
- removed TP501, TP502, TP503, TP601, TP602: TestPoint, TestPoint:TestPoint_Pad_D1.5mm
- added C501: 100nf, Capacitor_SMD:C_0402_1005Metric, F.Cu at (53.9, 81.9)
- added C502: 100nf, Capacitor_SMD:C_0402_1005Metric, F.Cu at (77.7, 43.4)
- added R501: 470k, Resistor_SMD:R_0402_1005Metric, F.Cu at (76.0, 43.4)
- added R502: 470k, Resistor_SMD:R_0402_1005Metric, F.Cu at (53.9, 84.2)
- moved C902 38.0 mm to (89.2, 63.6)
- moved C901 37.8 mm to (89.2, 70.1)
- moved TP901 37.8 mm to (86.2, 65.8)
- moved PS901 37.6 mm to (89.3, 66.8)
- moved C801 16.6 mm to (47.5, 69.1)
- moved C802 16.6 mm to (50.6, 69.1)
- moved C1008 10.5 mm to (90.4, 78.7)
- moved C1009 10.5 mm to (83.4, 86.2)
- moved C1010 10.5 mm to (82.9, 79.2)
- moved C1012 10.5 mm to (80.9, 86.2)
- moved C1013 10.5 mm to (85.4, 83.7)
- moved C1014 10.5 mm to (89.4, 80.7)
- moved L1002 10.5 mm to (83.4, 82.7)
- moved R1007 10.5 mm to (87.4, 78.7)
- moved R1008 10.5 mm to (89.4, 77.7)
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Routing:
- net GND: track 0.00 -> 51.4 mm, vias 17 -> 71
- net /acquisition/VIT_MOT_LIDAR: track 0.00 -> 50.3 mm, vias 0 -> 2
- net /acquisition/EN_MOT: track 0.00 -> 43.0 mm, vias 0 -> 4
- net /acquisition/EN_LIDAR: track 0.00 -> 42.8 mm, vias 0 -> 4
- net /controle/BTN_START: track 7.95 -> 50.4 mm, vias 0 -> 2
- net /controle/VCP_RX: track 7.09 -> 48.1 mm, vias 0 -> 2
- net /controle/SWDIO: track 4.68 -> 43.6 mm, vias 0 -> 2
- net /controle/VCP_TX: track 3.85 -> 42.6 mm, vias 0 -> 2
- net /controle/SWCLK: track 4.03 -> 42.4 mm, vias 0 -> 2
- net /controle/NRST: track 4.64 -> 31.5 mm, vias 0 -> 2
- net /Deplacement/Encoder A phase 2: track 22.6 -> 0.00 mm
- net /acquisition/AG_INT1: track 2.62 -> 24.6 mm, vias 0 -> 2
- net /acquisition/AG_INT2: track 2.79 -> 24.7 mm
- net /Deplacement/Encoder B phase 2: track 18.3 -> 0.00 mm
- net /acquisition/AG_CSN: track 2.00 -> 19.9 mm, vias 0 -> 2
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- added copper zone on F.Cu, net /Deplacement/Driver_Motor1/OUT1
- added copper zone on F.Cu, net /Deplacement/Driver_Motor1/OUT2
- added copper zone on F.Cu, net /Deplacement/Driver_Motor2/OUT1
- added copper zone on F.Cu, net /Deplacement/Driver_Motor2/OUT2
- added copper zone on In1.Cu, net GND

Commit message: création schématique inductance
Parts:
- moved C1008 1.19 mm to (90.1, 77.5)
- moved C1009 1.19 mm to (83.1, 85.0)
- moved C1010 1.19 mm to (82.6, 78.0)
- moved C1012 1.19 mm to (80.6, 85.0)
- moved C1013 1.19 mm to (85.1, 82.5)
- moved C1014 1.19 mm to (89.1, 79.5)
- moved L1002 1.19 mm to (83.1, 81.5)
- moved R1007 1.19 mm to (87.1, 77.5)
- moved R1008 1.19 mm to (89.1, 76.5)
- moved R1009 1.19 mm to (88.6, 78.0)
- moved R1010 1.19 mm to (84.6, 77.5)
- moved R1011 1.19 mm to (87.1, 82.5)
- moved R1012 1.19 mm to (89.1, 80.5)
- moved TP1001 1.19 mm to (80.6, 82.0)
- moved TP1003 1.19 mm to (85.1, 75.5)
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Routing:
- net /Deplacement/Encoder A phase 1: track 0.00 -> 50.4 mm, vias 0 -> 1
- net /acquisition/TX_LIDAR: track 0.00 -> 49.7 mm, vias 0 -> 1
- net /acquisition/RX_LIDAR: track 0.00 -> 49.0 mm, vias 0 -> 3
- net /Deplacement/Encoder A phase 2: track 0.00 -> 34.5 mm, vias 0 -> 1
- net /Deplacement/Encoder B phase 1: track 0.00 -> 31.8 mm, vias 0 -> 1
- net /Deplacement/Encoder B phase 2: track 0.00 -> 18.3 mm, vias 0 -> 1
- net Net-(BT1-+): track 0.00 -> 9.66 mm
- net /acquisition/VIT_MOT_LIDAR: track 50.3 -> 56.0 mm
- net /acquisition/AG_MISO: track 18.8 -> 13.3 mm, vias 2 -> 0
- net /controle/BTN_MODE: track 27.8 -> 31.4 mm
- net /Deplacement/FWD1: track 20.0 -> 23.2 mm
- net /controle/SWDIO: track 43.6 -> 46.6 mm
- net /controle/SWCLK: track 42.4 -> 45.3 mm
- net /acquisition/EN_MOT: track 43.0 -> 45.0 mm
- net /acquisition/EN_LIDAR: track 42.8 -> 44.5 mm
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
Commit message: maj routage
Parts:
- BT1: footprint Connector_JST:JST_XH_S2B-XH-A-1_1x02_P2.50mm_Horizontal -> Connector_JST:JST_XH_S2B-XH-A_1x02_P2.50mm_Horizontal
- J3: footprint Connector_JST:JST_XH_S8B-XH-A-1_1x08_P2.50mm_Horizontal -> Connector_JST:JST_XH_S8B-XH-A_1x08_P2.50mm_Horizontal
- J4, J5: footprint Connector_JST:JST_XH_S3B-XH-A-1_1x03_P2.50mm_Horizontal -> Connector_JST:JST_XH_S3B-XH-A_1x03_P2.50mm_Horizontal
- L1002: footprint Inductor_SMD:L_0402_1005Metric -> Library:Inductance L1
- moved L1002 10.6 mm to (72.5, 81.1)
- moved C1008 0.99 mm to (90.6, 76.6)
- moved C1009 0.99 mm to (83.6, 84.1)
- moved C1010 0.99 mm to (83.1, 77.1)
- moved C1011 0.99 mm to (81.0, 78.2)
- moved C1012 0.99 mm to (81.1, 84.1), turned to 90 degrees
- moved C1013 0.99 mm to (85.6, 81.6)
- moved C1014 0.99 mm to (89.6, 78.6)
- moved IC1002 0.99 mm to (86.5, 79.1)
- moved R1007 0.99 mm to (87.6, 76.6)
- moved R1008 0.99 mm to (89.6, 75.6)
- moved R1009 0.99 mm to (89.1, 77.1)
- moved R1010 0.99 mm to (85.1, 76.6)
- moved R1011 0.99 mm to (87.6, 81.6)
- moved R1012 0.99 mm to (89.6, 79.6)
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Routing:
- net +5V: track 0.00 -> 13.0 mm, vias 0 -> 10
- net /acquisition/AG_MISO: track 13.3 -> 18.1 mm, vias 0 -> 2
- net /acquisition/VIT_MOT_LIDAR: track 56.0 -> 51.7 mm
- net /acquisition/RX_LIDAR: track 49.0 -> 46.1 mm, vias 3 -> 2
- net /controle/SWDIO: track 46.6 -> 43.8 mm
- net /controle/SWCLK: track 45.3 -> 42.8 mm
- net /acquisition/EN_MOT: track 45.0 -> 42.5 mm
- net /acquisition/EN_LIDAR: track 44.5 -> 42.1 mm
- net /Deplacement/Encoder A phase 1: track 50.4 -> 52.6 mm
- net /acquisition/TX_LIDAR: track 49.7 -> 48.0 mm
- net /acquisition/AG_INT2: track 25.2 -> 24.1 mm
- net /acquisition/AG_INT1: track 24.4 -> 23.4 mm
- net /Deplacement/FWD1: track 23.2 -> 22.3 mm
- net /Deplacement/FWD2: track 9.13 -> 8.32 mm
- net /acquisition/AG_MOSI: track 18.2 -> 17.6 mm
