File: Pojet_V-NOM_KiCAD/Pojet_V-NOM_KiCAD.kicad_pcb (KiCad board)
At the start: 4 copper layers, 57 x 54 mm, 75 parts, among them IC1002 MP1475SGJ-P, J1 Conn_ST_STDC14, J3 Conn_01x08, J301 Conn_01x06, J302 Conn_01x06, J4 Conn_01x03, J5 Conn_01x03, J6 Switch ON/OFF, SW501 SW_Push, SW502 SW_Push, U1 STM32G431CBU6, U2 ADXL343, U701 ZXBM5210-SP, U801 ZXBM5210-SP, Y1 16 MHz

Commit message: maj routage
Parts:
- moved L1002 88.7 mm to (158.8, 60.6)
- moved C1012 75.5 mm to (154.1, 64.5), turned to 180 degrees
- moved C1013 74.9 mm to (155.2, 54.2), turned to 0 degrees
- moved C1009 72.5 mm to (154.1, 67.2), turned to 180 degrees
- moved R1011 70.7 mm to (153.6, 56.4), turned to 90 degrees
- moved C1011 70.4 mm to (150.0, 64.2), turned to 180 degrees
- moved TP1001 70.3 mm to (145.7, 53.4)
- moved C1010 69.0 mm to (150.5, 62.5), turned to 180 degrees
- moved IC1002 67.0 mm to (150.5, 59.3), turned to 90 degrees
- moved C1014 65.1 mm to (150.7, 55.9)
- moved R1010 64.5 mm to (147.5, 60.4), turned to 180 degrees
- moved R1008 63.9 mm to (149.7, 53.9), turned to -90 degrees
- moved R1007 63.4 mm to (147.8, 56.9), turned to -90 degrees
- moved C1008 61.6 mm to (147.8, 53.9), turned to -90 degrees
- moved TP1003 60.9 mm to (144.8, 60.4)
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Routing:
- net Net-(IC1002-SW): track 4.16 -> 15.0 mm
- net Net-(IC1002-VCC): track 7.18 -> 17.5 mm, vias 0 -> 2
- net Net-(IC1002-EN/SYNC): track 1.58 -> 11.4 mm, vias 0 -> 2
- net +BATT: track 0.00 -> 5.92 mm
- net +5V: track 13.0 -> 18.8 mm, vias 10 -> 6
- net Net-(C1008-Pad2): track 3.01 -> 5.41 mm
- net GND: track 52.2 -> 53.8 mm
- net Net-(C1013-Pad1): track 1.01 -> 2.51 mm
- net Net-(IC1002-BST): track 1.78 -> 2.63 mm

Commit message: maj routage 24
Parts:
- moved L1002 73.2 mm to (88.7, 81.7)
- moved C1009 71.5 mm to (86.0, 89.2)
- moved C1008 71.5 mm to (79.8, 75.8)
- moved C1012 71.5 mm to (86.0, 86.4)
- moved R1009 71.5 mm to (78.3, 78.7)
- moved R1010 71.5 mm to (79.5, 82.3)
- moved C1010 71.5 mm to (82.5, 84.3)
- moved C1011 71.5 mm to (82.0, 86.1)
- moved C1013 71.5 mm to (87.2, 76.1)
- moved C1014 71.5 mm to (82.6, 77.8)
- moved IC1002 71.5 mm to (82.5, 81.2)
- moved R1007 71.5 mm to (79.8, 78.8)
- moved R1008 71.5 mm to (81.6, 75.8)
- moved R1011 71.5 mm to (85.6, 78.3)
- moved R1012 71.5 mm to (79.3, 83.9)
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Routing:
- net /acquisition/RX_LIDAR: track 46.1 -> 49.8 mm
- net Net-(IC1002-SW): track 15.0 -> 11.5 mm
- net /acquisition/TX_LIDAR: track 48.0 -> 51.5 mm
- net /acquisition/VIT_MOT_LIDAR: track 51.7 -> 54.6 mm
- net /Deplacement/VREF2: track 9.56 -> 11.9 mm
- net /controle/SWDIO: track 43.8 -> 46.1 mm
- net Net-(BT1-+): track 9.66 -> 11.8 mm
- net +BATT: track 5.92 -> 8.00 mm
- net /controle/SWCLK: track 42.8 -> 44.6 mm
- net +3.3V: track 2.73 -> 4.37 mm, vias 1 -> 2
- net /acquisition/EN_LIDAR: track 42.1 -> 43.6 mm
- net /Deplacement/FWD1: track 22.4 -> 21.4 mm
- net /acquisition/EN_MOT: track 42.5 -> 43.3 mm
- net /Deplacement/Encoder B phase 1: track 31.7 -> 32.4 mm
- net Net-(IC1002-EN/SYNC): track 11.4 -> 12.0 mm
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
Commit message: Maj final rootage + logo
Parts:
- added G***: LOGO, LOGO:VNOM, F.Cu at (63.1, 85.9)
- moved TP901 2.17 mm to (85.9, 63.6)
- moved C201 0.76 mm to (60.5, 60.1)
- moved C6 0.76 mm to (61.5, 60.1)
- moved C202 0.63 mm to (59.7, 62.6)
- moved L1 0.39 mm to (60.7, 62.7)
- moved C501 0.38 mm to (53.9, 82.3)
- moved C2 0.37 mm to (68.1, 67.7)
- moved R1 0.36 mm to (68.1, 68.7)
- moved C7 0.09 mm to (65.5, 73.5)
Routing:
- net +3.3V: track 4.37 -> 22.9 mm, vias 2 -> 16
- net +BATT: track 8.00 -> 25.1 mm, vias 0 -> 9
- net /controle/SWDIO: track 46.1 -> 39.1 mm
- net +5V: track 19.1 -> 14.3 mm, vias 10 -> 9
- net GND: track 53.6 -> 50.0 mm, vias 71 -> 69
- net Net-(IC1002-EN/SYNC): track 12.0 -> 10.3 mm
- net Net-(IC1002-VCC): track 17.5 -> 16.0 mm
- net /controle/BTN_MODE: track 31.6 -> 30.2 mm
- net /acquisition/TX_LIDAR: track 51.5 -> 50.4 mm
- net /controle/VCP_TX: track 42.9 -> 43.7 mm
- net /Deplacement/Encoder B phase 2: track 18.5 -> 17.8 mm
- net /Deplacement/FWD2: track 8.40 -> 7.81 mm
- net Net-(IC1002-SW): track 11.5 -> 12.1 mm
- net /Deplacement/VREF1: track 18.8 -> 19.3 mm
- added copper zone on In2.Cu, net +5V
- added copper zone on In2.Cu, net +BATT

Commit message: maj final aprés correction du prof + logo ensea
Parts:
- added C203: 100nF, Capacitor_SMD:C_0402_1005Metric, F.Cu at (67.7, 67.7)
- added G***: LOGO, kicad:ensea-logo, F.Cu at (50.5, 51.3)
- moved C6 13.3 mm to (67.3, 72.1), turned to -90 degrees
- moved C701 3.81 mm to (57.0, 51.7), turned to 90 degrees
- moved C801 3.15 mm to (51.2, 69.1), turned to 180 degrees
- moved C3 3.10 mm to (73.0, 58.0), turned to 180 degrees
- moved C802 3.05 mm to (48.1, 69.1)
- moved C4 2.74 mm to (70.2, 57.9), turned to 0 degrees
- moved C201 2.52 mm to (60.8, 62.6)
- moved C702 2.29 mm to (57.0, 48.6), turned to -90 degrees
- moved L1 2.14 mm to (60.2, 60.6), turned to 0 degrees
- moved C1013 1.89 mm to (86.7, 77.9)
- moved C8 1.77 mm to (68.2, 74.0), turned to 180 degrees
- moved G*** 1.61 mm to (62.6, 84.4)
- moved R1 1.55 mm to (69.6, 68.7)
- moved C1 1.55 mm to (73.1, 70.0)
- moved C2 1.55 mm to (69.6, 67.7)
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Connections:
- C201 pad 1: +3.3V -> Net-(U1-VDDA)
Routing:
- net Net-(IC1002-SW): track 12.1 -> 2.88 mm
- net GND: track 50.0 -> 45.7 mm, vias 69 -> 63
- net Net-(U1-VDDA): track 1.81 -> 5.84 mm
- net +BATT: track 25.1 -> 21.3 mm, vias 9 -> 10
- net +5V: track 14.3 -> 11.0 mm
- net +3.3V: track 22.9 -> 25.0 mm, vias 16 -> 13
- net Net-(U1-PF1): track 1.98 -> 3.73 mm
- net Net-(U1-PF0): track 7.68 -> 9.18 mm
- net Net-(C1013-Pad1): track 2.51 -> 1.28 mm
- net /acquisition/AG_INT1: track 23.1 -> 24.2 mm
- net /acquisition/TOF2: track 40.8 -> 41.6 mm
- net /controle/VCP_TX: track 43.7 -> 44.5 mm
- net /controle/VCP_RX: track 49.0 -> 49.7 mm
- net Net-(IC1002-BST): track 2.63 -> 1.94 mm
- net /acquisition/RX_LIDAR: track 49.6 -> 50.3 mm
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- added copper zone on F.Cu, net +5V
- added copper zone on B.Cu, net GND
- added copper zone on F.Cu, net GND
- added copper zone on F.Cu, net Net-(IC1002-SW)
Other:
- board text added: "+3.3V"
- board text added: "+5V"
- board text added: "BATTERY"
- board text added: "Batt"
- board text added: "CS"
- board text added: "Capteurs bordures"
- board text added: "Driver 1"
- board text added: "Driver 2"
- board text added: "FWD"
- board text added: "Lidar"
- board text added: "MISO"
- board text added: "MOSI"
- board text added: "Mode"
- board text added: "Moteur 1"
- board text added: "Moteur 2"
- board text added: "ON/OFF"
- board text added: "PG/VCC"
- board text added: "Quartz"
- board text added: "REV"
- board text added: "Régul/+3.3V"
- board text added: "Régul/+5V"
- board text added: "SCLK"
- board text added: "ST Link"
- board text added: "Start"
- board text added: "VCP RX"
- board text added: "VCP TX"

Commit message: Modif
dernier_Modification
Parts:
- removed the G*** at (62.6, 84.4)
- added G***: LOGO, LOGO:V-NOM, F.Cu at (63.6, 81.6)
Routing:
- net +5V: track 11.0 -> 9.23 mm
- net /controle/SWDIO: track 39.1 -> 38.4 mm

Commit message: final
Connections:
- U1 pad 10: unconnected-(U1-PA2-Pad10) -> /acquisition/TOF1
- U1 pad 3: /acquisition/TOF1 -> unconnected-(U1-PC14-Pad3)
Routing:
- net /acquisition/TOF1: track 26.1 -> 29.9 mm, vias 0 -> 2
- net /controle/NRST: track 31.2 -> 32.4 mm
- net /acquisition/TOF2: track 41.6 -> 41.0 mm

Commit message: FINAL
Parts:
- removed the G*** at (63.6, 81.6)
- added G***: LOGO, LOGO:LOGO, F.Cu at (66.1, 84.4)
- moved G*** 0.26 mm to (50.7, 51.1)
Routing:
- net /acquisition/TOF1: track 29.9 -> 30.4 mm
